File: SkywalkerPID/SkywalkerPID.kicad_sch (KiCad schematic)
At the start: 27 parts

Commit message: update
Connections:
- net at N2.: now also Check_Valve4., Electronic_Reg1., Solenoid3.
- net at QD2.: now also Check_Valve3.
- net at Check_Valve3.: now also Ball_Valve2., Nitrous1.; no longer QD2.
- new net: Check_Valve1., Ethanol1., SPRV1.
- new net: Check_Valve1., Check_Valve2., Electronic_Reg1.
- new net: Check_Valve2., Nitrous1., PT3., SPRV2.
- new net: Ball_Valve1., Ethanol1., Manual_Ball_Valve1.
- now unconnected: Ball_Valve1., Ball_Valve2., PT3., SPRV1., SPRV2., Solenoid3.
Other:
- note removed: "ENGINE"
Changed lines of the file:
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@@
 		)
 	)
-	(text "ENGINE\n"
-		(exclude_from_sim no)
-		(at 105.664 139.954 0)
-		(effects
-			(font
-				(size 1.27 1.27)
-			)
-		)
-	)
-	(symbol
-		(lib_name "P_ID_symbols:Check_Valve")
+	(symbol
 		(lib_id "P_ID_symbols:Check_Valve")
 		(at 101.6 52.07 270)
@@
 	)
 	(symbol
-		(lib_name "P_ID_symbols:Tank")
 		(lib_id "P_ID_symbols:Tank")
 		(at 104.14 26.67 0)
@@
 	)
 	(symbol
-		(lib_name "P_ID_symbols:Quick_Disconnect")
 		(lib_id "P_ID_symbols:Quick_Disconnect")
 		(at 138.43 132.08 90)
@@
 	)
 	(symbol
-		(lib_name "P_ID_symbols:Pressure_Transducer")
 		(lib_id "P_ID_symbols:Pressure_Transducer")
 		(at 120.65 139.7 0)
@@
 	)
 	(symbol
-		(lib_name "P_ID_symbols:Tank")
 		(lib_id "P_ID_symbols:Tank")
 		(at 107.95 90.17 0)
@@
 	)
 	(symbol
-		(lib_name "P_ID_symbols:Burst_Disc")
 		(lib_id "P_ID_symbols:Burst_Disc")
 		(at 74.93 74.93 0)
@@
 	)
 	(symbol
-		(lib_name "P_ID_symbols:Tank")
 		(lib_id "P_ID_symbols:Tank")
 		(at 100.33 90.17 0)
@@
 	)
 	(symbol
-		(lib_name "P_ID_symbols:Solenoid")
 		(lib_id "P_ID_symbols:Solenoid")
 		(at 121.92 27.94 90)
@@
 	)
 	(symbol
-		(lib_name "P_ID_symbols:Pressure_Transducer")
 		(lib_id "P_ID_symbols:Pressure_Transducer")
 		(at 92.71 96.52 0)
@@
 	)
 	(symbol
-		(lib_name "P_ID_symbols:Check_Valve")
 		(lib_id "P_ID_symbols:Check_Valve")
 		(at 147.32 30.48 180)
@@
 	)
 	(symbol
-		(lib_name "P_ID_symbols:Solenoid")
 		(lib_id "P_ID_symbols:Solenoid")
 		(at 133.985 106.68 0)
@@
 	)
 	(symbol
-		(lib_name "P_ID_symbols:Ball_Valve")
 		(lib_id "P_ID_symbols:Ball_Valve")
 		(at 118.11 76.2 0)
@@
 	)
 	(symbol
-		(lib_name "P_ID_symbols:Burst_Disc")
 		(lib_id "P_ID_symbols:Burst_Disc")
 		(at 130.81 82.55 0)
@@
 	)
 	(symbol
-		(lib_name "P_ID_symbols:Check_Valve")
 		(lib_id "P_ID_symbols:Check_Valve")
 		(at 109.22 52.07 270)
@@
 	)
 	(symbol
-		(lib_name "P_ID_symbols:SPRV")
 		(lib_id "P_ID_symbols:SPRV")
 		(at 59.69 68.58 0)
@@
 	)
 	(symbol
-		(lib_name "P_ID_symbols:Ball_Valve")
 		(lib_id "P_ID_symbols:Ball_Valve")
 		(at 109.22 128.27 90)
@@
 	)
 	(symbol
-		(lib_name "P_ID_symbols:Pressure_Transducer")
 		(lib_id "P_ID_symbols:Pressure_Transducer")
 		(at 119.38 96.52 0)
@@
 	)
 	(symbol
-		(lib_name "P_ID_symbols:Ball_Valve")
 		(lib_id "P_ID_symbols:Ball_Valve")
 		(at 71.12 115.57 0)
@@
 	)
 	(symbol
-		(lib_name "P_ID_symbols:Check_Valve")
 		(lib_id "P_ID_symbols:Check_Valve")
 		(at 138.43 125.73 90)
@@
 	)
 	(symbol
-		(lib_name "P_ID_symbols:SPRV")
 		(lib_id "P_ID_symbols:SPRV")
 		(at 133.35 71.12 0)
@@
 	)
 	(symbol
-		(lib_name "P_ID_symbols:Quick_Disconnect")
 		(lib_id "P_ID_symbols:Quick_Disconnect")
 		(at 162.56 140.97 90)
@@
 	)
 	(symbol
-		(lib_name "P_ID_symbols:Solenoid")
 		(lib_id "P_ID_symbols:Solenoid")
 		(at 78.105 106.68 0)
@@
 	)
 	(symbol
-		(lib_name "P_ID_symbols:Pressure_Transducer")
 		(lib_id "P_ID_symbols:Pressure_Transducer")
 		(at 119.38 59.69 0)
@@
 	)
 	(symbol
-		(lib_name "P_ID_symbols:Quick_Disconnect")
 		(lib_id "P_ID_symbols:Quick_Disconnect")
 		(at 63.5 128.27 90)
@@
 	)
 	(symbol
-		(lib_name "P_ID_symbols:Ball_Valve")
 		(lib_id "P_ID_symbols:Ball_Valve")
 		(at 101.6 128.27 90)
@@
 	)
 	(symbol
-		(lib_name "P_ID_symbols:Pressure_Transducer")
 		(lib_id "P_ID_symbols:Pressure_Transducer")
 		(at 90.17 139.7 0)
