File: AnswerKey.kicad_sch (KiCad schematic)
At the start: 37 parts

Commit message: added hotfire P&ID setup
Parts:
- gave numbers to parts that had none: 1
Connections:
- net at N2.: now also Check_Valve8., Pressure_Regulator2., Pressure_Regulator3.
- net at Engine2.: now also PT6.; no longer PT10.
- net at PT6.: no longer Engine2.
- net at Pmatic_B_Valve3.: now also PnSOL1.
- net at PnSOL1.: now also Ball_Valve19., Ball_Valve9., PnSol2., PnSol3.; no longer Pmatic_B_Valve3.
- net at Solenoid5.: now also Ball_Valve9., Solenoid6.
- net at QD5.: now also Check_Valve7.
- net at Check_Valve7.: now also Nitrous2., Pmatic_B_Valve1.; no longer QD5.
- net at PT8.: now also Check_Valve6., Nitrous2., SPRV4.
- new net: Engine2., PT10.
- new net: Ball_Valve6., Ball_Valve7., Engine2.
- new net: Check_Valve5., Check_Valve6., Pressure_Regulator2.
- new net: Check_Valve5., Ethanol2., SPRV3.
- now unconnected: Pmatic_B_Valve1., SPRV3., SPRV4., Solenoid6.
Changed lines of the file:
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@@
 		(dnp no)
 		(fields_autoplaced yes)
-		(property "Reference" "Ball_Valve?"
+		(property "Reference" "Ball_Valve19"
 			(at 186.69 22.86 0)
 			(effects
@@
 			(project ""
 				(path "/045f1f05-3134-4b6d-91b6-463031104f1e/8ff5724e-b29b-49c2-a1fa-190081404476"
-					(reference "Ball_Valve?")
+					(reference "Ball_Valve19")
 					(unit 1)
 				)

Commit message: no message
Connections:
- net at N2.: now also Check_Valve8., Pressure_Regulator2., Pressure_Regulator3.
- net at Engine2.: now also PT6.; no longer PT10.
- net at PT6.: no longer Engine2.
- net .: now reaches PT9.
- net .: now also Ball_Valve8., Burst_Disc3., Burst_Disc4., PT7., Pmatic_B_Valve2., Solenoid4.
- net at Pmatic_B_Valve3.: now also PnSOL1.
- net at PnSOL1.: now also Ball_Valve19., Ball_Valve9., PnSol2., PnSol3.; no longer Pmatic_B_Valve3.
- net ATM: now reaches Solenoid5.
- net ATM: now also Ball_Valve8., Pmatic_B_Valve2., SPRV3., SPRV4., Solenoid4., Solenoid6.
- net at QD5.: now also Check_Valve7.
- net at Check_Valve7.: now also Nitrous2., Pmatic_B_Valve1.; no longer QD5.
- net at PT8.: now also Check_Valve6., Nitrous2., SPRV4.
- new net: Engine2., PT10.
- new net: Ball_Valve6., Ball_Valve7., Engine2.
- new net: Check_Valve5., Check_Valve6., Pressure_Regulator2.
- new net: Check_Valve5., Ethanol2., SPRV3.
- new net: Ball_Valve9., Solenoid5., Solenoid6.
- now unconnected: Pmatic_B_Valve1.
Changed lines of the file:
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@@
+		)
+	)
+	(label "."
+		(at 142.24 86.36 0)
+		(fields_autoplaced yes)
+		(effects
+			(font
+				(size 1.27 1.27)
+			)
+			(justify left bottom)
+		)
+	)
+	(label "ATM"
+		(at 101.6 73.66 180)
+		(fields_autoplaced yes)
+		(effects
+			(font
+				(size 1.27 1.27)
+			)
+			(justify right bottom)
+		)
+	)
+	(label "ATM"
+		(at 240.03 35.56 0)
+		(fields_autoplaced yes)
+		(effects
+			(font
+				(size 1.27 1.27)
+			)
+			(justify left bottom)
+		)
+	)
+	(label "ATM"
+		(at 190.5 73.66 0)
+		(fields_autoplaced yes)
+		(effects
+			(font
+				(size 1.27 1.27)
+			)
+			(justify left bottom)
+		)
+	)
+	(label "."
+		(at 157.48 87.63 0)
+		(fields_autoplaced yes)
+		(effects
+			(font
+				(size 1.27 1.27)
+			)
+			(justify left bottom)
+		)
+	)
+	(label "."
+		(at 157.48 95.25 0)
+		(fields_autoplaced yes)
+		(effects
+			(font
+				(size 1.27 1.27)
+			)
+			(justify left bottom)
+		)
+	)
+	(label "ATM"
+		(at 184.15 107.95 0)
+		(fields_autoplaced yes)
+		(effects
+			(font
+				(size 1.27 1.27)
+			)
+			(justify left bottom)
+		)
+	)
+	(label "."
+		(at 154.94 97.79 0)
+		(fields_autoplaced yes)
+		(effects
+			(font
+				(size 1.27 1.27)
+			)
+			(justify left bottom)
+		)
+	)
+	(label "ATM"
+		(at 172.72 81.28 0)
+		(fields_autoplaced yes)
+		(effects
+			(font
+				(size 1.27 1.27)
+			)
+			(justify left bottom)
+		)
+	)
+	(label "."
+		(at 144.78 97.79 0)
+		(fields_autoplaced yes)
+		(effects
+			(font
+				(size 1.27 1.27)
+			)
+			(justify left bottom)
+		)
+	)
+	(label "."
+		(at 142.24 95.25 0)
+		(fields_autoplaced yes)
+		(effects
+			(font
+				(size 1.27 1.27)
+			)
+			(justify left bottom)
+		)
+	)
+	(label "ATM"
+		(at 111.76 111.76 180)
+		(fields_autoplaced yes)
+		(effects
+			(font
+				(size 1.27 1.27)
+			)
+			(justify right bottom)
+		)
+	)
+	(label "ATM"
+		(at 240.03 24.13 0)
+		(fields_autoplaced yes)
+		(effects
+			(font
+				(size 1.27 1.27)
+			)
+			(justify left bottom)
+		)
+	)
+	(label "."
+		(at 154.94 83.82 0)
+		(fields_autoplaced yes)
+		(effects
+			(font
+				(size 1.27 1.27)
+			)
+			(justify left bottom)
 		)
 	)

Commit message: update, someone needs to finish adding torch igniter to answerkey, allow it im on holi
Parts:
- removed Pmatic_B_Valve2: ~, symbol PID_symbols:Pneumatic_Rotary_Ball_Valve
- added Ball_Valve?: ~, symbol PID_symbols:Ball_Valve
- added Check_Valve?: ~, symbol PID_symbols:Check_Valve
- added G_N20, T?: ~, symbol PID_symbols:Tank
- added Pmatic_B_Valve?: ~, symbol PID_symbols:Pneumatic_Rotary_Ball_Valve
- added Pressure_Regulator?: ~, symbol PID_symbols:Pressure_Regulator
Connections:
- net ATM: now also Pmatic_B_Valve?.
- net at N2.: now also Check_Valve8., Pressure_Regulator2., Pressure_Regulator3.
- net at Engine2.: now also PT6.; no longer PT10.
- net at PT6.: no longer Engine2.
- net at Pmatic_B_Valve3.: now also PnSOL1.
- net at PnSOL1.: now also Ball_Valve19., Ball_Valve9., PnSol2., PnSol3.; no longer Pmatic_B_Valve3.
- net at QD5.: now also Check_Valve7.
- net at PT8.: now also Check_Valve6., Nitrous2., SPRV4.
- new net: Engine2., PT10.
- new net: Ball_Valve6., Ball_Valve7., Engine2.
- new net: Check_Valve5., Check_Valve6., Pressure_Regulator2., Pressure_Regulator?.
- new net: Check_Valve5., Ethanol2., SPRV3.
- new net: Check_Valve?., G_N20.
- new net: Ball_Valve?., Check_Valve?.
- new net: Pmatic_B_Valve?., PnSol3.
- new net: Check_Valve7., Nitrous2., Pmatic_B_Valve1., Pmatic_B_Valve?.
- new net: Ball_Valve9., Solenoid5., Solenoid6.
- now unconnected: Pmatic_B_Valve1.
Other:
- moved on the sheet: Ball_Valve19, Ball_Valve5, Ball_Valve6, Ball_Valve7, Ball_Valve8, Ball_Valve9, Burst_Disc3, Burst_Disc4, Check_Valve5, Check_Valve6, Check_Valve7, Check_Valve8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
