File: AnswerKey.kicad_sch (KiCad schematic)
At the start: 46 parts

Commit message: no message
Parts:
- removed Reg? (x2): ~, symbol PID_symbols:Pressure_Regulator
Connections:
- net at N2.: now also Check_Valve9., Reg?., Reg?.
- net at Engine2.: now also PT6.; no longer PT10.
- net at PT6.: no longer Engine2.
- net at EthBuffer?.: now also Solenoid?.; no longer Ball_Valve?.
- net at Solenoid?.: now also T_I?.; no longer EthBuffer?.
- net at G_N?.: now also Solenoid?.; no longer Ball_Valve?.
- net at Solenoid?.: now also T_I?.; no longer G_N?.
- net at Pmatic_B_Valve2.: now also PnSOL1.
- net at PnSOL1.: now also Ball_Valve?., Ball_Valve?., PnSol2., PnSol?.; no longer Pmatic_B_Valve2.
- net at Pmatic_B_Valve3.: now also PnSol?.
- net at QD5.: now also Check_Valve10.
- net at Check_Valve10.: now also Nitrous2.; no longer QD5.
- new net: Engine2., PT10.
- new net: Ball_Valve6., Ball_Valve7., Engine2.
- new net: Check_Valve7., Ethanol2., SPRV3.
- new net: Ball_Valve?., EthBuffer?.
- new net: Ball_Valve?., G_N?.
- new net: Ball_Valve?., Solenoid6., Solenoid?.
- new net: Check_Valve8., Nitrous2., SPRV4.
Changed lines of the file:
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@@
-	)
-	(symbol
-		(lib_id "PID_symbols:Pressure_Regulator")
-		(at 160.02 91.44 0)
-		(unit 1)
-		(exclude_from_sim no)
-		(in_bom yes)
-		(on_board yes)
-		(dnp no)
-		(property "Reference" "Reg?"
-			(at 160.274 86.106 0)
-			(effects
-				(font
-					(size 1.27 1.27)
-				)
-			)
-		)
-		(property "Value" "~"
-			(at 163.8925 85.09 0)
-			(effects
-				(font
-					(size 1.27 1.27)
-				)
-			)
-		)
-		(property "Footprint" ""
-			(at 160.02 91.44 0)
-			(effects
-				(font
-					(size 1.27 1.27)
-				)
-				(hide yes)
-			)
-		)
-		(property "Datasheet" ""
-			(at 160.02 91.44 0)
-			(effects
-				(font
-					(size 1.27 1.27)
-				)
-				(hide yes)
-			)
-		)
-		(property "Description" "Pressure Regulator"
-			(at 160.02 91.44 0)
-			(effects
-				(font
-					(size 1.27 1.27)
-				)
-				(hide yes)
-			)
-		)
-		(pin ""
-		)
-		(pin ""
-		)
 	)
 	(symbol
@@
 			(effects
 				(font
-					(size 1.27 1.27)
-				)
-				(hide yes)
-			)
-		)
-		(pin ""
-		)
-		(pin ""
-		)
-	)
-	(symbol
-		(lib_id "PID_symbols:Pressure_Regulator")
-		(at 171.45 102.87 90)
-		(unit 1)
-		(exclude_from_sim no)
-		(in_bom yes)
-		(on_board yes)
-		(dnp no)
-		(fields_autoplaced yes)
-		(property "Reference" "Reg?"
-			(at 175.26 98.3624 90)
-			(effects
-				(font
-					(size 1.27 1.27)
-				)
-				(justify right)
-			)
-		)
-		(property "Value" "~"
-			(at 175.26 100.2675 90)
-			(effects
-				(font
-					(size 1.27 1.27)
-				)
-				(justify right)
-			)
-		)
-		(property "Footprint" ""
-			(at 171.45 102.87 0)
-			(effects
-				(font
-					(size 1.27 1.27)
-				)
-				(hide yes)
-			)
-		)
-		(property "Datasheet" ""
-			(at 171.45 102.87 0)
-			(effects
-				(font
-					(size 1.27 1.27)
-				)
-				(hide yes)
-			)
-		)
-		(property "Description" "Pressure Regulator"
-			(at 171.45 102.87 0)
-			(effects
-				(font
