File: AnswerKey1.kicad_sch (KiCad schematic)
At the start: 46 parts

Commit message: camebackfromhol
Parts:
- removed Ball_Valve? (x2): ~, symbol PID_symbols:Ball_Valve
- removed Solenoid? (x2): ~, symbol PID_symbols:Solenoid
- added Ball_Valve9Pneumatic?, Ball_ValvePneumatic?: ~, symbol PID_symbols:Ball_Valve
- renumbered Ball_Valve7 to Ball_Valve?, Ball_Valve6 to Ball_Valve?, Ball_Valve10 to Ball_Valve?, Ball_Valve5 to Ball_Valve?, Burst_Disc4 to Burst_Disc?, Burst_Disc3 to Burst_Disc?, Check_Valve9 to Check_Valve?, Check_Valve7 to Check_Valve?, Check_Valve10 to Check_Valve?, Check_Valve8 to Check_Valve?, Engine2 to Engine?, Ethanol2 to Ethanol?, N2 to N?, Nitrous2 to Nitrous?, PT10 to PT?, PT9 to PT?, PT6 to PT?, PT7 to PT?, Pmatic_B_Valve2 to Pmatic_B_Valve?, Pmatic_B_Valve3 to Pmatic_B_Valve?, Pmatic_B_Valve1 to Pmatic_B_Valve?, PnSOL1 to PnSOL?, PnSol2 to PnSol?, QD6 to QD?, QD5 to QD?, QD4 to QD?, SPRV3 to SPRV?, SPRV4 to SPRV?, Solenoid6 to Solenoid?, Solenoid4 to Solenoid?
Connections:
- net .: now also Ball_ValvePneumatic?.
- net at N?.: now also Check_Valve?., Reg?., Reg?.
- net at Engine?.: now also PT?.; no longer PT?.
- net at PT?.: no longer Engine?.
- net at EthBuffer?.: now also T_I?.
- net at G_N?.: now also T_I?.
- net at Ball_Valve?., Ball_Valve?., Ethanol?.: now also Ball_Valve9Pneumatic?.
- net at Pmatic_B_Valve?.: now also PnSOL?.
- net at PnSOL?.: now also Ball_Valve?., Ball_Valve?., PnSol?., PnSol?.; no longer Pmatic_B_Valve?.
- net at Pmatic_B_Valve?.: now also PnSol?.
- net at QD?.: now also Check_Valve?.
- net at Check_Valve?.: now also Nitrous?.; no longer QD?.
- net at Reg?.: now also Ball_Valve?., Reg?.
- new net: Engine?., PT?.
- new net: Ball_Valve?., Ball_Valve?., Engine?.
- new net: Check_Valve?., Ethanol?., SPRV?.
- new net: Ball_Valve9Pneumatic?., EthBuffer?.
- new net: Ball_ValvePneumatic?., G_N?.
- new net: Ball_Valve?., Solenoid?., Solenoid?.
- new net: Check_Valve?., Nitrous?., SPRV?.
- now unconnected: Reg?.
Other:
- moved on the sheet: EthBuffer?, G_N?, T_I?
