File: Hopper_Hotfire_TestStand.kicad_sch (KiCad schematic)
At the start: 27 parts

Commit message: no message
Parts:
- added Flow_Sensor: ~, symbol PID_symbols:Pneumatic_Rotary_Ball_Valve
- gave numbers to parts that had none: 27
Connections:
- net at Check_Valve9.: now also Ball_Valve12., Nitrous_PT1., Thomas1.; no longer Nitrous_Fill1.
- net at Ball_Valve14.: now also Check_Valve11., Solenoid8.
- net at Fuel_Injector_PT1.: now also Ball_Valve13., Engine3.
- net at Nitrogen_PT1.: now also N2CYL1., Pressure_Regulator4.
- new net: Check_Valve9., Nitrous_Fill1.
- new net: Ball_Valve12., Engine3., Ox_Injector_PT1.
- new net: Ball_Valve11., Burst_Disc5., Check_Valve10., Check_Valve11., SPRV5.
- new net: Flow_Sensor., Fuel_PT1., Fuel_Tank2., Needle_Valve1.
- new net: Ball_Valve13., Flow_Sensor.
- now unconnected: Burst_Disc5., Engine3., Engine3., Fuel_PT1., Fuel_Tank2., N2CYL1., Nitrous_PT1., Ox_Injector_PT1., SPRV5., Solenoid8.
Other:
- moved on the sheet: N2CYL1

Commit message: no message
Parts:
- renumbered Ball_Valve13 to Fuel_Main, Ball_Valve11 to Nitrogen_Fill, Ball_Valve10 to Nitrous_Vent, Ball_Valve12 to Ox_Vent
Connections:
- net at Check_Valve9.: now also Nitrous_PT1., Ox_Vent., Thomas1.; no longer Nitrous_Fill1.
- net at Ball_Valve14.: now also Check_Valve11., Solenoid8.
- net at Fuel_Injector_PT1.: now also Engine3., Fuel_Main.
- net at Flow_Sensor.: now also Fuel_Main.
- net at Nitrogen_PT1.: now also N2CYL1., Pressure_Regulator4.
- new net: Check_Valve9., Nitrous_Fill1.
- new net: Engine3., Ox_Injector_PT1., Ox_Vent.
- new net: Burst_Disc5., Check_Valve10., Check_Valve11., Nitrogen_Fill., SPRV5.
- new net: Flow_Sensor., Fuel_PT1., Fuel_Tank2., Needle_Valve1.
- now unconnected: Burst_Disc5., Engine3., Engine3., Fuel_PT1., Fuel_Tank2., N2CYL1., Nitrous_PT1., Ox_Injector_PT1., SPRV5., Solenoid8.
Changed lines of the file:
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@@
 		)
 		(stroke
-			(width 0)
+			(width 0.635)
 			(type default)
 		)
@@
 		(on_board yes)
 		(dnp no)
-		(property "Reference" "Ball_Valve12"
+		(property "Reference" "Ox_Vent"
 			(at 123.698 132.08 90)
 			(effects
@@
 			(project "P_IDs"
 				(path "/045f1f05-3134-4b6d-91b6-463031104f1e/12264f82-10ad-4f8b-aee0-7883d457c15c"
-					(reference "Ball_Valve12")
+					(reference "Ox_Vent")
 					(unit 1)
 				)
@@
 		(dnp no)
 		(fields_autoplaced yes)
-		(property "Reference" "Ball_Valve11"
+		(property "Reference" "Nitrogen_Fill"
 			(at 134.62 62.8649 90)
 			(effects
@@
 			(project "P_IDs"
 				(path "/045f1f05-3134-4b6d-91b6-463031104f1e/12264f82-10ad-4f8b-aee0-7883d457c15c"
-					(reference "Ball_Valve11")
+					(reference "Nitrogen_Fill")
 					(unit 1)
 				)
@@
 		(on_board yes)
 		(dnp no)
-		(property "Reference" "Ball_Valve10"
+		(property "Reference" "Nitrous_Vent"
 			(at 129.54 83.566 0)
 			(effects
@@
 			(project "P_IDs"
 				(path "/045f1f05-3134-4b6d-91b6-463031104f1e/12264f82-10ad-4f8b-aee0-7883d457c15c"
-					(reference "Ball_Valve10")
+					(reference "Nitrous_Vent")
 					(unit 1)
 				)
@@
 		(on_board yes)
 		(dnp no)
-		(property "Reference" "Ball_Valve13"
+		(property "Reference" "Fuel_Main"
 			(at 163.322 132.08 90)
 			(effects
@@
 			(project "P_IDs"
 				(path "/045f1f05-3134-4b6d-91b6-463031104f1e/12264f82-10ad-4f8b-aee0-7883d457c15c"
-					(reference "Ball_Valve13")
-					(unit 1)
-				)
+					(reference "Fuel_Main")
+					(unit 1)
+				)

Commit message: camebackfromhol
Parts:
- renumbered Ball_Valve14 to Ball_Valve13, Check_Valve9 to Check_Valve11, Check_Valve10 to Check_Valve12, Check_Valve11 to Check_Valve13, Flow_Sensor to Flow_Sensor1, Fuel_Main to Fuel_Main1, Nitrogen_Fill to Nitrogen_Fill1, Nitrous_Vent to Nitrous_Vent1, Ox_Vent to Ox_Vent1, Pressure_Regulator4 to Pressure_Regulator7
Connections:
- net at Check_Valve11.: now also Nitrous_PT1., Ox_Vent1., Thomas1.; no longer Nitrous_Fill1.
- net at Ball_Valve13.: now also Check_Valve13., Solenoid8.
- net at Fuel_Injector_PT1.: now also Engine3., Fuel_Main1.
- net at Flow_Sensor1.: now also Fuel_Main1.
- net at Nitrogen_PT1.: now also N2CYL1., Pressure_Regulator7.
- new net: Check_Valve11., Nitrous_Fill1.
- new net: Engine3., Ox_Injector_PT1., Ox_Vent1.
- new net: Burst_Disc5., Check_Valve12., Check_Valve13., Nitrogen_Fill1., SPRV5.
- new net: Flow_Sensor1., Fuel_PT1., Fuel_Tank2., Needle_Valve1.
- now unconnected: Burst_Disc5., Engine3., Engine3., Fuel_PT1., Fuel_Tank2., N2CYL1., Nitrous_PT1., Ox_Injector_PT1., SPRV5., Solenoid8.
Changed lines of the file:
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@@
 	)
 	(symbol
-		(lib_name "Check_Valve_2")
 		(lib_id "PID_symbols:Check_Valve")
 		(at 99.06 104.14 0)
@@
 		(on_board yes)
 		(dnp no)
-		(property "Reference" "Check_Valve9"
+		(property "Reference" "Check_Valve11"
 			(at 100.584 111.506 0)
 			(effects
@@
 			(project "P_IDs"
 				(path "/045f1f05-3134-4b6d-91b6-463031104f1e/12264f82-10ad-4f8b-aee0-7883d457c15c"
-					(reference "Check_Valve9")
-					(unit 1)
-				)
-			)
-		)
-	)
-	(symbol
-		(lib_name "Ball_Valve_8")
+					(reference "Check_Valve11")
+					(unit 1)
+				)
+			)
+		)
+	)
+	(symbol
 		(lib_id "PID_symbols:Ball_Valve")
 		(at 49.53 69.85 270)
@@
 	)
 	(symbol
-		(lib_name "Ball_Valve_5")
 		(lib_id "PID_symbols:Ball_Valve")
 		(at 151.13 85.09 0)
@@
 		(on_board yes)
 		(dnp no)
-		(property "Reference" "Ball_Valve14"
+		(property "Reference" "Ball_Valve13"
 			(at 154.94 90.17 0)
 			(effects
@@
 			(project "P_IDs"
 				(path "/045f1f05-3134-4b6d-91b6-463031104f1e/12264f82-10ad-4f8b-aee0-7883d457c15c"
-					(reference "Ball_Valve14")
-					(unit 1)
-				)
-			)
-		)
-	)
-	(symbol
-		(lib_name "Ball_Valve_7")
+					(reference "Ball_Valve13")
+					(unit 1)
+				)
+			)
+		)
+	)
+	(symbol
 		(lib_id "PID_symbols:Ball_Valve")
 		(at 137.16 135.89 90)
@@
 		(on_board yes)
 		(dnp no)
-		(property "Reference" "Ox_Vent"
+		(property "Reference" "Ox_Vent1"
 			(at 123.698 132.08 90)
 			(effects
@@
 			(project "P_IDs"
 				(path "/045f1f05-3134-4b6d-91b6-463031104f1e/12264f82-10ad-4f8b-aee0-7883d457c15c"
-					(reference "Ox_Vent")
+					(reference "Ox_Vent1")
 					(unit 1)
 				)
@@
 	)
 	(symbol
-		(lib_name "Check_Valve_1")
 		(lib_id "PID_symbols:Check_Valve")
 		(at 140.97 69.85 0)
@@
 		(on_board yes)
 		(dnp no)
-		(property "Reference" "Check_Valve11"
+		(property "Reference" "Check_Valve13"
 			(at 143.51 73.914 0)
 			(effects
@@
 			(project "P_IDs"
 				(path "/045f1f05-3134-4b6d-91b6-463031104f1e/12264f82-10ad-4f8b-aee0-7883d457c15c"
-					(reference "Check_Valve11")
+					(reference "Check_Valve13")
 					(unit 1)
 				)
@@
 	)
 	(symbol
-		(lib_name "Solenoid_1")
 		(lib_id "PID_symbols:Solenoid")
 		(at 151.13 78.74 0)
@@
 	)
 	(symbol
-		(lib_name "Pressure_Transducer_2")
 		(lib_id "PID_symbols:Pressure_Transducer")
 		(at 114.3 114.3 0)
@@
 	)
 	(symbol
-		(lib_name "Needle_Valve_1")
 		(lib_id "PID_symbols:Needle_Valve")
 		(at 181.61 69.85 0)
@@
 	)
 	(symbol
-		(lib_name "Tank_5")
 		(lib_id "PID_symbols:Tank")
 		(at 109.22 99.06 0)
@@
 	)
 	(symbol
-		(lib_name "SPRV_1")
 		(lib_id "PID_symbols:SPRV")
 		(at 110.49 67.31 90)
@@
 	)
 	(symbol
-		(lib_name "Ball_Valve_4")
 		(lib_id "PID_symbols:Ball_Valve")
 		(at 130.81 59.69 270)
@@
 		(dnp no)
 		(fields_autoplaced yes)
-		(property "Reference" "Nitrogen_Fill"
+		(property "Reference" "Nitrogen_Fill1"
 			(at 134.62 62.8649 90)
 			(effects
@@
 			(project "P_IDs"
 				(path "/045f1f05-3134-4b6d-91b6-463031104f1e/12264f82-10ad-4f8b-aee0-7883d457c15c"
-					(reference "Nitrogen_Fill")
+					(reference "Nitrogen_Fill1")
 					(unit 1)
 				)
@@
 		(dnp no)
 		(fields_autoplaced yes)
-		(property "Reference" "Flow_Sensor"
+		(property "Reference" "Flow_Sensor1"
 			(at 175.26 88.2649 90)
 			(effects
@@
 			(project ""
 				(path "/045f1f05-3134-4b6d-91b6-463031104f1e/12264f82-10ad-4f8b-aee0-7883d457c15c"
-					(reference "Flow_Sensor")
-					(unit 1)
-				)
-			)
-		)
-	)
-	(symbol
-		(lib_name "Pressure_Transducer_4")
+					(reference "Flow_Sensor1")
+					(unit 1)
+				)
+			)
+		)
+	)
+	(symbol
 		(lib_id "PID_symbols:Pressure_Transducer")
 		(at 175.26 80.01 0)
@@
 	)
 	(symbol
-		(lib_name "Pressure_Transducer_3")
 		(lib_id "PID_symbols:Pressure_Transducer")
 		(at 140.97 45.72 0)
@@
 	)
 	(symbol
-		(lib_name "Pressure_Regulator_1")
 		(lib_id "PID_symbols:Pressure_Regulator")
 		(at 130.81 57.15 90)
@@
 		(dnp no)
 		(fields_autoplaced yes)
-		(property "Reference" "Pressure_Regulator4"
+		(property "Reference" "Pressure_Regulator7"
 			(at 134.62 52.6424 90)
 			(effects
@@
 			)
 		)
-		(property "Description" ""
+		(property "Description" "Pressure Regulator"
 			(at 130.81 57.15 0)
 			(effects
@@
 			(project "P_IDs"
 				(path "/045f1f05-3134-4b6d-91b6-463031104f1e/12264f82-10ad-4f8b-aee0-7883d457c15c"
-					(reference "Pressure_Regulator4")
-					(unit 1)
-				)
-			)
-		)
-	)
-	(symbol
-		(lib_name "Tank_3")
+					(reference "Pressure_Regulator7")
+					(unit 1)
+				)
+			)
+		)
+	)
+	(symbol
 		(lib_id "PID_symbols:Tank")
 		(at 129.54 27.94 0)
@@
 	)
 	(symbol
-		(lib_name "Ball_Valve_6")
 		(lib_id "PID_symbols:Ball_Valve")
 		(at 113.03 83.82 0)
@@
 		(on_board yes)
 		(dnp no)
-		(property "Reference" "Nitrous_Vent"
+		(property "Reference" "Nitrous_Vent1"
 			(at 129.54 83.566 0)
 			(effects
@@
 			(project "P_IDs"
 				(path "/045f1f05-3134-4b6d-91b6-463031104f1e/12264f82-10ad-4f8b-aee0-7883d457c15c"
-					(reference "Nitrous_Vent")
-					(unit 1)
-				)
-			)
-		)
-	)
-	(symbol
-		(lib_name "Check_Valve_3")
+					(reference "Nitrous_Vent1")
+					(unit 1)
+				)
+			)
+		)
+	)
+	(symbol
 		(lib_id "PID_symbols:Check_Valve")
 		(at 110.49 72.39 270)
@@
 		(on_board yes)
 		(dnp no)
-		(property "Reference" "Check_Valve10"
+		(property "Reference" "Check_Valve12"
 			(at 112.776 74.93 90)
 			(effects
@@
 			(project "P_IDs"
 				(path "/045f1f05-3134-4b6d-91b6-463031104f1e/12264f82-10ad-4f8b-aee0-7883d457c15c"
-					(reference "Check_Valve10")
-					(unit 1)
-				)
-			)
-		)
-	)
-	(symbol
-		(lib_name "Tank_6")
+					(reference "Check_Valve12")
+					(unit 1)
+				)
+			)
+		)
+	)
+	(symbol
 		(lib_id "PID_symbols:Tank")
 		(at 48.26 64.77 0)
@@
 	)
 	(symbol
-		(lib_name "Solenoid_2")
 		(lib_id "PID_symbols:Solenoid")
 		(at 100.33 83.82 0)
@@
 	)
 	(symbol
-		(lib_name "Tank_4")
 		(lib_id "PID_symbols:Tank")
 		(at 166.37 54.61 0)
@@
 	)
 	(symbol
-		(lib_name "Ball_Valve_4")
 		(lib_id "PID_symbols:Ball_Valve")
 		(at 149.86 128.27 270)
@@
 		(on_board yes)
 		(dnp no)
-		(property "Reference" "Fuel_Main"
+		(property "Reference" "Fuel_Main1"
 			(at 163.322 132.08 90)
 			(effects
@@
 			(project "P_IDs"
 				(path "/045f1f05-3134-4b6d-91b6-463031104f1e/12264f82-10ad-4f8b-aee0-7883d457c15c"
-					(reference "Fuel_Main")
-					(unit 1)
-				)
+					(reference "Fuel_Main1")
+					(unit 1)
+				)

Commit message: deleted answer keys
Parts:
- renumbered Ball_Valve13 to Ball_Valve4, Burst_Disc5 to Burst_Disc3, Check_Valve12 to Check_Valve10, Check_Valve13 to Check_Valve11, Check_Valve11 to Check_Valve9, Engine3 to Engine2, Pressure_Regulator7 to Pressure_Regulator1, SPRV5 to SPRV3, Solenoid7 to Solenoid8, Solenoid8 to Solenoid9
Connections:
- net at Check_Valve9.: now also Nitrous_PT1., Ox_Vent1., Thomas1.; no longer Nitrous_Fill1.
- net at Ball_Valve4.: now also Check_Valve11., Solenoid9.
- net at Fuel_Injector_PT1.: now also Engine2., Fuel_Main1.
- net at Flow_Sensor1.: now also Fuel_Main1.
- net at Nitrogen_PT1.: now also N2CYL1., Pressure_Regulator1.
- new net: Check_Valve9., Nitrous_Fill1.
- new net: Engine2., Ox_Injector_PT1., Ox_Vent1.
- new net: Burst_Disc3., Check_Valve10., Check_Valve11., Nitrogen_Fill1., SPRV3.
- new net: Flow_Sensor1., Fuel_PT1., Fuel_Tank2., Needle_Valve1.
- now unconnected: Burst_Disc3., Engine2., Engine2., Fuel_PT1., Fuel_Tank2., N2CYL1., Nitrous_PT1., Ox_Injector_PT1., SPRV3., Solenoid9.
Changed lines of the file:
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@@
 		(on_board yes)
 		(dnp no)
-		(property "Reference" "Check_Valve11"
+		(property "Reference" "Check_Valve9"
 			(at 100.584 111.506 0)
 			(effects
@@
 			(project "P_IDs"
 				(path "/045f1f05-3134-4b6d-91b6-463031104f1e/12264f82-10ad-4f8b-aee0-7883d457c15c"
-					(reference "Check_Valve11")
+					(reference "Check_Valve9")
 					(unit 1)
 				)
@@
 		(on_board yes)
 		(dnp no)
-		(property "Reference" "Ball_Valve13"
+		(property "Reference" "Ball_Valve4"
 			(at 154.94 90.17 0)
 			(effects
@@
 			(project "P_IDs"
 				(path "/045f1f05-3134-4b6d-91b6-463031104f1e/12264f82-10ad-4f8b-aee0-7883d457c15c"
-					(reference "Ball_Valve13")
+					(reference "Ball_Valve4")
 					(unit 1)
 				)
@@
 		(dnp no)
 		(fields_autoplaced yes)
-		(property "Reference" "Engine3"
+		(property "Reference" "Engine2"
 			(at 149.86 149.4718 0)
 			(effects
@@
 			(project "P_IDs"
 				(path "/045f1f05-3134-4b6d-91b6-463031104f1e/12264f82-10ad-4f8b-aee0-7883d457c15c"
-					(reference "Engine3")
+					(reference "Engine2")
 					(unit 1)
 				)
@@
 		(on_board yes)
 		(dnp no)
-		(property "Reference" "Check_Valve13"
+		(property "Reference" "Check_Valve11"
 			(at 143.51 73.914 0)
 			(effects
@@
 			(project "P_IDs"
 				(path "/045f1f05-3134-4b6d-91b6-463031104f1e/12264f82-10ad-4f8b-aee0-7883d457c15c"
-					(reference "Check_Valve13")
+					(reference "Check_Valve11")
 					(unit 1)
 				)
@@
 		(on_board yes)
 		(dnp no)
-		(property "Reference" "Solenoid8"
+		(property "Reference" "Solenoid9"
 			(at 154.94 71.882 0)
 			(effects
@@
 			(project "P_IDs"
 				(path "/045f1f05-3134-4b6d-91b6-463031104f1e/12264f82-10ad-4f8b-aee0-7883d457c15c"
-					(reference "Solenoid8")
+					(reference "Solenoid9")
 					(unit 1)
 				)
@@
 		(on_board yes)
 		(dnp no)
-		(property "Reference" "Burst_Disc5"
+		(property "Reference" "Burst_Disc3"
 			(at 87.122 70.104 0)
 			(effects
@@
 			(project "P_IDs"
 				(path "/045f1f05-3134-4b6d-91b6-463031104f1e/12264f82-10ad-4f8b-aee0-7883d457c15c"
-					(reference "Burst_Disc5")
+					(reference "Burst_Disc3")
 					(unit 1)
 				)
@@
 		(on_board yes)
 		(dnp no)
-		(property "Reference" "SPRV5"
+		(property "Reference" "SPRV3"
 			(at 107.95 53.34 90)
 			(effects
@@
 			(project "P_IDs"
 				(path "/045f1f05-3134-4b6d-91b6-463031104f1e/12264f82-10ad-4f8b-aee0-7883d457c15c"
-					(reference "SPRV5")
+					(reference "SPRV3")
 					(unit 1)
 				)
@@
 		(dnp no)
 		(fields_autoplaced yes)
-		(property "Reference" "Pressure_Regulator7"
+		(property "Reference" "Pressure_Regulator1"
 			(at 134.62 52.6424 90)
 			(effects
@@
 			(project "P_IDs"
 				(path "/045f1f05-3134-4b6d-91b6-463031104f1e/12264f82-10ad-4f8b-aee0-7883d457c15c"
-					(reference "Pressure_Regulator7")
+					(reference "Pressure_Regulator1")
 					(unit 1)
 				)
@@
 		(on_board yes)
 		(dnp no)
-		(property "Reference" "Check_Valve12"
+		(property "Reference" "Check_Valve10"
 			(at 112.776 74.93 90)
 			(effects
@@
 			(project "P_IDs"
 				(path "/045f1f05-3134-4b6d-91b6-463031104f1e/12264f82-10ad-4f8b-aee0-7883d457c15c"
-					(reference "Check_Valve12")
+					(reference "Check_Valve10")
 					(unit 1)
 				)
@@
 		(on_board yes)
 		(dnp no)
-		(property "Reference" "Solenoid7"
+		(property "Reference" "Solenoid8"
 			(at 89.408 83.82 0)
 			(effects
@@
 			(project "P_IDs"
 				(path "/045f1f05-3134-4b6d-91b6-463031104f1e/12264f82-10ad-4f8b-aee0-7883d457c15c"
-					(reference "Solenoid7")
-					(unit 1)
-				)
+					(reference "Solenoid8")
+					(unit 1)
+				)

Commit message: no message
Parts:
- renumbered Check_Valve9 to Check_Valve7, Check_Valve10 to Check_Valve8, Check_Valve11 to Check_Valve9
Connections:
- net at Check_Valve7.: now also Nitrous_PT1., Ox_Vent1., Thomas1.; no longer Nitrous_Fill1.
- net at Ball_Valve4.: now also Check_Valve9., Solenoid9.
- net at Fuel_Injector_PT1.: now also Engine2., Fuel_Main1.
- net at Flow_Sensor1.: now also Fuel_Main1.
- net at Nitrogen_PT1.: now also N2CYL1., Pressure_Regulator1.
- new net: Check_Valve7., Nitrous_Fill1.
- new net: Engine2., Ox_Injector_PT1., Ox_Vent1.
- new net: Burst_Disc3., Check_Valve8., Check_Valve9., Nitrogen_Fill1., SPRV3.
- new net: Flow_Sensor1., Fuel_PT1., Fuel_Tank2., Needle_Valve1.
- now unconnected: Burst_Disc3., Engine2., Engine2., Fuel_PT1., Fuel_Tank2., N2CYL1., Nitrous_PT1., Ox_Injector_PT1., SPRV3., Solenoid9.
Changed lines of the file:
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@@
 	)
 	(symbol
+		(lib_name "PID_symbols:Pressure_Transducer")
 		(lib_id "PID_symbols:Pressure_Transducer")
 		(at 143.51 135.89 0)
@@
 		(pin ""
 		)
+		(pin ""
+		)
 		(instances
 			(project "P_IDs"
@@
 		(on_board yes)
 		(dnp no)
-		(property "Reference" "Check_Valve9"
+		(property "Reference" "Check_Valve7"
 			(at 100.584 111.506 0)
 			(effects
@@
 			(project "P_IDs"
 				(path "/045f1f05-3134-4b6d-91b6-463031104f1e/12264f82-10ad-4f8b-aee0-7883d457c15c"
-					(reference "Check_Valve9")
-					(unit 1)
-				)
-			)
-		)
-	)
-	(symbol
+					(reference "Check_Valve7")
+					(unit 1)
+				)
+			)
+		)
+	)
+	(symbol
+		(lib_name "PID_symbols:Ball_Valve")
 		(lib_id "PID_symbols:Ball_Valve")
 		(at 49.53 69.85 270)
@@
 	)
 	(symbol
+		(lib_name "PID_symbols:Ball_Valve")
 		(lib_id "PID_symbols:Ball_Valve")
 		(at 151.13 85.09 0)
@@
 	)
 	(symbol
+		(lib_name "PID_symbols:Pressure_Transducer")
 		(lib_id "PID_symbols:Pressure_Transducer")
 		(at 153.67 140.97 0)
@@
 				(hide yes)
 			)
+		)
+		(pin ""
 		)
 		(pin ""
@@
 	)
 	(symbol
+		(lib_name "PID_symbols:Check_Valve")
 		(lib_id "PID_symbols:Check_Valve")
 		(at 140.97 69.85 0)
@@
 		(on_board yes)
 		(dnp no)
-		(property "Reference" "Check_Valve11"
+		(property "Reference" "Check_Valve9"
 			(at 143.51 73.914 0)
 			(effects
@@
 			(project "P_IDs"
 				(path "/045f1f05-3134-4b6d-91b6-463031104f1e/12264f82-10ad-4f8b-aee0-7883d457c15c"
-					(reference "Check_Valve11")
+					(reference "Check_Valve9")
 					(unit 1)
 				)
@@
 		(pin ""
 		)
+		(pin ""
+		)
 		(instances
 			(project "P_IDs"
@@
 		(pin ""
 		)
+		(pin ""
+		)
 		(instances
 			(project "P_IDs"
@@
 	)
 	(symbol
+		(lib_name "PID_symbols:Pressure_Transducer")
 		(lib_id "PID_symbols:Pressure_Transducer")
 		(at 114.3 114.3 0)
@@
 				(hide yes)
 			)
+		)
+		(pin ""
 		)
 		(pin ""
@@
 	)
 	(symbol
+		(lib_name "PID_symbols:Pressure_Transducer")
 		(lib_id "PID_symbols:Pressure_Transducer")
 		(at 132.08 143.51 0)
@@
 		(pin ""
 		)
+		(pin ""
+		)
 		(instances
 			(project "P_IDs"
@@
 	)
 	(symbol
+		(lib_name "PID_symbols:Ball_Valve")
 		(lib_id "PID_symbols:Ball_Valve")
 		(at 130.81 59.69 270)
@@
 	)
 	(symbol
+		(lib_name "PID_symbols:Pressure_Transducer")
 		(lib_id "PID_symbols:Pressure_Transducer")
 		(at 175.26 80.01 0)
@@
 		(pin ""
 		)
+		(pin ""
+		)
 		(instances
 			(project "P_IDs"
@@
 	)
 	(symbol
+		(lib_name "PID_symbols:Pressure_Transducer")
 		(lib_id "PID_symbols:Pressure_Transducer")
 		(at 140.97 45.72 0)
@@
 		(pin ""
 		)
+		(pin ""
+		)
 		(instances
 			(project "P_IDs"
@@
 	)
 	(symbol
+		(lib_name "PID_symbols:Tank")
 		(lib_id "PID_symbols:Tank")
 		(at 129.54 27.94 0)
@@
 	)
 	(symbol
+		(lib_name "PID_symbols:Ball_Valve")
 		(lib_id "PID_symbols:Ball_Valve")
 		(at 113.03 83.82 0)
@@
 	)
 	(symbol
+		(lib_name "PID_symbols:Check_Valve")
 		(lib_id "PID_symbols:Check_Valve")
 		(at 110.49 72.39 270)
@@
 		(on_board yes)
 		(dnp no)
-		(property "Reference" "Check_Valve10"
+		(property "Reference" "Check_Valve8"
 			(at 112.776 74.93 90)
 			(effects
@@
 			(project "P_IDs"
 				(path "/045f1f05-3134-4b6d-91b6-463031104f1e/12264f82-10ad-4f8b-aee0-7883d457c15c"
-					(reference "Check_Valve10")
-					(unit 1)
-				)
-			)
-		)
-	)
-	(symbol
+					(reference "Check_Valve8")
+					(unit 1)
+				)
+			)
+		)
+	)
+	(symbol
+		(lib_name "PID_symbols:Tank")
 		(lib_id "PID_symbols:Tank")
 		(at 48.26 64.77 0)
@@
 	)
 	(symbol
+		(lib_name "PID_symbols:Solenoid")
 		(lib_id "PID_symbols:Solenoid")
 		(at 100.33 83.82 0)
@@
 	)
 	(symbol
+		(lib_name "PID_symbols:Tank")
 		(lib_id "PID_symbols:Tank")
 		(at 166.37 54.61 0)
@@
 	)
 	(symbol
+		(lib_name "PID_symbols:Ball_Valve")
 		(lib_id "PID_symbols:Ball_Valve")
 		(at 149.86 128.27 270)
