File: Hopper_Hotfire_TestStand.kicad_sch (KiCad schematic)
At the start: 28 parts

Commit message: no message
Parts:
- renumbered Nitrous_Fill1 to BV1, Ox_Vent1 to BV1, Nitrogen_Fill1 to BV1, Nitrous_Vent1 to BV1, Fuel_Main1 to BV1, Ball_Valve4 to BV4, Check_Valve7 to CV7, Check_Valve8 to CV8, Check_Valve9 to CV9, Warm_Fuel_Injector_PT1 to PT1, Fuel_Injector_PT1 to PT1, Chamber_PT1 to PT1, Nitrous_PT1 to PT1, Ox_Injector_PT1 to PT1, Fuel_PT1 to PT1, Nitrogen_PT1 to PT1, Flow_Sensor1 to Pmatic_B_Valve1, Pressure_Regulator1 to Reg1, Thomas1 to T1, TNitrou_Cylinder1 to T1, Fuel_Tank2 to T2, N2CYL1 to T?, Solenoid8 to nO_Sol8, Solenoid9 to nO_Sol9
Connections:
- net at CV7.: now also BV1., PT1., T1.; no longer BV1.
- net at BV4.: now also CV9., nO_Sol9.
- net at PT1.: now also BV1., Engine2.
- net at Pmatic_B_Valve1.: now also BV1.
- net at PT1.: now also Reg1., T?.
- new net: BV1., CV7.
- new net: BV1., Engine2., PT1.
- new net: BV1., Burst_Disc3., CV8., CV9., SPRV3.
- new net: Needle_Valve1., PT1., Pmatic_B_Valve1., T2.
- now unconnected: Burst_Disc3., Engine2., Engine2., PT1., PT1., PT1., SPRV3., T2., T?., nO_Sol9.
Changed lines of the file:
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@@
 		(on_board yes)
 		(dnp no)
-		(property "Reference" "Warm_Fuel_Injector_PT1"
+		(property "Reference" "PT1"
 			(at 143.51 121.666 90)
 			(effects
@@
 			(project "P_IDs"
 				(path "/045f1f05-3134-4b6d-91b6-463031104f1e/12264f82-10ad-4f8b-aee0-7883d457c15c"
-					(reference "Warm_Fuel_Injector_PT1")
+					(reference "PT1")
 					(unit 1)
 				)
@@
 		(on_board yes)
 		(dnp no)
-		(property "Reference" "Check_Valve7"
+		(property "Reference" "CV7"
 			(at 100.584 111.506 0)
 			(effects
@@
 			(project "P_IDs"
 				(path "/045f1f05-3134-4b6d-91b6-463031104f1e/12264f82-10ad-4f8b-aee0-7883d457c15c"
-					(reference "Check_Valve7")
+					(reference "CV7")
 					(unit 1)
 				)
@@
 		(dnp no)
 		(fields_autoplaced yes)
-		(property "Reference" "Nitrous_Fill1"
+		(property "Reference" "BV1"
 			(at 53.34 73.0249 90)
 			(effects
@@
 			(project "P_IDs"
 				(path "/045f1f05-3134-4b6d-91b6-463031104f1e/12264f82-10ad-4f8b-aee0-7883d457c15c"
-					(reference "Nitrous_Fill1")
+					(reference "BV1")
 					(unit 1)
 				)
@@
 		(on_board yes)
 		(dnp no)
-		(property "Reference" "Ball_Valve4"
+		(property "Reference" "BV4"
 			(at 154.94 90.17 0)
 			(effects
@@
 			(project "P_IDs"
 				(path "/045f1f05-3134-4b6d-91b6-463031104f1e/12264f82-10ad-4f8b-aee0-7883d457c15c"
-					(reference "Ball_Valve4")
+					(reference "BV4")
 					(unit 1)
 				)
@@
 		(on_board yes)
 		(dnp no)
-		(property "Reference" "Ox_Vent1"
+		(property "Reference" "BV1"
 			(at 123.698 132.08 90)
 			(effects
@@
 			(project "P_IDs"
 				(path "/045f1f05-3134-4b6d-91b6-463031104f1e/12264f82-10ad-4f8b-aee0-7883d457c15c"
-					(reference "Ox_Vent1")
+					(reference "BV1")
 					(unit 1)
 				)
@@
 		(on_board yes)
 		(dnp no)
-		(property "Reference" "Fuel_Injector_PT1"
+		(property "Reference" "PT1"
 			(at 165.354 140.97 0)
 			(effects
@@
 			(project "P_IDs"
 				(path "/045f1f05-3134-4b6d-91b6-463031104f1e/12264f82-10ad-4f8b-aee0-7883d457c15c"
-					(reference "Fuel_Injector_PT1")
+					(reference "PT1")
 					(unit 1)
 				)
@@
 		(on_board yes)
 		(dnp no)
-		(property "Reference" "Check_Valve9"
+		(property "Reference" "CV9"
 			(at 143.51 73.914 0)
 			(effects
@@
 			(project "P_IDs"
 				(path "/045f1f05-3134-4b6d-91b6-463031104f1e/12264f82-10ad-4f8b-aee0-7883d457c15c"
-					(reference "Check_Valve9")
+					(reference "CV9")
 					(unit 1)
 				)
@@
 		(on_board yes)
 		(dnp no)
-		(property "Reference" "Chamber_PT1"
+		(property "Reference" "PT1"
 			(at 122.682 149.86 0)
 			(effects
@@
 			(project "P_IDs"
 				(path "/045f1f05-3134-4b6d-91b6-463031104f1e/12264f82-10ad-4f8b-aee0-7883d457c15c"
-					(reference "Chamber_PT1")
+					(reference "PT1")
 					(unit 1)
 				)
@@
 		(on_board yes)
 		(dnp no)
-		(property "Reference" "Solenoid9"
+		(property "Reference" "nO_Sol9"
 			(at 154.94 71.882 0)
 			(effects
@@
 			(project "P_IDs"
 				(path "/045f1f05-3134-4b6d-91b6-463031104f1e/12264f82-10ad-4f8b-aee0-7883d457c15c"
-					(reference "Solenoid9")
+					(reference "nO_Sol9")
 					(unit 1)
 				)
@@
 		(on_board yes)
 		(dnp no)
-		(property "Reference" "Nitrous_PT1"
+		(property "Reference" "PT1"
 			(at 114.3 118.872 0)
 			(effects
@@
 			(project "P_IDs"
 				(path "/045f1f05-3134-4b6d-91b6-463031104f1e/12264f82-10ad-4f8b-aee0-7883d457c15c"
-					(reference "Nitrous_PT1")
+					(reference "PT1")
 					(unit 1)
 				)
@@
 		(on_board yes)
 		(dnp no)
-		(property "Reference" "Ox_Injector_PT1"
+		(property "Reference" "PT1"
 			(at 122.682 143.51 0)
 			(effects
@@
 			(project "P_IDs"
 				(path "/045f1f05-3134-4b6d-91b6-463031104f1e/12264f82-10ad-4f8b-aee0-7883d457c15c"
-					(reference "Ox_Injector_PT1")
+					(reference "PT1")
 					(unit 1)
 				)
@@
 		(on_board yes)
 		(dnp no)
-		(property "Reference" "Thomas1"
+		(property "Reference" "T1"
 			(at 106.68 93.98 0)
 			(effects
@@
 			(project "P_IDs"
 				(path "/045f1f05-3134-4b6d-91b6-463031104f1e/12264f82-10ad-4f8b-aee0-7883d457c15c"
-					(reference "Thomas1")
+					(reference "T1")
 					(unit 1)
 				)
@@
 		(dnp no)
 		(fields_autoplaced yes)
-		(property "Reference" "Nitrogen_Fill1"
+		(property "Reference" "BV1"
 			(at 134.62 62.8649 90)
 			(effects
@@
 			(project "P_IDs"
 				(path "/045f1f05-3134-4b6d-91b6-463031104f1e/12264f82-10ad-4f8b-aee0-7883d457c15c"
-					(reference "Nitrogen_Fill1")
+					(reference "BV1")
 					(unit 1)
 				)
@@
 		(dnp no)
 		(fields_autoplaced yes)
-		(property "Reference" "Flow_Sensor1"
+		(property "Reference" "Pmatic_B_Valve1"
 			(at 175.26 88.2649 90)
 			(effects
@@
 			(project ""
 				(path "/045f1f05-3134-4b6d-91b6-463031104f1e/12264f82-10ad-4f8b-aee0-7883d457c15c"
-					(reference "Flow_Sensor1")
+					(reference "Pmatic_B_Valve1")
 					(unit 1)
 				)
@@
 		(dnp no)
 		(fields_autoplaced yes)
-		(property "Reference" "Fuel_PT1"
+		(property "Reference" "PT1"
 			(at 175.26 74.93 0)
 			(effects
@@
 			(project "P_IDs"
 				(path "/045f1f05-3134-4b6d-91b6-463031104f1e/12264f82-10ad-4f8b-aee0-7883d457c15c"
-					(reference "Fuel_PT1")
+					(reference "PT1")
 					(unit 1)
 				)
@@
 		(dnp no)
 		(fields_autoplaced yes)
-		(property "Reference" "Nitrogen_PT1"
+		(property "Reference" "PT1"
 			(at 140.97 40.64 0)
 			(effects
@@
 			(project "P_IDs"
 				(path "/045f1f05-3134-4b6d-91b6-463031104f1e/12264f82-10ad-4f8b-aee0-7883d457c15c"
-					(reference "Nitrogen_PT1")
+					(reference "PT1")
 					(unit 1)
 				)
@@
 		(dnp no)
 		(fields_autoplaced yes)
-		(property "Reference" "Pressure_Regulator1"
+		(property "Reference" "Reg1"
 			(at 134.62 52.6424 90)
 			(effects
@@
 			(project "P_IDs"
 				(path "/045f1f05-3134-4b6d-91b6-463031104f1e/12264f82-10ad-4f8b-aee0-7883d457c15c"
-					(reference "Pressure_Regulator1")
+					(reference "Reg1")
 					(unit 1)
 				)
@@
 		(dnp no)
 		(fields_autoplaced yes)
-		(property "Reference" "N2CYL1"
+		(property "Reference" "T?"
 			(at 135.89 22.8599 0)
 			(effects
@@
 			(project "P_IDs"
 				(path "/045f1f05-3134-4b6d-91b6-463031104f1e/12264f82-10ad-4f8b-aee0-7883d457c15c"
-					(reference "N2CYL1")
+					(reference "T?")
 					(unit 1)
 				)
@@
 		(on_board yes)
 		(dnp no)
-		(property "Reference" "Nitrous_Vent1"
+		(property "Reference" "BV1"
 			(at 129.54 83.566 0)
 			(effects
@@
 			(project "P_IDs"
 				(path "/045f1f05-3134-4b6d-91b6-463031104f1e/12264f82-10ad-4f8b-aee0-7883d457c15c"
-					(reference "Nitrous_Vent1")
+					(reference "BV1")
 					(unit 1)
 				)
@@
 		(on_board yes)
 		(dnp no)
-		(property "Reference" "Check_Valve8"
+		(property "Reference" "CV8"
 			(at 112.776 74.93 90)
 			(effects
@@
 			(project "P_IDs"
 				(path "/045f1f05-3134-4b6d-91b6-463031104f1e/12264f82-10ad-4f8b-aee0-7883d457c15c"
-					(reference "Check_Valve8")
+					(reference "CV8")
 					(unit 1)
 				)
@@
 		(dnp no)
 		(fields_autoplaced yes)
-		(property "Reference" "TNitrou_Cylinder1"
+		(property "Reference" "T1"
 			(at 54.61 59.6899 0)
 			(effects
@@
 			(project "P_IDs"
 				(path "/045f1f05-3134-4b6d-91b6-463031104f1e/12264f82-10ad-4f8b-aee0-7883d457c15c"
-					(reference "TNitrou_Cylinder1")
+					(reference "T1")
 					(unit 1)
 				)
@@
 		(on_board yes)
 		(dnp no)
-		(property "Reference" "Solenoid8"
+		(property "Reference" "nO_Sol8"
 			(at 89.408 83.82 0)
 			(effects
@@
 			(project "P_IDs"
 				(path "/045f1f05-3134-4b6d-91b6-463031104f1e/12264f82-10ad-4f8b-aee0-7883d457c15c"
-					(reference "Solenoid8")
+					(reference "nO_Sol8")
 					(unit 1)
 				)
@@
 		(dnp no)
 		(fields_autoplaced yes)
-		(property "Reference" "Fuel_Tank2"
+		(property "Reference" "T2"
 			(at 172.72 49.5299 0)
 			(effects
@@
 			(project "P_IDs"
 				(path "/045f1f05-3134-4b6d-91b6-463031104f1e/12264f82-10ad-4f8b-aee0-7883d457c15c"
-					(reference "Fuel_Tank2")
+					(reference "T2")
 					(unit 1)
 				)
@@
 		(on_board yes)
 		(dnp no)
-		(property "Reference" "Fuel_Main1"
+		(property "Reference" "BV1"
 			(at 163.322 132.08 90)
 			(effects
@@
 			(project "P_IDs"
 				(path "/045f1f05-3134-4b6d-91b6-463031104f1e/12264f82-10ad-4f8b-aee0-7883d457c15c"
-					(reference "Fuel_Main1")
-					(unit 1)
-				)
+					(reference "BV1")
+					(unit 1)
+				)

Commit message: no message
Connections:
- net at CV7.: now also BV1., PT1., T1.; no longer BV1.
- net at BV4.: now also CV9., nO_Sol9.
- net at PT1.: now also BV1., Engine2.
- net at Pmatic_B_Valve1.: now also BV1.
- net at PT1.: now also Reg1., T?.
- new net: BV1., CV7.
- new net: BV1., Engine2., PT1.
- new net: BV1., Burst_Disc3., CV8., CV9., SPRV3.
- new net: Needle_Valve1., PT1., Pmatic_B_Valve1., T2.
- now unconnected: Burst_Disc3., Engine2., Engine2., PT1., PT1., PT1., SPRV3., T2., T?., nO_Sol9.
Changed lines of the file:
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@@
 	)
 	(symbol
+		(lib_name "PID_symbols:Check_Valve")
 		(lib_id "PID_symbols:Check_Valve")
 		(at 99.06 104.14 0)
@@
 	)
 	(symbol
+		(lib_name "PID_symbols:Ball_Valve")
 		(lib_id "PID_symbols:Ball_Valve")
 		(at 137.16 135.89 90)
@@
 	)
 	(symbol
+		(lib_name "PID_symbols:Pressure_Transducer")
 		(lib_id "PID_symbols:Pressure_Transducer")
 		(at 132.08 149.86 0)
@@
 	)
 	(symbol
+		(lib_name "PID_symbols:Tank")
 		(lib_id "PID_symbols:Tank")
 		(at 109.22 99.06 0)
@@
 	)
 	(symbol
-		(lib_name "PID_symbols:Ball_Valve")
 		(lib_id "PID_symbols:Ball_Valve")
 		(at 130.81 59.69 270)
@@
 	)
 	(symbol
-		(lib_name "PID_symbols:Pressure_Transducer")
 		(lib_id "PID_symbols:Pressure_Transducer")
 		(at 175.26 80.01 0)
@@
 	)
 	(symbol
-		(lib_name "PID_symbols:Check_Valve")
 		(lib_id "PID_symbols:Check_Valve")
 		(at 110.49 72.39 270)
@@
 	)
 	(symbol
-		(lib_name "PID_symbols:Tank")
 		(lib_id "PID_symbols:Tank")
 		(at 48.26 64.77 0)
@@
 	)
 	(symbol
-		(lib_name "PID_symbols:Solenoid")
 		(lib_id "PID_symbols:Solenoid")
 		(at 100.33 83.82 0)
