File: IgniterTest.kicad_sch (KiCad schematic)
At the start: 16 parts

Commit message: ho tin leung
Connections:
- net at Fuel_Main_Servo1.: now also Check_Valve6.; no longer Fuel_Tank1.
- net at N2_Line_Vent_Manual1.: now also Fuel_Press1., N2_Reg1.
- net at N2_Bottle1.: now also N2_Reg1.
- net at N2O_Bottle1.: now also Ox_Main_Servo1.
- net at Ox_Main_Servo1.: now also Check_Valve5.; no longer N2O_Bottle1.
- new net: Check_Valve6., Fuel_Inj_Pressure1., Torch_Ignitor1.
- new net: Check_Valve5., Ox_Inj_Pressure1., Torch_Ignitor1.
- new net: Fuel_Main_Servo1., Fuel_Tank1.
- now unconnected: Fuel_Inj_Pressure1., Ox_Inj_Pressure1.
Changed lines of the file:
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@@
+				)
+			)
+			(project "IgniterTest"
+				(path "/1fe58bd7-d6db-4cdb-9816-3cf1e5c4b0ec"
+					(reference "Torch_Ignitor")
+					(unit 1)
 				)
 			)
@@
 		(dnp no)
 		(property "Reference" "Chamber_Pressure1"
-			(at 151.384 157.226 0)
+			(at 152.146 157.48 0)
 			(effects
 				(font
@@
 				(path "/045f1f05-3134-4b6d-91b6-463031104f1e/6a55bbd5-ed21-4b79-a194-d378f68dea1b"
 					(reference "Chamber_Pressure1")
+					(unit 1)
+				)
+			)
+			(project "IgniterTest"
+				(path "/1fe58bd7-d6db-4cdb-9816-3cf1e5c4b0ec"
+					(reference "Chamber_Pressure")
 					(unit 1)
 				)
@@
 				)
 			)
+			(project "IgniterTest"
+				(path "/1fe58bd7-d6db-4cdb-9816-3cf1e5c4b0ec"
+					(reference "Fuel_Main_Servo")
+					(unit 1)
+				)
+			)
 		)
 	)
@@
 				(path "/045f1f05-3134-4b6d-91b6-463031104f1e/6a55bbd5-ed21-4b79-a194-d378f68dea1b"
 					(reference "N2_Line_Vent_Manual1")
+					(unit 1)
+				)
+			)
+			(project "IgniterTest"
+				(path "/1fe58bd7-d6db-4cdb-9816-3cf1e5c4b0ec"
+					(reference "N2_Line_Vent_Manual")
 					(unit 1)
 				)
@@
 				)
 			)
+			(project "IgniterTest"
+				(path "/1fe58bd7-d6db-4cdb-9816-3cf1e5c4b0ec"
+					(reference "N2_Bottle")
+					(unit 1)
+				)
+			)
 		)
 	)
@@
 				)
 			)
+			(project "IgniterTest"
+				(path "/1fe58bd7-d6db-4cdb-9816-3cf1e5c4b0ec"
+					(reference "Fuel_Tank")
+					(unit 1)
+				)
+			)
 		)
 	)
@@
 		(dnp no)
 		(property "Reference" "Fuel_Inj_Pressure1"
-			(at 151.384 149.606 0)
+			(at 151.638 149.86 0)
 			(effects
 				(font
@@
 				(path "/045f1f05-3134-4b6d-91b6-463031104f1e/6a55bbd5-ed21-4b79-a194-d378f68dea1b"
 					(reference "Fuel_Inj_Pressure1")
+					(unit 1)
+				)
+			)
+			(project "IgniterTest"
+				(path "/1fe58bd7-d6db-4cdb-9816-3cf1e5c4b0ec"
+					(reference "Fuel_Inj_Pressure")
 					(unit 1)
 				)
@@
 				)
 			)
+			(project "IgniterTest"
+				(path "/1fe58bd7-d6db-4cdb-9816-3cf1e5c4b0ec"
+					(reference "Ox_Inj_Pressure")
+					(unit 1)
+				)
+			)
 		)
 	)
@@
 				)
 			)
-		)
-	)
-	(symbol
-		(lib_name "PID_symbols:Check_Valve")
+			(project "IgniterTest"
+				(path "/1fe58bd7-d6db-4cdb-9816-3cf1e5c4b0ec"
+					(reference "N2O_Bottle")
+					(unit 1)
+				)
+			)
+		)
+	)
+	(symbol
 		(lib_id "PID_symbols:Check_Valve")
 		(at 116.84 134.62 270)
@@
 				)
 			)
-		)
-	)
-	(symbol
-		(lib_name "PID_symbols:Check_Valve")
+			(project "IgniterTest"
+				(path "/1fe58bd7-d6db-4cdb-9816-3cf1e5c4b0ec"
+					(reference "Check_Valve?")
+					(unit 1)
+				)
+			)
+		)
+	)
+	(symbol
 		(lib_id "PID_symbols:Check_Valve")
 		(at 134.62 134.62 270)
@@
 				)
 			)
+			(project "IgniterTest"
+				(path "/1fe58bd7-d6db-4cdb-9816-3cf1e5c4b0ec"
+					(reference "Check_Valve?")
+					(unit 1)
+				)
+			)
 		)
 	)
@@
 				)
 			)
+			(project "IgniterTest"
+				(path "/1fe58bd7-d6db-4cdb-9816-3cf1e5c4b0ec"
+					(reference "Fuel_Tank_Pressure")
+					(unit 1)
+				)
+			)
 		)
 	)
@@
 				)
 			)
+			(project "IgniterTest"
+				(path "/1fe58bd7-d6db-4cdb-9816-3cf1e5c4b0ec"
+					(reference "Fuel_Vent_Servo")
+					(unit 1)
+				)
+			)
 		)
 	)
@@
 				)
 			)
+			(project "IgniterTest"
+				(path "/1fe58bd7-d6db-4cdb-9816-3cf1e5c4b0ec"
+					(reference "Fuel_Press")
+					(unit 1)
+				)
+			)
 		)
 	)
@@
 				(path "/045f1f05-3134-4b6d-91b6-463031104f1e/6a55bbd5-ed21-4b79-a194-d378f68dea1b"
 					(reference "N2_Reg1")
+					(unit 1)
+				)
+			)
+			(project "IgniterTest"
+				(path "/1fe58bd7-d6db-4cdb-9816-3cf1e5c4b0ec"
+					(reference "N2_Reg")
 					(unit 1)
 				)
@@
 				)
 			)
-		)
-	)
+			(project "IgniterTest"
+				(path "/1fe58bd7-d6db-4cdb-9816-3cf1e5c4b0ec"
+					(reference "Ox_Main_Servo")
+					(unit 1)
+				)
+			)
+		)
+	)
+	(sheet_instances
+		(path "/"
+			(page "1")
+		)
+	)

Commit message: added answer key and gitignore
Connections:
- net at Fuel_Main_Servo1.: now also Check_Valve6.; no longer Fuel_Tank1.
- net at N2_Line_Vent_Manual1.: now also Fuel_Press1., N2_Reg1.
- net at N2_Bottle1.: now also N2_Reg1.
- net at N2O_Bottle1.: now also Ox_Main_Servo1.
- net at Ox_Main_Servo1.: now also Check_Valve5.; no longer N2O_Bottle1.
- new net: Check_Valve6., Fuel_Inj_Pressure1., Torch_Ignitor1.
- new net: Check_Valve5., Ox_Inj_Pressure1., Torch_Ignitor1.
- new net: Fuel_Main_Servo1., Fuel_Tank1.
- now unconnected: Fuel_Inj_Pressure1., Ox_Inj_Pressure1.
Changed lines of the file:
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@@
 	)
 	(symbol
-		(lib_name "PID_symbols:Pressure_Transducer")
 		(lib_id "PID_symbols:Pressure_Transducer")
 		(at 139.7 157.48 0)
@@
 	)
 	(symbol
-		(lib_name "PnID_symbols:Tank")
 		(lib_id "PnID_symbols:Tank")
 		(at 133.35 52.07 0)
@@
 	)
 	(symbol
-		(lib_name "PnID_symbols:Tank")
 		(lib_id "PnID_symbols:Tank")
 		(at 133.35 105.41 0)
@@
 	)
 	(symbol
-		(lib_name "PID_symbols:Pressure_Transducer")
 		(lib_id "PID_symbols:Pressure_Transducer")
 		(at 139.7 149.86 0)
@@
 	)
 	(symbol
-		(lib_name "PID_symbols:Pressure_Transducer")
 		(lib_id "PID_symbols:Pressure_Transducer")
 		(at 111.76 149.86 0)
@@
 	)
 	(symbol
-		(lib_name "PnID_symbols:Tank")
 		(lib_id "PnID_symbols:Tank")
 		(at 115.57 105.41 0)
@@
 	)
 	(symbol
-		(lib_name "PID_symbols:Pressure_Transducer")
 		(lib_id "PID_symbols:Pressure_Transducer")
 		(at 127 90.17 0)

Commit message: deleted answer keys
Parts:
- renumbered Check_Valve5 to Check_Valve1, Check_Valve6 to Check_Valve2
Connections:
- net at Fuel_Main_Servo1.: now also Check_Valve2.; no longer Fuel_Tank1.
- net at N2_Line_Vent_Manual1.: now also Fuel_Press1., N2_Reg1.
- net at N2_Bottle1.: now also N2_Reg1.
- net at N2O_Bottle1.: now also Ox_Main_Servo1.
- net at Ox_Main_Servo1.: now also Check_Valve1.; no longer N2O_Bottle1.
- new net: Check_Valve2., Fuel_Inj_Pressure1., Torch_Ignitor1.
- new net: Check_Valve1., Ox_Inj_Pressure1., Torch_Ignitor1.
- new net: Fuel_Main_Servo1., Fuel_Tank1.
- now unconnected: Fuel_Inj_Pressure1., Ox_Inj_Pressure1.
Changed lines of the file:
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@@
 		(dnp no)
 		(fields_autoplaced yes)
-		(property "Reference" "Check_Valve5"
+		(property "Reference" "Check_Valve1"
 			(at 120.65 136.3979 90)
 			(effects
@@
 			(project "P_IDs"
 				(path "/045f1f05-3134-4b6d-91b6-463031104f1e/6a55bbd5-ed21-4b79-a194-d378f68dea1b"
-					(reference "Check_Valve5")
+					(reference "Check_Valve1")
 					(unit 1)
 				)
@@
 		(dnp no)
 		(fields_autoplaced yes)
-		(property "Reference" "Check_Valve6"
+		(property "Reference" "Check_Valve2"
 			(at 138.43 136.3979 90)
 			(effects
@@
 			(project "P_IDs"
 				(path "/045f1f05-3134-4b6d-91b6-463031104f1e/6a55bbd5-ed21-4b79-a194-d378f68dea1b"
-					(reference "Check_Valve6")
+					(reference "Check_Valve2")
 					(unit 1)
 				)

Commit message: no message
Connections:
- net at Fuel_Main_Servo1.: now also Check_Valve2.; no longer Fuel_Tank1.
- net at N2_Line_Vent_Manual1.: now also Fuel_Press1., N2_Reg1.
- net at N2_Bottle1.: now also N2_Reg1.
- net at N2O_Bottle1.: now also Ox_Main_Servo1.
- net at Ox_Main_Servo1.: now also Check_Valve1.; no longer N2O_Bottle1.
- new net: Check_Valve2., Fuel_Inj_Pressure1., Torch_Ignitor1.
- new net: Check_Valve1., Ox_Inj_Pressure1., Torch_Ignitor1.
- new net: Fuel_Main_Servo1., Fuel_Tank1.
- now unconnected: Fuel_Inj_Pressure1., Ox_Inj_Pressure1.
Changed lines of the file:
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@@
 	)
 	(symbol
+		(lib_name "PID_symbols:Pressure_Transducer")
 		(lib_id "PID_symbols:Pressure_Transducer")
 		(at 139.7 157.48 0)
@@
 				(hide yes)
 			)
+		)
+		(pin ""
 		)
 		(pin ""
@@
 	)
 	(symbol
+		(lib_name "PID_symbols:Pressure_Transducer")
 		(lib_id "PID_symbols:Pressure_Transducer")
 		(at 139.7 149.86 0)
@@
 		(pin ""
 		)
+		(pin ""
+		)
 		(instances
 			(project "P_IDs"
@@
 				(hide yes)
 			)
+		)
+		(pin ""
 		)
 		(pin ""
@@
 	)
 	(symbol
+		(lib_name "PID_symbols:Check_Valve")
 		(lib_id "PID_symbols:Check_Valve")
 		(at 134.62 134.62 270)
@@
 	)
 	(symbol
+		(lib_name "PID_symbols:Pressure_Transducer")
 		(lib_id "PID_symbols:Pressure_Transducer")
 		(at 127 90.17 0)
@@
 		)
 		(pin ""
+		)
+		(pin ""

Commit message: no message
Parts:
- renumbered Fuel_Vent_Servo1 to BV1, Check_Valve1 to CV1, Check_Valve2 to CV2, N2_Line_Vent_Manual1 to Needle_Valve?, Chamber_Pressure1 to PT1, Fuel_Inj_Pressure1 to PT1, Ox_Inj_Pressure1 to PT1, Fuel_Tank_Pressure1 to PT1
Connections:
- net at Fuel_Main_Servo1.: now also CV2.; no longer Fuel_Tank1.
- net at Needle_Valve?.: now also Fuel_Press1., N2_Reg1.
- net at N2_Bottle1.: now also N2_Reg1.
- net at N2O_Bottle1.: now also Ox_Main_Servo1.
- net at Ox_Main_Servo1.: now also CV1.; no longer N2O_Bottle1.
- new net: CV2., PT1., Torch_Ignitor1.
- new net: CV1., PT1., Torch_Ignitor1.
- new net: Fuel_Main_Servo1., Fuel_Tank1.
- now unconnected: PT1., PT1.
Changed lines of the file:
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@@
 		(on_board yes)
 		(dnp no)
-		(property "Reference" "Chamber_Pressure1"
+		(property "Reference" "PT1"
 			(at 152.146 157.48 0)
 			(effects
@@
 			(project "P_IDs"
 				(path "/045f1f05-3134-4b6d-91b6-463031104f1e/6a55bbd5-ed21-4b79-a194-d378f68dea1b"
-					(reference "Chamber_Pressure1")
+					(reference "PT1")
 					(unit 1)
 				)
@@
 		(on_board yes)
 		(dnp no)
-		(property "Reference" "N2_Line_Vent_Manual1"
+		(property "Reference" "Needle_Valve?"
 			(at 154.94 65.786 0)
 			(effects
@@
 			(project "P_IDs"
 				(path "/045f1f05-3134-4b6d-91b6-463031104f1e/6a55bbd5-ed21-4b79-a194-d378f68dea1b"
-					(reference "N2_Line_Vent_Manual1")
+					(reference "Needle_Valve?")
 					(unit 1)
 				)
@@
 		(on_board yes)
 		(dnp no)
-		(property "Reference" "Fuel_Inj_Pressure1"
+		(property "Reference" "PT1"
 			(at 151.638 149.86 0)
 			(effects
@@
 			(project "P_IDs"
 				(path "/045f1f05-3134-4b6d-91b6-463031104f1e/6a55bbd5-ed21-4b79-a194-d378f68dea1b"
-					(reference "Fuel_Inj_Pressure1")
+					(reference "PT1")
 					(unit 1)
 				)
@@
 		(on_board yes)
 		(dnp no)
-		(property "Reference" "Ox_Inj_Pressure1"
+		(property "Reference" "PT1"
 			(at 100.838 149.606 0)
 			(effects
@@
 			(project "P_IDs"
 				(path "/045f1f05-3134-4b6d-91b6-463031104f1e/6a55bbd5-ed21-4b79-a194-d378f68dea1b"
-					(reference "Ox_Inj_Pressure1")
+					(reference "PT1")
 					(unit 1)
 				)
@@
 		(dnp no)
 		(fields_autoplaced yes)
-		(property "Reference" "Check_Valve1"
+		(property "Reference" "CV1"
 			(at 120.65 136.3979 90)
 			(effects
@@
 			(project "P_IDs"
 				(path "/045f1f05-3134-4b6d-91b6-463031104f1e/6a55bbd5-ed21-4b79-a194-d378f68dea1b"
-					(reference "Check_Valve1")
+					(reference "CV1")
 					(unit 1)
 				)
@@
 		(dnp no)
 		(fields_autoplaced yes)
-		(property "Reference" "Check_Valve2"
+		(property "Reference" "CV2"
 			(at 138.43 136.3979 90)
 			(effects
@@
 			(project "P_IDs"
 				(path "/045f1f05-3134-4b6d-91b6-463031104f1e/6a55bbd5-ed21-4b79-a194-d378f68dea1b"
-					(reference "Check_Valve2")
+					(reference "CV2")
 					(unit 1)
 				)
@@
 		(on_board yes)
 		(dnp no)
-		(property "Reference" "Fuel_Tank_Pressure1"
+		(property "Reference" "PT1"
 			(at 113.538 89.916 0)
 			(effects
@@
 			(project "P_IDs"
 				(path "/045f1f05-3134-4b6d-91b6-463031104f1e/6a55bbd5-ed21-4b79-a194-d378f68dea1b"
-					(reference "Fuel_Tank_Pressure1")
+					(reference "PT1")
 					(unit 1)
 				)
@@
 		(on_board yes)
 		(dnp no)
-		(property "Reference" "Fuel_Vent_Servo1"
+		(property "Reference" "BV1"
 			(at 154.94 85.852 0)
 			(effects
@@
 			(project "P_IDs"
 				(path "/045f1f05-3134-4b6d-91b6-463031104f1e/6a55bbd5-ed21-4b79-a194-d378f68dea1b"
-					(reference "Fuel_Vent_Servo1")
-					(unit 1)
-				)
+					(reference "BV1")
+					(unit 1)
+				)

Commit message: no message
Connections:
- net at Fuel_Main_Servo1.: now also CV2.; no longer Fuel_Tank1.
- net at Needle_Valve?.: now also Fuel_Press1., N2_Reg1.
- net at N2_Bottle1.: now also N2_Reg1.
- net at N2O_Bottle1.: now also Ox_Main_Servo1.
- net at Ox_Main_Servo1.: now also CV1.; no longer N2O_Bottle1.
- new net: CV2., PT1., Torch_Ignitor1.
- new net: CV1., PT1., Torch_Ignitor1.
- new net: Fuel_Main_Servo1., Fuel_Tank1.
- now unconnected: PT1., PT1.
Changed lines of the file:
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@@
 	)
 	(symbol
-		(lib_name "PID_symbols:Pressure_Transducer")
 		(lib_id "PID_symbols:Pressure_Transducer")
 		(at 139.7 157.48 0)
@@
 	)
 	(symbol
+		(lib_name "PID_symbols:Pressure_Transducer")
 		(lib_id "PID_symbols:Pressure_Transducer")
 		(at 111.76 149.86 0)

Commit message: update
Parts:
- gave numbers to parts that had none: 1
- renumbered PT1 to PT2, PT1 to PT3, PT1 to PT4
Connections:
- net at Fuel_Main_Servo1.: now also CV2.; no longer Fuel_Tank1.
- net at Needle_Valve1.: now also Fuel_Press1., N2_Reg1.
- net at N2_Bottle1.: now also N2_Reg1.
- net at N2O_Bottle1.: now also Ox_Main_Servo1.
- net at Ox_Main_Servo1.: now also CV1.; no longer N2O_Bottle1.
- new net: CV2., PT3., Torch_Ignitor1.
- new net: CV1., PT1., Torch_Ignitor1.
- new net: Fuel_Main_Servo1., Fuel_Tank1.
- now unconnected: PT1., PT3.
Changed lines of the file:
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@@
 		(on_board yes)
 		(dnp no)
-		(property "Reference" "PT1"
+		(property "Reference" "PT4"
 			(at 152.146 157.48 0)
 			(effects
@@
 			(project "P_IDs"
 				(path "/045f1f05-3134-4b6d-91b6-463031104f1e/6a55bbd5-ed21-4b79-a194-d378f68dea1b"
-					(reference "PT1")
+					(reference "PT4")
 					(unit 1)
 				)
@@
 		(on_board yes)
 		(dnp no)
-		(property "Reference" "Needle_Valve?"
+		(property "Reference" "Needle_Valve1"
 			(at 154.94 65.786 0)
 			(effects
@@
 			(project "P_IDs"
 				(path "/045f1f05-3134-4b6d-91b6-463031104f1e/6a55bbd5-ed21-4b79-a194-d378f68dea1b"
-					(reference "Needle_Valve?")
+					(reference "Needle_Valve1")
 					(unit 1)
 				)
@@
 		(on_board yes)
 		(dnp no)
-		(property "Reference" "PT1"
+		(property "Reference" "PT3"
 			(at 151.638 149.86 0)
 			(effects
@@
 			(project "P_IDs"
 				(path "/045f1f05-3134-4b6d-91b6-463031104f1e/6a55bbd5-ed21-4b79-a194-d378f68dea1b"
-					(reference "PT1")
+					(reference "PT3")
 					(unit 1)
 				)
@@
 		(on_board yes)
 		(dnp no)
-		(property "Reference" "PT1"
+		(property "Reference" "PT2"
 			(at 113.538 89.916 0)
 			(effects
@@
 			(project "P_IDs"
 				(path "/045f1f05-3134-4b6d-91b6-463031104f1e/6a55bbd5-ed21-4b79-a194-d378f68dea1b"
-					(reference "PT1")
-					(unit 1)
-				)
+					(reference "PT2")
+					(unit 1)
+				)

Commit message: added L9 P&ID from Babs, he had problems using git
Parts:
- BV1, CV1, CV2, Needle_Valve1: value ~ -> (none)
- PT1, PT2, PT3, PT4: value 100 -> (none)
Connections:
- net at Fuel_Main_Servo1.: now also CV2.; no longer Fuel_Tank1.
- net at Needle_Valve1.: now also Fuel_Press1., N2_Reg1.
- net at N2_Bottle1.: now also N2_Reg1.
- net at N2O_Bottle1.: now also Ox_Main_Servo1.
- net at Ox_Main_Servo1.: now also CV1.; no longer N2O_Bottle1.
- new net: CV2., PT3., Torch_Ignitor1.
- new net: CV1., PT1., Torch_Ignitor1.
- new net: Fuel_Main_Servo1., Fuel_Tank1.
- now unconnected: PT1., PT3.
Changed lines of the file:
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@@
 		(dnp no)
 		(property "Reference" "PT4"
-			(at 152.146 157.48 0)
-			(effects
-				(font
-					(size 1.27 1.27)
-				)
-			)
-		)
-		(property "Value" "100"
-			(at 139.7 158.496 0)
-			(effects
-				(font
-					(size 1.27 1.27)
-				)
+			(at 139.7 161.29 0)
+			(effects
+				(font
+					(size 1.27 1.27)
+				)
+			)
+		)
+		(property "Value" ""
+			(at 139.7 158.75 0)
+			(effects
+				(font
+					(size 1.27 1.27)
+				)
+				(hide yes)
 			)
 		)
@@
 		(dnp no)
 		(property "Reference" "Needle_Valve1"
-			(at 154.94 65.786 0)
-			(effects
-				(font
-					(size 1.27 1.27)
-				)
-			)
-		)
-		(property "Value" "~"
-			(at 154.94 66.04 0)
+			(at 154.686 74.93 0)
+			(effects
+				(font
+					(size 1.27 1.27)
+				)
+			)
+		)
+		(property "Value" ""
+			(at 151.13 71.12 0)
 			(effects
 				(font
@@
 		(dnp no)
 		(property "Reference" "PT3"
-			(at 151.638 149.86 0)
-			(effects
-				(font
-					(size 1.27 1.27)
-				)
-			)
-		)
-		(property "Value" "100"
-			(at 139.7 150.876 0)
-			(effects
-				(font
-					(size 1.27 1.27)
-				)
+			(at 139.7 153.67 0)
+			(effects
+				(font
+					(size 1.27 1.27)
+				)
+			)
+		)
+		(property "Value" ""
+			(at 139.7 151.13 0)
+			(effects
+				(font
+					(size 1.27 1.27)
+				)
+				(hide yes)
 			)
 		)
@@
 		(dnp no)
 		(property "Reference" "PT1"
-			(at 100.838 149.606 0)
-			(effects
-				(font
-					(size 1.27 1.27)
-				)
-			)
-		)
-		(property "Value" "100"
-			(at 111.76 150.876 0)
-			(effects
-				(font
-					(size 1.27 1.27)
-				)
+			(at 111.76 153.67 0)
+			(effects
+				(font
+					(size 1.27 1.27)
+				)
+			)
+		)
+		(property "Value" ""
+			(at 111.76 151.13 0)
+			(effects
+				(font
+					(size 1.27 1.27)
+				)
+				(hide yes)
 			)
 		)
@@
 		(fields_autoplaced yes)
 		(property "Reference" "CV1"
-			(at 120.65 136.3979 90)
+			(at 120.65 137.0329 90)
 			(effects
 				(font
@@
 				)
 				(justify left)
-				(hide yes)
-			)
-		)
-		(property "Value" "~"
-			(at 120.65 138.303 90)
-			(effects
-				(font
-					(size 1.27 1.27)
-				)
-				(justify left)
+			)
+		)
+		(property "Value" ""
+			(at 116.84 134.62 0)
+			(effects
+				(font
+					(size 1.27 1.27)
+				)
 			)
 		)
@@
 		(fields_autoplaced yes)
 		(property "Reference" "CV2"
-			(at 138.43 136.3979 90)
+			(at 138.43 137.0329 90)
 			(effects
 				(font
@@
 				)
 				(justify left)
-				(hide yes)
-			)
-		)
-		(property "Value" "~"
-			(at 138.43 138.303 90)
-			(effects
-				(font
-					(size 1.27 1.27)
-				)
-				(justify left)
+			)
+		)
+		(property "Value" ""
+			(at 134.62 134.62 0)
+			(effects
+				(font
+					(size 1.27 1.27)
+				)
 			)
 		)
@@
 		(dnp no)
 		(property "Reference" "PT2"
-			(at 113.538 89.916 0)
-			(effects
-				(font
-					(size 1.27 1.27)
-				)
-			)
-		)
-		(property "Value" "100"
-			(at 127 91.186 0)
-			(effects
-				(font
-					(size 1.27 1.27)
-				)
+			(at 127 93.98 0)
+			(effects
+				(font
+					(size 1.27 1.27)
+				)
+			)
+		)
+		(property "Value" ""
+			(at 127 91.44 0)
+			(effects
+				(font
+					(size 1.27 1.27)
+				)
+				(hide yes)
 			)
 		)
@@
 		(dnp no)
 		(property "Reference" "BV1"
-			(at 154.94 85.852 0)
-			(effects
-				(font
-					(size 1.27 1.27)
-				)
-			)
-		)
-		(property "Value" "~"
-			(at 154.94 86.36 0)
-			(effects
-				(font
+			(at 154.94 94.488 0)
+			(effects
+				(font
+					(size 1.27 1.27)
+				)
+			)
+		)
+		(property "Value" ""
+			(at 151.13 90.17 0)
+			(effects
+				(font
