File: GroundFillingStation.kicad_sch (KiCad schematic)
At the start: 19 parts

Commit message: overwriting babz
Parts:
- renumbered BV28 to BV32, BV29 to BV33, BV_Nitrogen2 to BV_Nitrogen1, BV_Nitrous2 to BV_Nitrous1, CV30 to CV32, CV31 to CV33, H5 to H8, NitrogenBottle to NitrogenBottle1, NitrousCylinder to NitrousCylinder1, NitrousCylinder to NitrousCylinder2, PT55 to PT56, PT53 to PT57, PT54 to PT58, QD14 to QD19, QD15 to QD20
Connections:
- new net: BV33., CV33.
- new net: BV32., CV32.
Changed lines of the file:
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@@
 		(dnp no)
 		(fields_autoplaced yes)
-		(property "Reference" "BV_Nitrogen2"
+		(property "Reference" "BV_Nitrogen1"
 			(at 172.72 83.8199 90)
 			(effects
@@
 			(project "P_IDs"
 				(path "/045f1f05-3134-4b6d-91b6-463031104f1e/a942ff8e-b572-4ca0-bc2e-001c1a49fd10/8e320f35-5e7f-414e-91e4-92bfb9958dbc"
-					(reference "BV_Nitrogen2")
+					(reference "BV_Nitrogen1")
 					(unit 1)
 				)
@@
 		(dnp no)
 		(fields_autoplaced yes)
-		(property "Reference" "PT53"
+		(property "Reference" "PT57"
 			(at 81.28 129.54 0)
 			(effects
@@
 			(project "P_IDs"
 				(path "/045f1f05-3134-4b6d-91b6-463031104f1e/a942ff8e-b572-4ca0-bc2e-001c1a49fd10/8e320f35-5e7f-414e-91e4-92bfb9958dbc"
-					(reference "PT53")
+					(reference "PT57")
 					(unit 1)
 				)
@@
 		(dnp no)
 		(fields_autoplaced yes)
-		(property "Reference" "CV31"
+		(property "Reference" "CV33"
 			(at 127 127.7619 90)
 			(effects
@@
 			(project "P_IDs"
 				(path "/045f1f05-3134-4b6d-91b6-463031104f1e/a942ff8e-b572-4ca0-bc2e-001c1a49fd10/8e320f35-5e7f-414e-91e4-92bfb9958dbc"
-					(reference "CV31")
+					(reference "CV33")
 					(unit 1)
 				)
@@
 		(dnp no)
 		(fields_autoplaced yes)
-		(property "Reference" "PT55"
+		(property "Reference" "PT56"
 			(at 187.96 107.315 0)
 			(effects
@@
 			(project "P_IDs"
 				(path "/045f1f05-3134-4b6d-91b6-463031104f1e/a942ff8e-b572-4ca0-bc2e-001c1a49fd10/8e320f35-5e7f-414e-91e4-92bfb9958dbc"
-					(reference "PT55")
+					(reference "PT56")
 					(unit 1)
 				)
@@
 		(dnp no)
 		(fields_autoplaced yes)
-		(property "Reference" "QD15"
+		(property "Reference" "QD20"
 			(at 165.1 43.8149 90)
 			(effects
@@
 			(project "P_IDs"
 				(path "/045f1f05-3134-4b6d-91b6-463031104f1e/a942ff8e-b572-4ca0-bc2e-001c1a49fd10/8e320f35-5e7f-414e-91e4-92bfb9958dbc"
-					(reference "QD15")
+					(reference "QD20")
 					(unit 1)
 				)
@@
 		(on_board yes)
 		(dnp no)
-		(property "Reference" "BV29"
+		(property "Reference" "BV33"
 			(at 127 116.84 90)
 			(effects
@@
 			(project "P_IDs"
 				(path "/045f1f05-3134-4b6d-91b6-463031104f1e/a942ff8e-b572-4ca0-bc2e-001c1a49fd10/8e320f35-5e7f-414e-91e4-92bfb9958dbc"
-					(reference "BV29")
+					(reference "BV33")
 					(unit 1)
 				)
@@
 		(dnp no)
 		(fields_autoplaced yes)
-		(property "Reference" "QD14"
+		(property "Reference" "QD19"
 			(at 110.49 39.3699 90)
 			(effects
@@
 			(project "P_IDs"
 				(path "/045f1f05-3134-4b6d-91b6-463031104f1e/a942ff8e-b572-4ca0-bc2e-001c1a49fd10/8e320f35-5e7f-414e-91e4-92bfb9958dbc"
-					(reference "QD14")
+					(reference "QD19")
 					(unit 1)
 				)
@@
 		(dnp no)
 		(fields_autoplaced yes)
-		(property "Reference" "BV_Nitrous2"
+		(property "Reference" "BV_Nitrous1"
 			(at 118.11 79.3749 90)
 			(effects
@@
 			(project "P_IDs"
 				(path "/045f1f05-3134-4b6d-91b6-463031104f1e/a942ff8e-b572-4ca0-bc2e-001c1a49fd10/8e320f35-5e7f-414e-91e4-92bfb9958dbc"
-					(reference "BV_Nitrous2")
+					(reference "BV_Nitrous1")
 					(unit 1)
 				)
@@
 		(dnp no)
 		(fields_autoplaced yes)
-		(property "Reference" "H5"
+		(property "Reference" "H8"
 			(at 115.57 97.7899 0)
 			(effects
@@
 			(project "P_IDs"
 				(path "/045f1f05-3134-4b6d-91b6-463031104f1e/a942ff8e-b572-4ca0-bc2e-001c1a49fd10/8e320f35-5e7f-414e-91e4-92bfb9958dbc"
-					(reference "H5")
+					(reference "H8")
 					(unit 1)
 				)
@@
 		(dnp no)
 		(fields_autoplaced yes)
-		(property "Reference" "CV30"
+		(property "Reference" "CV32"
 			(at 107.95 127.7619 90)
 			(effects
@@
 			(project "P_IDs"
 				(path "/045f1f05-3134-4b6d-91b6-463031104f1e/a942ff8e-b572-4ca0-bc2e-001c1a49fd10/8e320f35-5e7f-414e-91e4-92bfb9958dbc"
-					(reference "CV30")
+					(reference "CV32")
 					(unit 1)
 				)
@@
 		(dnp no)
 		(fields_autoplaced yes)
-		(property "Reference" "NitrogenBottle"
+		(property "Reference" "NitrogenBottle1"
 			(at 173.99 121.2849 0)
 			(effects
@@
 			(project "P_IDs"
 				(path "/045f1f05-3134-4b6d-91b6-463031104f1e/a942ff8e-b572-4ca0-bc2e-001c1a49fd10/8e320f35-5e7f-414e-91e4-92bfb9958dbc"
-					(reference "NitrogenBottle")
+					(reference "NitrogenBottle1")
 					(unit 1)
 				)
@@
 		(dnp no)
 		(fields_autoplaced yes)
-		(property "Reference" "BV28"
+		(property "Reference" "BV32"
 			(at 107.95 116.2049 90)
 			(effects
@@
 			(project "P_IDs"
 				(path "/045f1f05-3134-4b6d-91b6-463031104f1e/a942ff8e-b572-4ca0-bc2e-001c1a49fd10/8e320f35-5e7f-414e-91e4-92bfb9958dbc"
-					(reference "BV28")
+					(reference "BV32")
 					(unit 1)
 				)
@@
 		(dnp no)
 		(fields_autoplaced yes)
-		(property "Reference" "NitrousCylinder"
+		(property "Reference" "NitrousCylinder2"
 			(at 128.27 143.5099 0)
 			(effects
@@
 			(project "P_IDs"
 				(path "/045f1f05-3134-4b6d-91b6-463031104f1e/a942ff8e-b572-4ca0-bc2e-001c1a49fd10/8e320f35-5e7f-414e-91e4-92bfb9958dbc"
-					(reference "NitrousCylinder")
+					(reference "NitrousCylinder2")
 					(unit 1)
 				)
@@
 		(on_board yes)
 		(dnp no)
-		(property "Reference" "NitrousCylinder"
+		(property "Reference" "NitrousCylinder1"
 			(at 85.09 143.51 0)
 			(effects
@@
 			(project "P_IDs"
 				(path "/045f1f05-3134-4b6d-91b6-463031104f1e/a942ff8e-b572-4ca0-bc2e-001c1a49fd10/8e320f35-5e7f-414e-91e4-92bfb9958dbc"
-					(reference "NitrousCylinder")
+					(reference "NitrousCylinder1")
 					(unit 1)
 				)
@@
 		(dnp no)
 		(fields_autoplaced yes)
-		(property "Reference" "PT54"
+		(property "Reference" "PT58"
 			(at 146.05 129.54 0)
 			(effects
@@
 			(project "P_IDs"
 				(path "/045f1f05-3134-4b6d-91b6-463031104f1e/a942ff8e-b572-4ca0-bc2e-001c1a49fd10/8e320f35-5e7f-414e-91e4-92bfb9958dbc"
-					(reference "PT54")
-					(unit 1)
-				)
+					(reference "PT58")
+					(unit 1)
+				)

Commit message: New year update
Parts:
- renumbered BV32 to BV78, BV33 to BV79, BV_Depressurise_Nitrogen2 to BV_Depressurise_Nitrogen4, BV_Depressurise_Nitrous2 to BV_Depressurise_Nitrous4, BV_Nitrogen1 to BV_Nitrogen2, BV_Nitrous1 to BV_Nitrous2, CV32 to CV77, CV33 to CV78, H8 to H16, Needle_Valve_Nitrogen2 to Needle_Valve_Nitrogen6, Needle_Valve_Nitrous2 to Needle_Valve_Nitrous4, NitrogenBottle1 to NitrogenBottle2, NitrousCylinder1 to NitrousCylinder3, NitrousCylinder2 to NitrousCylinder4, PT57 to PT139, PT58 to PT140, PT56 to PT141, QD19 to QD49, QD20 to QD50
Connections:
- new net: BV79., CV78.
- new net: BV78., CV77.
