File: Pluto.kicad_sch (KiCad schematic)
At the start: 46 parts

Commit message: overwriting babz
Parts:
- renumbered BV27 to BV31, Ball_Valve(ServoControlled)101 to Ball_Valve(ServoControlled)2, BurstDisc124 to BurstDisc2, Burst_Disc6 to Burst_Disc12, Burst_Disc11 to Burst_Disc13, Check_Valve6 to Check_Valve10, Check_Valve8 to Check_Valve6, Check_Valve113 to Check_Valve8, Engine8 to Engine10, Engine7 to Engine9, Needle_Valve5 to Needle_Valve7, Needle_Valve6 to Needle_Valve8, PT47 to PT48, PT52 to PT49, PT8 to PT51, PT28 to PT52, PT49 to PT53, PT48 to PT54, PT51 to PT55, Pressure_Regulator124 to Pressure_Regulator2, QD10 to QD16, QD11 to QD17, QD13 to QD18, Reg12 to Reg14, SPRV12 to SPRV16, SPRV13 to SPRV17, SPRV11 to SPRV18, Solenoid7 to Solenoid10, Solenoid5 to Solenoid11, Solenoid8 to Solenoid12, Solenoid6 to Solenoid9, Tank201 to Tank2, U21 to U20, U23 to U21, U19 to U22, U22 to U23
Connections:
- net at PT54.: no longer Engine10.
- new net: Needle_Valve8., U23.
- new net: Engine10., PT54.

Commit message: New year update
Parts:
- renumbered BV31 to BV77, Ball_Valve(ServoControlled)2 to Ball_Valve(ServoControlled)6, Ball_Valve4 to Ball_Valve10, Ball_Valve5 to Ball_Valve11, Ball_Valve6 to Ball_Valve12, BurstDisc2 to BurstDisc6, Burst_Disc12 to Burst_Disc29, Burst_Disc13 to Burst_Disc30, Check_Valve8 to Check_Valve18, Check_Valve10 to Check_Valve19, Check_Valve7 to Check_Valve20, Check_Valve6 to Check_Valve21, Check_Valve9 to Check_Valve22, CommonDomeTank3 to CommonDomeTank7, CommonDomeTank4 to CommonDomeTank8, Engine9 to Engine23, Engine10 to Engine24, Manual_Pressure_Gauge4 to Manual_Pressure_Gauge16, Needle_Valve7 to Needle_Valve23, Needle_Valve8 to Needle_Valve24, NitrogenTank2 to NitrogenTank4, PT51 to PT131, PT52 to PT132, PT48 to PT133, PT54 to PT134, PT53 to PT135, PT50 to PT136, PT55 to PT137, PT49 to PT138, Pressure_Regulator2 to Pressure_Regulator6, QD16 to QD46, QD17 to QD47, QD18 to QD48, Reg14 to Reg30, SPRV18 to SPRV40, SPRV16 to SPRV41, SPRV17 to SPRV42, Solenoid11 to Solenoid21, Solenoid9 to Solenoid22, Solenoid10 to Solenoid23, Solenoid12 to Solenoid24, Tank2 to Tank6, U22 to U65, U20 to U66, U23 to U67, U21 to U68
Connections:
- net at PT134.: no longer Engine24.
- new net: Needle_Valve24., U67.
- new net: Engine24., PT134.
