File: J-0_N2O_Bottles.kicad_sch (KiCad schematic)
At the start: 19 parts

Commit message: andrei it support
Parts:
- renumbered BV1 to BV?, C1 to C?, CV3 to CV?, Filter3 to Filter?, Hose1 to Hose?, Hose5 to Hose?, SPRV1 to SPRV?
Connections:
- net at Hose3.: now also CV5.; no longer BV3.
- net at CV5.: now also CV4., CV6., CV?., Hose?.; no longer Hose3.
- net at Hose?.: now also CV?.; no longer BV?.
- new net: BV3., Hose3.
- new net: BV?., Hose?.
Changed lines of the file:
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@@
 		(dnp no)
 		(fields_autoplaced yes)
-		(property "Reference" "Hose1"
+		(property "Reference" "Hose?"
 			(at 127 56.515 90)
 			(effects
@@
 		)
 		(instances
-			(project ""
-				(path "/045f1f05-3134-4b6d-91b6-463031104f1e/a0b6300e-76e9-4a18-afd6-e2d656b0d8f9/d375e00a-1ce3-4f93-9279-82acf09c7292/4f024983-2e1e-4582-8230-72c25523eed0"
-					(reference "Hose1")
+			(project "P_IDs"
+				(path "/045f1f05-3134-4b6d-91b6-463031104f1e/a0b6300e-76e9-4a18-afd6-e2d656b0d8f9/d375e00a-1ce3-4f93-9279-82acf09c7292/4f024983-2e1e-4582-8230-72c25523eed0"
+					(reference "Hose?")
 					(unit 1)
 				)
@@
 		(dnp no)
 		(fields_autoplaced yes)
-		(property "Reference" "BV1"
+		(property "Reference" "BV?"
 			(at 116.84 54.61 0)
 			(effects
@@
 		)
 		(instances
-			(project ""
-				(path "/045f1f05-3134-4b6d-91b6-463031104f1e/a0b6300e-76e9-4a18-afd6-e2d656b0d8f9/d375e00a-1ce3-4f93-9279-82acf09c7292/4f024983-2e1e-4582-8230-72c25523eed0"
-					(reference "BV1")
+			(project "P_IDs"
+				(path "/045f1f05-3134-4b6d-91b6-463031104f1e/a0b6300e-76e9-4a18-afd6-e2d656b0d8f9/d375e00a-1ce3-4f93-9279-82acf09c7292/4f024983-2e1e-4582-8230-72c25523eed0"
+					(reference "BV?")
 					(unit 1)
 				)
@@
 		(dnp no)
 		(fields_autoplaced yes)
-		(property "Reference" "Hose5"
+		(property "Reference" "Hose?"
 			(at 163.83 87.63 90)
 			(effects
@@
 		)
 		(instances
-			(project ""
-				(path "/045f1f05-3134-4b6d-91b6-463031104f1e/a0b6300e-76e9-4a18-afd6-e2d656b0d8f9/d375e00a-1ce3-4f93-9279-82acf09c7292/4f024983-2e1e-4582-8230-72c25523eed0"
-					(reference "Hose5")
+			(project "P_IDs"
+				(path "/045f1f05-3134-4b6d-91b6-463031104f1e/a0b6300e-76e9-4a18-afd6-e2d656b0d8f9/d375e00a-1ce3-4f93-9279-82acf09c7292/4f024983-2e1e-4582-8230-72c25523eed0"
+					(reference "Hose?")
 					(unit 1)
 				)
@@
 		(dnp no)
 		(fields_autoplaced yes)
-		(property "Reference" "Filter3"
+		(property "Reference" "Filter?"
 			(at 174.625 94.742 0)
 			(effects
@@
 		)
 		(instances
-			(project ""
-				(path "/045f1f05-3134-4b6d-91b6-463031104f1e/a0b6300e-76e9-4a18-afd6-e2d656b0d8f9/d375e00a-1ce3-4f93-9279-82acf09c7292/4f024983-2e1e-4582-8230-72c25523eed0"
-					(reference "Filter3")
+			(project "P_IDs"
+				(path "/045f1f05-3134-4b6d-91b6-463031104f1e/a0b6300e-76e9-4a18-afd6-e2d656b0d8f9/d375e00a-1ce3-4f93-9279-82acf09c7292/4f024983-2e1e-4582-8230-72c25523eed0"
+					(reference "Filter?")
 					(unit 1)
 				)
@@
 		(dnp no)
 		(fields_autoplaced yes)
-		(property "Reference" "SPRV1"
+		(property "Reference" "SPRV?"
 			(at 190.5 80.6449 90)
 			(effects
@@
 		)
 		(instances
-			(project ""
-				(path "/045f1f05-3134-4b6d-91b6-463031104f1e/a0b6300e-76e9-4a18-afd6-e2d656b0d8f9/d375e00a-1ce3-4f93-9279-82acf09c7292/4f024983-2e1e-4582-8230-72c25523eed0"
-					(reference "SPRV1")
+			(project "P_IDs"
+				(path "/045f1f05-3134-4b6d-91b6-463031104f1e/a0b6300e-76e9-4a18-afd6-e2d656b0d8f9/d375e00a-1ce3-4f93-9279-82acf09c7292/4f024983-2e1e-4582-8230-72c25523eed0"
+					(reference "SPRV?")
 					(unit 1)
 				)
@@
 		(on_board yes)
 		(dnp no)
-		(property "Reference" "C1"
+		(property "Reference" "C?"
 			(at 95.25 111.76 90)
 			(effects
@@
 		)
 		(instances
-			(project ""
-				(path "/045f1f05-3134-4b6d-91b6-463031104f1e/a0b6300e-76e9-4a18-afd6-e2d656b0d8f9/d375e00a-1ce3-4f93-9279-82acf09c7292/4f024983-2e1e-4582-8230-72c25523eed0"
-					(reference "C1")
+			(project "P_IDs"
+				(path "/045f1f05-3134-4b6d-91b6-463031104f1e/a0b6300e-76e9-4a18-afd6-e2d656b0d8f9/d375e00a-1ce3-4f93-9279-82acf09c7292/4f024983-2e1e-4582-8230-72c25523eed0"
+					(reference "C?")
 					(unit 1)
 				)
@@
 		(dnp no)
 		(fields_autoplaced yes)
-		(property "Reference" "CV3"
+		(property "Reference" "CV?"
 			(at 143.383 54.61 0)
 			(effects
@@
 		)
 		(instances
-			(project ""
-				(path "/045f1f05-3134-4b6d-91b6-463031104f1e/a0b6300e-76e9-4a18-afd6-e2d656b0d8f9/d375e00a-1ce3-4f93-9279-82acf09c7292/4f024983-2e1e-4582-8230-72c25523eed0"
-					(reference "CV3")
-					(unit 1)
-				)
+			(project "P_IDs"
+				(path "/045f1f05-3134-4b6d-91b6-463031104f1e/a0b6300e-76e9-4a18-afd6-e2d656b0d8f9/d375e00a-1ce3-4f93-9279-82acf09c7292/4f024983-2e1e-4582-8230-72c25523eed0"
+					(reference "CV?")
+					(unit 1)
+				)
