File: JO_N2_Bay.kicad_sch (KiCad schematic)
At the start: 16 parts

Commit message: andrei it support
Connections:
- net at Hose6.: now also MB_V1.; no longer CV8.
- net at MB_V1.: now also C6.; no longer Hose6.
- net at Hose7.: now also MB_V2.; no longer CV9.
- new net: CV8., Hose6.
- new net: CV9., Hose7.
Changed lines of the file:
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@@
 		(pin ""
-		)
-		(instances
-			(project ""
-				(path "/045f1f05-3134-4b6d-91b6-463031104f1e/a0b6300e-76e9-4a18-afd6-e2d656b0d8f9/d375e00a-1ce3-4f93-9279-82acf09c7292/4685d168-feae-4fe5-a995-eaab704f316f"
-					(reference "CV8")
-					(unit 1)
-				)
-			)
 		)
 	)
@@
 		(pin ""
 		)
-		(instances
-			(project ""
-				(path "/045f1f05-3134-4b6d-91b6-463031104f1e/a0b6300e-76e9-4a18-afd6-e2d656b0d8f9/d375e00a-1ce3-4f93-9279-82acf09c7292/4685d168-feae-4fe5-a995-eaab704f316f"
-					(reference "Hose6")
-					(unit 1)
-				)
-			)
-		)
 	)
 	(symbol
@@
 		(pin ""
 		)
-		(instances
-			(project ""
-				(path "/045f1f05-3134-4b6d-91b6-463031104f1e/a0b6300e-76e9-4a18-afd6-e2d656b0d8f9/d375e00a-1ce3-4f93-9279-82acf09c7292/4685d168-feae-4fe5-a995-eaab704f316f"
-					(reference "C6")
-					(unit 1)
-				)
-			)
-		)
 	)
 	(symbol
@@
 		(pin ""
 		)
-		(instances
-			(project ""
-				(path "/045f1f05-3134-4b6d-91b6-463031104f1e/a0b6300e-76e9-4a18-afd6-e2d656b0d8f9/d375e00a-1ce3-4f93-9279-82acf09c7292/4685d168-feae-4fe5-a995-eaab704f316f"
-					(reference "MB_V1")
-					(unit 1)
-				)
-			)
-		)
-	)
+	)
