File: N2_Reg.kicad_sch (KiCad schematic)
At the start: 4 parts

Commit message: andrei it support
Parts:
- removed unit 1 of Servo_Reg1
- renumbered Dome1 to Dome2, PT6 to PT7, Reg to Reg1, Servo_Reg1 to Servo_Reg2
Connections:
- new net: Dome2., PT7., Servo_Reg2.
- now unconnected: PT7.
Other:
- added sheet Pressure Panel (PressurePanel.kicad_sch)
- note added: "Back Panel"
- note added: "Top Panel"
- moved on the sheet: Dome2, PT7, Reg1A, Servo_Reg2B
