File: J0_N2.kicad_sch (KiCad schematic)
At the start: 0 parts

Commit message: andrei it support
Parts:
- added C10, C11, C12, C13: ~, symbol PID_symbols:Cylinder
- added CV12, CV13, CV14, CV15: ~, symbol PID_symbols:Check_Valve
- added Hose10, Hose11, Hose12, Hose13: ~, symbol PID_symbols:Hose
- added MB_V11, MB_V12, MB_V13, MB_V5: ~, symbol PID_symbols:MBallValve
Connections:
- new net: CV14., Hose12.
- new net: C10., MB_V5.
- new net: Hose10., MB_V5.
- new net: Hose11., MB_V11.
- new net: CV13., Hose11.
- new net: CV12., Hose10.
- new net: C11., MB_V11.
- new net: C12., MB_V12.
- new net: Hose12., MB_V12.
- new net: CV15., Hose13.
- new net: Hose13., MB_V13.
- new net: C13., MB_V13.
- new net N2_HP: CV12., CV13., CV14., CV15.

Commit message: update
Parts:
- renumbered C12 to C?, C11 to C?, C13 to C?, C10 to C?, CV14 to CV?, CV12 to CV?, CV15 to CV?, CV13 to CV?, Hose11 to Hose?, Hose12 to Hose?, Hose13 to Hose?, Hose10 to Hose?, MB_V5 to MB_V?, MB_V11 to MB_V?, MB_V13 to MB_V?, MB_V12 to MB_V?
Connections:
- net at Hose?.: now also MB_V?.; no longer CV?. (x2)
- net at Hose?.: now also CV?.; no longer MB_V?.
- net at MB_V?.: now also C?.; no longer Hose?.
- new net: CV?., Hose?. (x2)
- new net: Hose?., MB_V?.
Changed lines of the file:
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@@
 		(dnp no)
 		(fields_autoplaced yes)
-		(property "Reference" "CV14"
+		(property "Reference" "CV?"
 			(at 146.685 87.5029 90)
 			(effects
@@
 			(project "P_IDs"
 				(path "/045f1f05-3134-4b6d-91b6-463031104f1e/a0b6300e-76e9-4a18-afd6-e2d656b0d8f9/d375e00a-1ce3-4f93-9279-82acf09c7292/5e417696-9b80-46cd-a7e0-3b030f339530"
-					(reference "CV14")
+					(reference "CV?")
 					(unit 1)
 				)
@@
 		(dnp no)
 		(fields_autoplaced yes)
-		(property "Reference" "MB_V5"
+		(property "Reference" "MB_V?"
 			(at 106.68 68.5799 90)
 			(effects
@@
 			(project "P_IDs"
 				(path "/045f1f05-3134-4b6d-91b6-463031104f1e/a0b6300e-76e9-4a18-afd6-e2d656b0d8f9/d375e00a-1ce3-4f93-9279-82acf09c7292/5e417696-9b80-46cd-a7e0-3b030f339530"
-					(reference "MB_V5")
+					(reference "MB_V?")
 					(unit 1)
 				)
@@
 		(dnp no)
 		(fields_autoplaced yes)
-		(property "Reference" "Hose11"
+		(property "Reference" "Hose?"
 			(at 125.095 78.7399 0)
 			(effects
@@
 			(project "P_IDs"
 				(path "/045f1f05-3134-4b6d-91b6-463031104f1e/a0b6300e-76e9-4a18-afd6-e2d656b0d8f9/d375e00a-1ce3-4f93-9279-82acf09c7292/5e417696-9b80-46cd-a7e0-3b030f339530"
-					(reference "Hose11")
+					(reference "Hose?")
 					(unit 1)
 				)
@@
 		(dnp no)
 		(fields_autoplaced yes)
-		(property "Reference" "CV12"
+		(property "Reference" "CV?"
 			(at 107.95 87.5029 90)
 			(effects
@@
 			(project "P_IDs"
 				(path "/045f1f05-3134-4b6d-91b6-463031104f1e/a0b6300e-76e9-4a18-afd6-e2d656b0d8f9/d375e00a-1ce3-4f93-9279-82acf09c7292/5e417696-9b80-46cd-a7e0-3b030f339530"
-					(reference "CV12")
+					(reference "CV?")
 					(unit 1)
 				)
@@
 		(dnp no)
 		(fields_autoplaced yes)
-		(property "Reference" "MB_V11"
+		(property "Reference" "MB_V?"
 			(at 126.365 68.5799 90)
 			(effects
@@
 			(project "P_IDs"
 				(path "/045f1f05-3134-4b6d-91b6-463031104f1e/a0b6300e-76e9-4a18-afd6-e2d656b0d8f9/d375e00a-1ce3-4f93-9279-82acf09c7292/5e417696-9b80-46cd-a7e0-3b030f339530"
-					(reference "MB_V11")
+					(reference "MB_V?")
 					(unit 1)
 				)
@@
 		(dnp no)
 		(fields_autoplaced yes)
-		(property "Reference" "C12"
+		(property "Reference" "C?"
 			(at 149.225 46.3549 0)
 			(effects
@@
 			(project "P_IDs"
 				(path "/045f1f05-3134-4b6d-91b6-463031104f1e/a0b6300e-76e9-4a18-afd6-e2d656b0d8f9/d375e00a-1ce3-4f93-9279-82acf09c7292/5e417696-9b80-46cd-a7e0-3b030f339530"
-					(reference "C12")
+					(reference "C?")
 					(unit 1)
 				)
@@
 		(dnp no)
 		(fields_autoplaced yes)
-		(property "Reference" "C11"
+		(property "Reference" "C?"
 			(at 130.175 46.3549 0)
 			(effects
@@
 			(project "P_IDs"
 				(path "/045f1f05-3134-4b6d-91b6-463031104f1e/a0b6300e-76e9-4a18-afd6-e2d656b0d8f9/d375e00a-1ce3-4f93-9279-82acf09c7292/5e417696-9b80-46cd-a7e0-3b030f339530"
-					(reference "C11")
+					(reference "C?")
 					(unit 1)
 				)
@@
 		(dnp no)
 		(fields_autoplaced yes)
-		(property "Reference" "Hose12"
+		(property "Reference" "Hose?"
 			(at 144.145 78.7399 0)
 			(effects
@@
 			(project "P_IDs"
 				(path "/045f1f05-3134-4b6d-91b6-463031104f1e/a0b6300e-76e9-4a18-afd6-e2d656b0d8f9/d375e00a-1ce3-4f93-9279-82acf09c7292/5e417696-9b80-46cd-a7e0-3b030f339530"
-					(reference "Hose12")
+					(reference "Hose?")
 					(unit 1)
 				)
@@
 		(dnp no)
 		(fields_autoplaced yes)
-		(property "Reference" "Hose13"
+		(property "Reference" "Hose?"
 			(at 163.83 79.3749 0)
 			(effects
@@
 			(project "P_IDs"
 				(path "/045f1f05-3134-4b6d-91b6-463031104f1e/a0b6300e-76e9-4a18-afd6-e2d656b0d8f9/d375e00a-1ce3-4f93-9279-82acf09c7292/5e417696-9b80-46cd-a7e0-3b030f339530"
-					(reference "Hose13")
+					(reference "Hose?")
 					(unit 1)
 				)
@@
 		(dnp no)
 		(fields_autoplaced yes)
-		(property "Reference" "CV15"
+		(property "Reference" "CV?"
 			(at 166.37 88.1379 90)
 			(effects
@@
 			(project "P_IDs"
 				(path "/045f1f05-3134-4b6d-91b6-463031104f1e/a0b6300e-76e9-4a18-afd6-e2d656b0d8f9/d375e00a-1ce3-4f93-9279-82acf09c7292/5e417696-9b80-46cd-a7e0-3b030f339530"
-					(reference "CV15")
+					(reference "CV?")
 					(unit 1)
 				)
@@
 		(dnp no)
 		(fields_autoplaced yes)
-		(property "Reference" "MB_V13"
+		(property "Reference" "MB_V?"
 			(at 165.1 69.2149 90)
 			(effects
@@
 			(project "P_IDs"
 				(path "/045f1f05-3134-4b6d-91b6-463031104f1e/a0b6300e-76e9-4a18-afd6-e2d656b0d8f9/d375e00a-1ce3-4f93-9279-82acf09c7292/5e417696-9b80-46cd-a7e0-3b030f339530"
-					(reference "MB_V13")
+					(reference "MB_V?")
 					(unit 1)
 				)
@@
 		(dnp no)
 		(fields_autoplaced yes)
-		(property "Reference" "C13"
+		(property "Reference" "C?"
 			(at 168.91 46.9899 0)
 			(effects
@@
 			(project "P_IDs"
 				(path "/045f1f05-3134-4b6d-91b6-463031104f1e/a0b6300e-76e9-4a18-afd6-e2d656b0d8f9/d375e00a-1ce3-4f93-9279-82acf09c7292/5e417696-9b80-46cd-a7e0-3b030f339530"
-					(reference "C13")
+					(reference "C?")
 					(unit 1)
 				)
@@
 		(dnp no)
 		(fields_autoplaced yes)
-		(property "Reference" "C10"
+		(property "Reference" "C?"
 			(at 110.49 46.3549 0)
 			(effects
@@
 			(project "P_IDs"
 				(path "/045f1f05-3134-4b6d-91b6-463031104f1e/a0b6300e-76e9-4a18-afd6-e2d656b0d8f9/d375e00a-1ce3-4f93-9279-82acf09c7292/5e417696-9b80-46cd-a7e0-3b030f339530"
-					(reference "C10")
+					(reference "C?")
 					(unit 1)
 				)
@@
 		(dnp no)
 		(fields_autoplaced yes)
-		(property "Reference" "CV13"
+		(property "Reference" "CV?"
 			(at 127.635 87.5029 90)
 			(effects
@@
 			(project "P_IDs"
 				(path "/045f1f05-3134-4b6d-91b6-463031104f1e/a0b6300e-76e9-4a18-afd6-e2d656b0d8f9/d375e00a-1ce3-4f93-9279-82acf09c7292/5e417696-9b80-46cd-a7e0-3b030f339530"
-					(reference "CV13")
+					(reference "CV?")
 					(unit 1)
 				)
@@
 		(dnp no)
 		(fields_autoplaced yes)
-		(property "Reference" "Hose10"
+		(property "Reference" "Hose?"
 			(at 105.41 78.7399 0)
 			(effects
@@
 			(project "P_IDs"
 				(path "/045f1f05-3134-4b6d-91b6-463031104f1e/a0b6300e-76e9-4a18-afd6-e2d656b0d8f9/d375e00a-1ce3-4f93-9279-82acf09c7292/5e417696-9b80-46cd-a7e0-3b030f339530"
-					(reference "Hose10")
+					(reference "Hose?")
 					(unit 1)
 				)
@@
 		(dnp no)
 		(fields_autoplaced yes)
-		(property "Reference" "MB_V12"
+		(property "Reference" "MB_V?"
 			(at 145.415 68.5799 90)
 			(effects
@@
 			(project "P_IDs"
 				(path "/045f1f05-3134-4b6d-91b6-463031104f1e/a0b6300e-76e9-4a18-afd6-e2d656b0d8f9/d375e00a-1ce3-4f93-9279-82acf09c7292/5e417696-9b80-46cd-a7e0-3b030f339530"
-					(reference "MB_V12")
-					(unit 1)
-				)
+					(reference "MB_V?")
+					(unit 1)
+				)
