File: EREG_calibration.kicad_sch (KiCad schematic)
At the start: 13 parts, among them T12 Low pressure water tank, T7 High pressure COTS tank

Commit message: pts i think
Parts:
- PT4: value 100 -> 300
Connections:
- net at Needle_Valve1.: now also PT4., Pmatic_B_Valve3., T12.
- net at PT5.: now also BV26.
- net at BV26.: now also Pmatic_B_Valve3.; no longer PT5.
- net at nO_Sol5.: now also BV25., Burst_Disc6., SPRV10.
- new net: BV12., BV25., T7.
- now unconnected: Burst_Disc6., PT4., SPRV10., T12., T7.
Changed lines of the file:
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@@
 			)
 		)
-		(property "Value" "100"
+		(property "Value" "300"
 			(at 215.9 41.91 0)
 			(effects

Commit message: ereg calib
Parts:
- removed Burst_Disc6: Burst disc, symbol PID_symbols:Burst_Disc
- added Burst_Disc10: Burst Disc, symbol PID_symbols:Burst_Disc
- added CV5: Check Valve, symbol PID_symbols:Check_Valve
- added H5: High Pressure hose, symbol PID_symbols:Hose
- added H6: High Pressure Hose, symbol PID_symbols:Hose
- added H7: Low Pressure Hose, symbol PID_symbols:Hose
- added Manual_Pressure_Gauge1: Manual Pressure Gauge, symbol PID_symbols:Manual_Pressure_Gauge
- added PT6: 300, symbol PID_symbols:Pressure_Transducer
- added Reg4: Mechanical regulator, symbol PID_symbols:Pressure_Regulator
- added nO_Sol6: Normally open Solenoid Valve, symbol PID_symbols:Normally Open Solenoid
- BV25: value Electronic regulator valve -> Electronic Regulator
- PT5: value 100 -> 300
- SPRV10: value Safety pressure relief valve -> Safety Pressure Relief Valve
- nO_Sol5: value Normally open solenoid vent valve -> Normally Open Solenoid Valve
Connections:
- net at Needle_Valve1.: now also Pmatic_B_Valve3., T12.
- net at BV12.: now also H5.2; no longer C1.
- net at PT5.: now also BV26.
- net at BV26.: now also H7.2; no longer PT5.
- net at nO_Sol5.: now also PT4., SPRV10., Burst_Disc10., CV5.
- new net: BV12., H6.1, Reg4., T7.
- new net: H7.1, Pmatic_B_Valve3.
- new net: BV25., H6.2, Manual_Pressure_Gauge1., PT6.
- new net: BV25., CV5.
- new net: Reg4., nO_Sol6.
- new net: C1., H5.1
- now unconnected: PT4., Pmatic_B_Valve3., Pmatic_B_Valve3., SPRV10., T12., T7.
Other:
- note added: "To water catch Tank"

Commit message: ereg
Parts:
- added PT8: 300, symbol PID_symbols:Pressure_Transducer
- nO_Sol5: value Normally Open Solenoid Valve -> Low pressure vent valve
- nO_Sol6: value Normally open Solenoid Valve -> High pressure vent valve
Connections:
- net at nO_Sol5.: now also Burst_Disc10., CV5., PT4., SPRV10.
- net at Needle_Valve1.: now also Pmatic_B_Valve3., T12.
- net at BV12., H5.2: now also PT8.
- net at PT5.: now also BV26.
- net at BV26.: now also H7.2; no longer PT5.
- net at Manual_Pressure_Gauge1.: now also BV25., H6.2, PT6.
- new net: BV12., H6.1, Reg4., T7.
- now unconnected: Burst_Disc10., PT4., PT6., Pmatic_B_Valve3., SPRV10., T12., T7.
Changed lines of the file:
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@@
+	)
+	(junction
+		(at 62.23 57.15)
+		(diameter 0)
+		(color 0 0 0 0)
 	)
 	(junction
@@
 	(wire
 		(pts
+			(xy 62.23 57.15) (xy 69.85 57.15)
+		)
+		(stroke
+			(width 0)
+			(type default)
+		)
+	)
+	(wire
+		(pts
 			(xy 163.83 113.03) (xy 143.51 113.03)
 		)
@@
 	(wire
 		(pts
-			(xy 77.47 57.15) (xy 88.9 57.15)
+			(xy 82.55 57.15) (xy 88.9 57.15)
 		)
 		(stroke
@@
 	(wire
 		(pts
-			(xy 53.34 57.15) (xy 64.77 57.15)
+			(xy 53.34 57.15) (xy 62.23 57.15)
 		)
 		(stroke
@@
 		(pts
 			(xy 162.56 71.12) (xy 176.53 71.12)
+		)
+		(stroke
+			(width 0)
+			(type default)
+		)
+	)
+	(wire
+		(pts
+			(xy 62.23 50.8) (xy 62.23 57.15)
 		)
 		(stroke
@@
 			)
 		)
-		(property "Value" "Normally Open Solenoid Valve"
-			(at 156.21 34.29 0)
+		(property "Value" "Low pressure vent valve"
+			(at 156.21 33.02 0)
 			(effects
 				(font
@@
 	(symbol
 		(lib_id "PID_symbols:Ball_Valve")
-		(at 67.31 57.15 0)
+		(at 72.39 57.15 0)
 		(unit 1)
 		(exclude_from_sim no)
@@
 		(fields_autoplaced yes)
 		(property "Reference" "BV12"
-			(at 71.12 50.8 0)
+			(at 76.2 50.8 0)
 			(effects
 				(font
@@
 		)
 		(property "Value" "High pressure valve"
-			(at 71.12 53.34 0)
-			(effects
-				(font
-					(size 1.27 1.27)
-				)
-			)
-		)
-		(property "Footprint" ""
-			(at 67.31 57.15 0)
-			(effects
-				(font
-					(size 1.27 1.27)
-				)
-				(hide yes)
-			)
-		)
-		(property "Datasheet" ""
-			(at 67.31 57.15 0)
-			(effects
-				(font
-					(size 1.27 1.27)
-				)
-				(hide yes)
-			)
-		)
-		(property "Description" ""
-			(at 67.31 57.15 0)
+			(at 76.2 53.34 0)
+			(effects
+				(font
+					(size 1.27 1.27)
+				)
+			)
+		)
+		(property "Footprint" ""
+			(at 72.39 57.15 0)
+			(effects
+				(font
+					(size 1.27 1.27)
+				)
+				(hide yes)
+			)
+		)
+		(property "Datasheet" ""
+			(at 72.39 57.15 0)
+			(effects
+				(font
+					(size 1.27 1.27)
+				)
+				(hide yes)
+			)
+		)
+		(property "Description" ""
+			(at 72.39 57.15 0)
 			(effects
 				(font
@@
 	)
 	(symbol
+		(lib_name "Pressure_Transducer_3")
+		(lib_id "PID_symbols:Pressure_Transducer")
+		(at 62.23 48.26 0)
+		(unit 1)
+		(exclude_from_sim no)
+		(in_bom yes)
+		(on_board yes)
+		(dnp no)
+		(fields_autoplaced yes)
+		(property "Reference" "PT8"
+			(at 62.23 43.18 0)
+			(effects
+				(font
+					(size 1.27 1.27)
+				)
+				(hide yes)
+			)
+		)
+		(property "Value" "300"
+			(at 62.23 49.53 0)
+			(effects
+				(font
+					(size 1.27 1.27)
+				)
+			)
+		)
+		(property "Footprint" ""
+			(at 62.23 48.26 0)
+			(effects
+				(font
+					(size 1.27 1.27)
+				)
+				(hide yes)
+			)
+		)
+		(property "Datasheet" ""
+			(at 62.23 48.26 0)
+			(effects
+				(font
+					(size 1.27 1.27)
+				)
+				(hide yes)
+			)
+		)
+		(property "Description" ""
+			(at 62.23 48.26 0)
+			(effects
+				(font
+					(size 1.27 1.27)
+				)
+				(hide yes)
+			)
+		)
+		(pin ""
+		)
+		(pin ""
+		)
+		(pin ""
+		)
+		(instances
+			(project ""
+				(path "/045f1f05-3134-4b6d-91b6-463031104f1e/e8ba80f5-7b5d-4dc5-95fa-8f3f89e19357"
+					(reference "PT8")
+					(unit 1)
+				)
+			)
+		)
+	)
+	(symbol
 		(lib_name "Normally Open Solenoid_1")
 		(lib_id "PID_symbols:Normally Open Solenoid")
@@
 			)
 		)
-		(property "Value" "Normally open Solenoid Valve"
+		(property "Value" "High pressure vent valve"
 			(at 92.71 87.6299 90)
 			(effects

Commit message: overwriting babz
Parts:
- renumbered BV12 to BV28, BV25 to BV29, BV26 to BV30, Burst_Disc10 to Burst_Disc11, CV5 to CV31, Manual_Pressure_Gauge1 to Manual_Pressure_Gauge3, Needle_Valve1 to Needle_Valve6, PT8 to PT44, PT6 to PT45, PT4 to PT46, PT5 to PT47, Reg4 to Reg13, SPRV10 to SPRV15, T12 to T11, T7 to T12, nO_Sol5 to nO_Sol18, nO_Sol6 to nO_Sol19
Connections:
- net at nO_Sol18.: now also Burst_Disc11., CV31., PT46., SPRV15.
- net at Needle_Valve6.: now also Pmatic_B_Valve3., T11.
- net at PT47.: now also BV30.
- net at BV30.: now also H7.2; no longer PT47.
- net at Manual_Pressure_Gauge3.: now also BV29., H6.2, PT45.
- new net: BV28., H6.1, Reg13., T12.
- now unconnected: Burst_Disc11., PT45., PT46., Pmatic_B_Valve3., SPRV15., T11., T12.
Changed lines of the file:
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@@
 		(dnp no)
 		(fields_autoplaced yes)
-		(property "Reference" "nO_Sol5"
+		(property "Reference" "nO_Sol18"
 			(at 156.21 31.75 0)
 			(effects
@@
 			(project ""
 				(path "/045f1f05-3134-4b6d-91b6-463031104f1e/e8ba80f5-7b5d-4dc5-95fa-8f3f89e19357"
-					(reference "nO_Sol5")
+					(reference "nO_Sol18")
 					(unit 1)
 				)
@@
 		(dnp no)
 		(fields_autoplaced yes)
-		(property "Reference" "SPRV10"
+		(property "Reference" "SPRV15"
 			(at 156.8451 30.48 90)
 			(effects
@@
 			(project ""
 				(path "/045f1f05-3134-4b6d-91b6-463031104f1e/e8ba80f5-7b5d-4dc5-95fa-8f3f89e19357"
-					(reference "SPRV10")
+					(reference "SPRV15")
 					(unit 1)
 				)
@@
 		(dnp no)
 		(fields_autoplaced yes)
-		(property "Reference" "Needle_Valve1"
+		(property "Reference" "Needle_Valve6"
 			(at 220.98 61.5949 90)
 			(effects
@@
 			(project ""
 				(path "/045f1f05-3134-4b6d-91b6-463031104f1e/e8ba80f5-7b5d-4dc5-95fa-8f3f89e19357"
-					(reference "Needle_Valve1")
+					(reference "Needle_Valve6")
 					(unit 1)
 				)
@@
 		(dnp no)
 		(fields_autoplaced yes)
-		(property "Reference" "BV12"
+		(property "Reference" "BV28"
 			(at 76.2 50.8 0)
 			(effects
@@
 			(project ""
 				(path "/045f1f05-3134-4b6d-91b6-463031104f1e/e8ba80f5-7b5d-4dc5-95fa-8f3f89e19357"
-					(reference "BV12")
+					(reference "BV28")
 					(unit 1)
 				)
@@
 		(dnp no)
 		(fields_autoplaced yes)
-		(property "Reference" "PT5"
+		(property "Reference" "PT47"
 			(at 163.83 97.79 0)
 			(effects
@@
 			(project ""
 				(path "/045f1f05-3134-4b6d-91b6-463031104f1e/e8ba80f5-7b5d-4dc5-95fa-8f3f89e19357"
-					(reference "PT5")
+					(reference "PT47")
 					(unit 1)
 				)
@@
 		(dnp no)
 		(fields_autoplaced yes)
-		(property "Reference" "Manual_Pressure_Gauge1"
+		(property "Reference" "Manual_Pressure_Gauge3"
 			(at 109.22 44.45 0)
 			(effects
@@
 			(project ""
 				(path "/045f1f05-3134-4b6d-91b6-463031104f1e/e8ba80f5-7b5d-4dc5-95fa-8f3f89e19357"
-					(reference "Manual_Pressure_Gauge1")
+					(reference "Manual_Pressure_Gauge3")
 					(unit 1)
 				)
@@
 		(dnp no)
 		(fields_autoplaced yes)
-		(property "Reference" "T12"
+		(property "Reference" "T11"
 			(at 194.31 25.3999 0)
 			(effects
@@
 			(project ""
 				(path "/045f1f05-3134-4b6d-91b6-463031104f1e/e8ba80f5-7b5d-4dc5-95fa-8f3f89e19357"
-					(reference "T12")
+					(reference "T11")
 					(unit 1)
 				)
@@
 		(dnp no)
 		(fields_autoplaced yes)
-		(property "Reference" "CV5"
+		(property "Reference" "CV31"
 			(at 159.893 50.8 0)
 			(effects
@@
 			(project ""
 				(path "/045f1f05-3134-4b6d-91b6-463031104f1e/e8ba80f5-7b5d-4dc5-95fa-8f3f89e19357"
-					(reference "CV5")
+					(reference "CV31")
 					(unit 1)
 				)
@@
 		(dnp no)
 		(fields_autoplaced yes)
-		(property "Reference" "Reg4"
+		(property "Reference" "Reg13"
 			(at 93.98 70.5474 90)
 			(effects
@@
 			(project ""
 				(path "/045f1f05-3134-4b6d-91b6-463031104f1e/e8ba80f5-7b5d-4dc5-95fa-8f3f89e19357"
-					(reference "Reg4")
+					(reference "Reg13")
 					(unit 1)
 				)
@@
 		(dnp no)
 		(fields_autoplaced yes)
-		(property "Reference" "Burst_Disc10"
+		(property "Reference" "Burst_Disc11"
 			(at 167.64 76.2 0)
 			(effects
@@
 			(project ""
 				(path "/045f1f05-3134-4b6d-91b6-463031104f1e/e8ba80f5-7b5d-4dc5-95fa-8f3f89e19357"
-					(reference "Burst_Disc10")
+					(reference "Burst_Disc11")
 					(unit 1)
 				)
@@
 		(dnp no)
 		(fields_autoplaced yes)
-		(property "Reference" "BV26"
+		(property "Reference" "BV30"
 			(at 193.04 102.2349 90)
 			(effects
@@
 			(project ""
 				(path "/045f1f05-3134-4b6d-91b6-463031104f1e/e8ba80f5-7b5d-4dc5-95fa-8f3f89e19357"
-					(reference "BV26")
+					(reference "BV30")
 					(unit 1)
 				)
@@
 		(dnp no)
 		(fields_autoplaced yes)
-		(property "Reference" "PT4"
+		(property "Reference" "PT46"
 			(at 160.02 66.04 0)
 			(effects
@@
 			(project ""
 				(path "/045f1f05-3134-4b6d-91b6-463031104f1e/e8ba80f5-7b5d-4dc5-95fa-8f3f89e19357"
-					(reference "PT4")
+					(reference "PT46")
 					(unit 1)
 				)
@@
 		(dnp no)
 		(fields_autoplaced yes)
-		(property "Reference" "PT6"
+		(property "Reference" "PT45"
 			(at 121.92 60.96 0)
 			(effects
@@
 			(project ""
 				(path "/045f1f05-3134-4b6d-91b6-463031104f1e/e8ba80f5-7b5d-4dc5-95fa-8f3f89e19357"
-					(reference "PT6")
+					(reference "PT45")
 					(unit 1)
 				)
@@
 		(dnp no)
 		(fields_autoplaced yes)
-		(property "Reference" "T7"
+		(property "Reference" "T12"
 			(at 93.98 35.5599 0)
 			(effects
@@
 			(project ""
 				(path "/045f1f05-3134-4b6d-91b6-463031104f1e/e8ba80f5-7b5d-4dc5-95fa-8f3f89e19357"
-					(reference "T7")
+					(reference "T12")
 					(unit 1)
 				)
@@
 		(dnp no)
 		(fields_autoplaced yes)
-		(property "Reference" "BV25"
+		(property "Reference" "BV29"
 			(at 142.24 50.8 0)
 			(effects
@@
 			(project ""
 				(path "/045f1f05-3134-4b6d-91b6-463031104f1e/e8ba80f5-7b5d-4dc5-95fa-8f3f89e19357"
-					(reference "BV25")
+					(reference "BV29")
 					(unit 1)
 				)
@@
 		(dnp no)
 		(fields_autoplaced yes)
-		(property "Reference" "PT8"
+		(property "Reference" "PT44"
 			(at 62.23 43.18 0)
 			(effects
@@
 			(project ""
 				(path "/045f1f05-3134-4b6d-91b6-463031104f1e/e8ba80f5-7b5d-4dc5-95fa-8f3f89e19357"
-					(reference "PT8")
+					(reference "PT44")
 					(unit 1)
 				)
@@
 		(dnp no)
 		(fields_autoplaced yes)
-		(property "Reference" "nO_Sol6"
+		(property "Reference" "nO_Sol19"
 			(at 82.55 88.2651 90)
 			(effects
@@
 			(project ""
 				(path "/045f1f05-3134-4b6d-91b6-463031104f1e/e8ba80f5-7b5d-4dc5-95fa-8f3f89e19357"
-					(reference "nO_Sol6")
-					(unit 1)
-				)
+					(reference "nO_Sol19")
+					(unit 1)
+				)

Commit message: New year update
Parts:
- renumbered BV28 to BV69, BV29 to BV70, BV30 to BV71, Burst_Disc11 to Burst_Disc28, C1 to C2, CV31 to CV72, H5 to H12, H6 to H13, H7 to H14, Manual_Pressure_Gauge3 to Manual_Pressure_Gauge13, Needle_Valve6 to Needle_Valve20, PT44 to PT119, PT45 to PT120, PT46 to PT121, PT47 to PT122, Pmatic_B_Valve3 to Pmatic_B_Valve5, Reg13 to Reg28, SPRV15 to SPRV39, T12 to T25, T11 to T26, nO_Sol19 to nO_Sol45, nO_Sol18 to nO_Sol46
Connections:
- net at nO_Sol46.: now also Burst_Disc28., CV72., PT121., SPRV39.
- net at Needle_Valve20.: now also Pmatic_B_Valve5., T26.
- net at PT122.: now also BV71.
- net at BV71.: now also H14.2; no longer PT122.
- net at Manual_Pressure_Gauge13.: now also BV70., H13.2, PT120.
- new net: BV69., H13.1, Reg28., T25.
- now unconnected: Burst_Disc28., PT120., PT121., Pmatic_B_Valve5., SPRV39., T25., T26.

Commit message: j0
Parts:
- renumbered BV69 to BV1, BV70 to BV2, BV71 to BV3, Burst_Disc28 to Burst_Disc1, C2 to C1, CV72 to CV1, H12 to H1, H13 to H2, H14 to H3, Manual_Pressure_Gauge13 to Manual_Pressure_Gauge3, Needle_Valve20 to Needle_Valve1, PT119 to PT1, PT120 to PT2, PT121 to PT3, PT122 to PT4, Pmatic_B_Valve5 to Pmatic_B_Valve1, Reg28 to Reg1, SPRV39 to SPRV2, T26 to T1, T25 to T2, nO_Sol46 to nO_Sol1, nO_Sol45 to nO_Sol2
Connections:
- net at nO_Sol1.: now also Burst_Disc1., CV1., PT3., SPRV2.
- net at Needle_Valve1.: now also Pmatic_B_Valve1., T1.
- net at PT4.: now also BV3.
- net at BV3.: now also H3.; no longer PT4.
- net at Pmatic_B_Valve1.: no longer H3.1
- net at Manual_Pressure_Gauge3.: now also BV2., H2., PT2.
- net at C1.: now also H1.; no longer H1.1
- new net: BV1., H2., Reg1., T2.
- new net: BV1., H1., PT1.
- new net: H3., Pmatic_B_Valve1.
- now unconnected: Burst_Disc1., PT1., PT2., PT3., Pmatic_B_Valve1., SPRV2., T1., T2.

Commit message: more silwood stuff
Parts:
- renumbered H1 to Hose1, H2 to Hose2, H3 to Hose3, PT1 to PT5, PT2 to PT6, PT3 to PT7, PT4 to PT8, Pmatic_B_Valve1 to Pmatic_B_Valve2, Reg1 to Servo_Reg1, T2 to T1, T1 to T2, nO_Sol2 to nO_Sol1, nO_Sol1 to nO_Sol2
Connections:
- net at nO_Sol2.: now also Burst_Disc1., CV1., PT7., SPRV2.
- net at Needle_Valve1.: now also Pmatic_B_Valve2., T2.
- net at PT8.: now also BV3.
- net at BV3.: now also Hose3.; no longer PT8.
- net at Pmatic_B_Valve2.: no longer Hose3.
- net at Manual_Pressure_Gauge3.: now also BV2., Hose2., PT6.
- new net: BV1., Hose2., Servo_Reg1., T1.
- new net: BV1., Hose1., PT5.
- new net: Hose3., Pmatic_B_Valve2.
- now unconnected: Burst_Disc1., PT5., PT6., PT7., Pmatic_B_Valve2., SPRV2., T1., T2.

Commit message: Formatiing
Parts:
- renumbered BV1 to BV69, BV2 to BV70, BV3 to BV71, Burst_Disc1 to Burst_Disc28, C1 to C2, CV1 to CV72, Hose1 to H12, Hose2 to H13, Hose3 to H14, Manual_Pressure_Gauge3 to Manual_Pressure_Gauge13, Needle_Valve1 to Needle_Valve20, PT5 to PT119, PT6 to PT120, PT7 to PT121, PT8 to PT122, Pmatic_B_Valve2 to Pmatic_B_Valve5, Servo_Reg1 to Reg28, SPRV2 to SPRV39, T1 to T25, T2 to T26, nO_Sol1 to nO_Sol45, nO_Sol2 to nO_Sol46
Connections:
- net at nO_Sol46.: now also Burst_Disc28., CV72., PT121., SPRV39.
- net at Needle_Valve20.: now also Pmatic_B_Valve5., T26.
- net at PT122.: now also BV71.
- net at BV71.: now also H14.2; no longer PT122.
- net at Pmatic_B_Valve5.: no longer H14.
- net at Manual_Pressure_Gauge13.: now also BV70., H13.2, PT120.
- net at C2.: now also H12.1; no longer H12.
- new net: BV69., H13.1, Reg28., T25.
- new net: BV69., H12.2, PT119.
- new net: H14.1, Pmatic_B_Valve5.
- now unconnected: Burst_Disc28., PT119., PT120., PT121., Pmatic_B_Valve5., SPRV39., T25., T26.
