File: Feed.kicad_sch (KiCad schematic)
At the start: 36 parts

Commit message: clean pnid
Parts:
- removed EREG_Fuel, OX_EREG: ~, symbol PID_symbols:Pressure_Regulator
- removed U38, U39: ~, symbol PID_symbols:stop
- added BV45: ~, symbol PID_symbols:Ball_Valve
- added Burst_Disc6: ~, symbol PID_symbols:Burst_Disc
- added CV16: ~, symbol PID_symbols:Check_Valve
- added Fuel_EREG, OX_EREG, Servo_Reg23, Servo_Reg9: ~, symbol PID_symbols:Pressure_Regulator
- added MB_V1: ~, symbol PID_symbols:MBallValve
- added PT24: ~, symbol PID_symbols:Pressure_Transducer
- added Pmatic_B_Valve17: ~, symbol PID_symbols:Pneumatic_Rotary_Ball_Valve
- added QD30: ~, symbol PID_symbols:Quick_Disconnect
- added SPRV11: ~, symbol PID_symbols:SPRV
- added TC15: ~, symbol PID_symbols:Thermocouple
- added nC_Sol14: ~, symbol PID_symbols:Normally_Closed_Solenoid
- added nO_Sol32: ~, symbol PID_symbols:Normally Open Solenoid
- renumbered SPRV to PRV
Connections:
- net 1-4: now also Fuel_EREG., OX_EREG.
- net 3-8: now also Fuel_EREG., OX_EREG.
Other:
- note added: "1 INCH"
- note added: "Burst Disk"
- note added: "Check-Valve"
- note added: "Manifold"
- note added: "Manual Ball Valve"
- note added: "Normally Closed Solenoid"
- note added: "Normally Open Solenoid"
- note added: "Pneumatic Actuated Valve, NO/NC (Normally Open/Closed)"
- note added: "Pressure Regulator"
- note added: "Pressure Relief Valve"
- note added: "Pressure Transducer"
- note added: "Quick-Disconnect"
- note added: "Servo Ball Valve"
- note added: "Servo-Actuated Pressure Regulator"
- note added: "Thermocouple"
- note removed: "->"
- note removed: "<-Pipe label"
- note removed: "Add global labels to define pipe types. (button on right of the screen)"
- note removed: "Add the 'stop' symbol to seperate pipes definitions:"
- note removed: "Default size is 10 (very small)"
- note removed: "Global label size only for demo."
- note removed: "[Normally stops are added at the Tee (circle) section]"
- note removed: "stop symbol"
- moved on the sheet: Burst_Disc, Burst_Disc5, CV, Chamber, Engine, FUELPT, FuelA, FuelFill_Needle_Valve, FuelMain_BV, Fuel_Inj, Fuel_Vent_Sol, N2A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

Commit message: euroc app
Parts:
- removed Fuel_EREG, OX_EREG, Servo_Reg9: ~, symbol PID_symbols:Pressure_Regulator
- removed Pmatic_B_Valve17: ~, symbol PID_symbols:Pneumatic_Rotary_Ball_Valve
- added CV26: ~, symbol PID_symbols:Check_Valve
- added E-REG (x3): ~, symbol PID_symbols:Ball_Valve
- added T16: ~, symbol PID_symbols:Tank
- renumbered FUELPT to FUEL_TK, N2FILLPT to N2_TK, OXEREGPT to OX_EREG
Connections:
- net 1-4: now also OXFill_QD., U72., CV26., E-REG., E-REG.
- net 3-8: now also E-REG., E-REG.; no longer OXFill_QD., U72.
- net OX_GSS: now reaches OXFill_QD.
- net FUEL_GSS: now reaches FuelFill_Needle_Valve.
- net N2_GSS: now reaches N2Fill_QD.
Other:
- note added: "Electronic Pressure Regulator (Ball Valve)"
- note added: "FUEL"
- note added: "N2"
- note added: "OX"
- note added: "Tank"
- note removed: "Pneumatic Actuated Valve, NO/NC (Normally Open/Closed)"
- note removed: "Servo-Actuated Pressure Regulator"
- company: (none) -> Imperial College London Rocketry
- title: (none) -> Ember Flight Vehicle P&ID
