File: GFS.kicad_sch (KiCad schematic)
At the start: 44 parts

Commit message: j0
Parts:
- renumbered 1 to 11, 11 to 111, 1 to 12, 1 to 13, 1 to 14, Adj_ChokeN2 to Adj_ChokeN1, CV1 to CV16, CV2 to CV17, Filter1 to Filter4, Filter2 to Filter5, Fuel to Fuel1, FuelVehicle to FuelVehicle1, Hose_FillN2 to Hose_FillN1, MB_FuelFill to MB_FuelFill1, MB_FuelPress to MB_FuelPress1, MB_FuelVent to MB_FuelVent1, Manual_Pressure_Gauge1 to Manual_Pressure_Gauge4, Manual_Pressure_Gauge2 to Manual_Pressure_Gauge5, Manual_Pressure_GaugeN2 to Manual_Pressure_GaugeN1, N2 to N1, N2O_QD to N2O_QD1, N2_QD to N2_QD1, Needle_Valve1 to Needle_Valve3, Needle_Valve2 to Needle_Valve4, Needle_Valve_Vent to Needle_Valve_Vent1, PT3 to PT15, PT5 to PT16, PT1 to PT17, PT2 to PT18, PT4 to PT19, Pmatic_FillN2 to Pmatic_FillN1, Pmatic_VentVehicle to Pmatic_VentVehicle1, Pmatic_VentVehicleN2 to Pmatic_VentVehicleN1, Relief_ValveN2O to Relief_ValveN2O1, U1 to U16, U2 to U17
Connections:
- net 1-4: no longer 13.
- net at 13.: no longer N2_QD1.
- net at PT19.: now also Adj_ChokeN1., Needle_Valve_Vent1.
- net at PT17.: now also BV_Fill1., Needle_Valve3.
- net at 11.: no longer N2O_QD1.
- net at 111.: no longer Filter5.
- net at Manual_Pressure_Gauge4.: now also N2O_1.
- net at Manual_Pressure_GaugeN1., N1.: no longer Hose_FillN1.
- net at Filter4.: no longer 14.
- net at MB_FuelFill1.: no longer 12.
- net at 12.: no longer FuelVehicle1.
- new net: Manual_Pressure_Gauge5., N2O_2.
- new net: CV16., CV17., PT15., Pmatic_VentVehicle1., Relief_ValveN2O1.
- new net: BV_Fill2., Needle_Valve4., PT18.
- now unconnected: 11., 111., 14., Filter4., Filter5., Hose_FillN1., Manual_Pressure_Gauge5., Needle_Valve3., Needle_Valve4., Needle_Valve_Vent1., PT15., PT18., Pmatic_VentVehicle1., Relief_ValveN2O1.

Commit message: more silwood stuff
Parts:
- renumbered 5/2Solenoid3 to 5/2Solenoid?, 5/2Solenoid2 to 5/2Solenoid?, 5/2Solenoid1 to 5/2Solenoid?, Adj_ChokeN1 to Adj_Choke1, BV_Fill1 to BV1, BV_Fill2 to BV2, Fuel1 to C1, N1 to C1, N2O_2 to C?, N2O_1 to C?, Hose_FillN1 to Hose1, 14 to Hose1, 11 to Hose2, 111 to Hose3, 13 to Hose4, 12 to Hose5, MB_FuelVent1 to MB_V1, MB_FuelFill1 to MB_V1, MB_FuelPress1 to MB_V1, Manual_Pressure_GaugeN1 to Manual_Pressure_Gauge1, Manual_Pressure_Gauge4 to Manual_Pressure_Gauge5, Manual_Pressure_Gauge5 to Manual_Pressure_Gauge6, Needle_Valve_Vent1 to Needle_Valve1, PT17 to PT24, PT15 to PT25, PT18 to PT26, PT19 to PT27, PT16 to PT28, Pmatic_FillN1 to Pmatic_B_Valve1, Pmatic_VentVehicle1 to Pmatic_B_Valve1, Pmatic_VentVehicleN1 to Pmatic_B_Valve1, FuelVehicle1 to QD1, N2O_QD1 to QD?, N2_QD1 to QD?, Relief_ValveN2O1 to Relief_Valve?, U16 to U25, U17 to U26
Connections:
- net at PT27.: now also Adj_Choke1., Needle_Valve1.
- net at PT24.: now also BV1., Needle_Valve3.
- net at Manual_Pressure_Gauge5.: now also C?.
- net at Manual_Pressure_Gauge1.: now also C1.
- new net: CV16., CV17., PT25., Pmatic_B_Valve1., Relief_Valve?.
- new net: BV2., Needle_Valve4., PT26.
- now unconnected: Needle_Valve1., Needle_Valve3., Needle_Valve4., PT25., PT26., Pmatic_B_Valve1., Relief_Valve?.

Commit message: Formatiing
Parts:
- removed U25, U26: ~, symbol PID_symbols:stop
- added U1, U2: ~, symbol PID_symbols:stop
- gave numbers to parts that had none: 8
- renumbered Hose4 to 1, Hose2 to 1, Hose5 to 1, Hose1 to 1, Hose3 to 11, Adj_Choke1 to Adj_ChokeN2, BV1 to BV_Fill1, BV2 to BV_Fill2, CV16 to CV1, CV17 to CV2, Filter4 to Filter1, Filter5 to Filter2, C1 to Fuel, QD1 to FuelVehicle, Hose1 to Hose_FillN2, MB_V1 to MB_FuelFill, MB_V1 to MB_FuelPress, MB_V1 to MB_FuelVent, Manual_Pressure_Gauge5 to Manual_Pressure_Gauge1, Manual_Pressure_Gauge6 to Manual_Pressure_Gauge2, Manual_Pressure_Gauge1 to Manual_Pressure_GaugeN2, C1 to N2, Needle_Valve3 to Needle_Valve1, Needle_Valve4 to Needle_Valve2, Needle_Valve1 to Needle_Valve_Vent, PT24 to PT1, PT26 to PT2, PT25 to PT3, PT27 to PT4, PT28 to PT5, Pmatic_B_Valve1 to Pmatic_FillN2, Pmatic_B_Valve1 to Pmatic_VentVehicle, Pmatic_B_Valve1 to Pmatic_VentVehicleN2
Connections:
- net 1-2: now also U1., U2.
- net 1-4: now also 1.
- net TI-HP: now also U1., U2.
- net at PT4.: now also Adj_ChokeN2., Hose_FillN2., Needle_Valve_Vent.
- net at PT1.: now also 1., BV_Fill1., Needle_Valve1.
- net at Manual_Pressure_Gauge2., N2O_2.: now also Filter2.
- net at N2O_QD.: now also 1.
- net at 11.: now also Filter2.
- net at 1.: now also CV1., CV2., PT3., Pmatic_VentVehicle., Relief_ValveN2O.
- net at Manual_Pressure_Gauge1.: now also Filter1., N2O_1.
- net at Hose_FillN2.: now also Manual_Pressure_GaugeN2., N2.
- net at Filter1.: now also 1.
- net at MB_FuelFill.: now also 1.
- net at 1.: now also FuelVehicle.
- new net: 1., N2_QD.
- new net: 11., BV_Fill2., Needle_Valve2., PT2.
- now unconnected: Manual_Pressure_GaugeN2., Needle_Valve1., Needle_Valve2., Needle_Valve_Vent., PT2., PT3., Pmatic_VentVehicle., Relief_ValveN2O.
Other:
- note added: "3-4 INCH"
- moved on the sheet: 5/2Solenoid1, 5/2Solenoid2, 5/2Solenoid3, Adj_ChokeN2, Air_Compressor1, BV_Fill1, BV_Fill2, CV1, CV2, Fuel, FuelVehicle, Hose_FillN2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
