File: GFS.kicad_sch (KiCad schematic)
At the start: 42 parts

Commit message: SPRVs GFS
Parts:
- added SPRV_N, SPRV_O(1), SPRV_O(2): ~, symbol PID_symbols:SPRV
Connections:
- net 1-4: now also SPRV_N., SPRV_O(1)., SPRV_O(2).; no longer PT.
- net at QD.: now also Hose.
- net at Hose.: no longer QD.
Other:
- moved on the sheet: PT

Commit message: clean pnid
Parts:
- removed 5/2Solenoid: ~, symbol PID_symbols:Solenoid_5/2
- removed U25, U26: ~, symbol PID_symbols:stop
- added BV46: ~, symbol PID_symbols:Ball_Valve
- added Burst_Disc24: ~, symbol PID_symbols:Burst_Disc
- added CF9: ~, symbol PID_symbols:Coriolis_Flow
- added CV17: ~, symbol PID_symbols:Check_Valve
- added DP9: ~, symbol PID_symbols:DP_Sensor
- added Dome9: ~, symbol PID_symbols:Dome_Reg
- added Filter4: ~, symbol PID_symbols:Filter
- added MB_V20: ~, symbol PID_symbols:MBallValve
- added Manual_Pressure_Gauge27: ~, symbol PID_symbols:Manual_Pressure_Gauge
- added PT25: ~, symbol PID_symbols:Pressure_Transducer
- added Pmatic_B_Valve18: ~, symbol PID_symbols:Pneumatic_Rotary_Ball_Valve
- added QD31: ~, symbol PID_symbols:Quick_Disconnect
- added SPRV12: ~, symbol PID_symbols:SPRV
- added Servo_Reg10, Servo_Reg24: ~, symbol PID_symbols:Pressure_Regulator
- added TC16: ~, symbol PID_symbols:Thermocouple
- added nC_Sol15: ~, symbol PID_symbols:Normally_Closed_Solenoid
- added nO_Sol33: ~, symbol PID_symbols:Normally Open Solenoid
- renumbered QD to Fuel_Vehicle, SPRV_O(1) to PRV, SPRV_N to PRV, SPRV_O(2) to PRV
Connections:
- net D: no longer Manual_BV.
- net Pn: now also Manual_BV.
- net at QD.: now also Hose.
- net at Hose.: no longer QD.
Other:
- note added: "1 INCH"
- note added: "3-4 INCH"
- note added: "Burst Disk"
- note added: "Check-Valve"
- note added: "Coriolis Flow Meter"
- note added: "Differential Pressure Transducer"
- note added: "Dome-Loaded Regulator"
- note added: "Filter"
- note added: "Manual Ball Valve"
- note added: "Normally Closed Solenoid"
- note added: "Normally Open Solenoid"
- note added: "Pneumatic Actuated Valve, NO/NC (Normally Open/Closed)"
- note added: "Pressure Gauge"
- note added: "Pressure Regulator"
- note added: "Pressure Relief Valve"
- note added: "Pressure Transducer"
- note added: "Quick-Disconnect"
- note added: "Servo Ball Valve"
- note added: "Servo-Actuated Pressure Regulator"
- note added: "Thermocouple"
- note added: "Valve Pneumatics Line"
- note removed: "->"
- note removed: "<-Pipe label"
- note removed: "Add global labels to define pipe types. (button on right of the screen)"
- note removed: "Add the 'stop' symbol to seperate pipes definitions:"
- note removed: "Default size is 10 (very small)"
- note removed: "Global label size only for demo."
- note removed: "[Normally stops are added at the Tee (circle) section]"
- note removed: "stop symbol"
- moved on the sheet: 5/2Solenoid?, Air_Compressor1, BV, BV_HighPressure, CV, Filter, Fuel, Fuel_Vehicle, Hose, Manual_BV, Manual_Pressure_Gauge, Manual_Pressure_Gauge5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

Commit message: euroc app
Parts:
- removed Air_Compressor1: ~, symbol PID_symbols:Air_Compressor
- removed Burst_Disc24: ~, symbol PID_symbols:Burst_Disc
- removed CF9: ~, symbol PID_symbols:Coriolis_Flow
- removed DP9: ~, symbol PID_symbols:DP_Sensor
- removed Dome9: ~, symbol PID_symbols:Dome_Reg
- removed Fuel: ~, symbol PID_symbols:Cylinder
- removed Relief_Valve: ~, symbol PID_symbols:Relief_Valve
- removed Servo_Reg10, Servo_Reg24: ~, symbol PID_symbols:Pressure_Regulator
- removed nC_Sol15: ~, symbol PID_symbols:Normally_Closed_Solenoid
- removed nO_Sol33: ~, symbol PID_symbols:Normally Open Solenoid
- added 5/2Solenoid: ~, symbol PID_symbols:Solenoid_5/2
- added Air_Compressor1, Air_Compressor2: ~, symbol PID_symbols:Air_Compressor
- added C5: ~, symbol PID_symbols:Cylinder
- added Hose33: ~, symbol PID_symbols:Hose
- added NeedleValve: ~, symbol PID_symbols:Needle_Valve
- added T14, T15: ~, symbol PID_symbols:Tank
- renumbered 5/2Solenoid to 5/2Solenoid?, Pmatic_B_Valve to NO
Connections:
- net 1-4: now also T14.
- net Pn: now also Manual_BV., 5/2Solenoid., Air_Compressor1.-UB, T14.
- net N20_Vehicle: now reaches QD.
- net at Hose.: no longer QD.
- net Fuel_Vehicle: now reaches Fuel_Vehicle.
- net N2_VEHICLE renamed N2_Vehicle
- new net: Hose., QD.
- new net: Air_Compressor1., Manual_BV.
Other:
- note added: "Air Compressor"
- note added: "Bottle"
- note added: "Ground Fuel"
- note added: "Ground Fuel Tank"
- note added: "Hose"
- note added: "Manual Pressure Gauge"
- note added: "Needle Valve"
- note removed: "Burst Disk"
- note removed: "Coriolis Flow Meter"
- note removed: "Differential Pressure Transducer"
- note removed: "Dome-Loaded Regulator"
- note removed: "Normally Closed Solenoid"
- note removed: "Normally Open Solenoid"
- note removed: "Pressure Gauge"
- note removed: "Pressure Regulator"
- note removed: "Servo-Actuated Pressure Regulator"
- note removed: "Valve Pneumatics Line"
- company: (none) -> Imperial College London Rocketry
- title: (none) -> Ground FIlling Station P&ID
- moved on the sheet: 5/2Solenoid?, OX

Commit message: euroc app 2
Parts:
- added Pneumatic: ~, symbol PID_symbols:Pressure_Transducer
- renumbered PT to N2_Bottle, PT to N2_Hose, PT to Ox_Bottle_1, PT26 to Ox_Bottle_2, PT to Ox_Hose
Connections:
- net 1-4: now also N2_Bottle.
- net Pn: now also Pneumatic.
- net at Hose.: no longer QD.
- new net: Hose., QD.
