File: L9.kicad_sch (KiCad schematic)
At the start: 38 parts

Commit message: added universal key
Connections:
- net at QD7.: now also CV13.
- net at CV13.: now also BV8., T3.; no longer QD7.
- net at PT23.: now also CV14., T3.
- net at CV15.: now also QD8.
- net at QD8.: no longer CV15.
- net at Engine2.: now also BV8., PT20.; no longer BV7.
- net at PT21.: no longer Engine2.
- net at Needle_Valve3.: now also BV7.
- new net: CV12., CV14., Reg6.
- new net: PT17., Reg6., Solenoid4., T1.
- new net: BV7., Engine2.
- new net: Engine2., PT21.
- now unconnected: PT17., PT20., Solenoid4., T1.
Changed lines of the file:
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@@
 	)
 	(symbol
+		(lib_name "Quick_Disconnect_2")
 		(lib_id "PID_symbols:Quick_Disconnect")
 		(at 213.36 153.67 0)
@@
 	)
 	(symbol
+		(lib_name "Pressure_Transducer_3")
 		(lib_id "PID_symbols:Pressure_Transducer")
 		(at 245.11 53.34 0)
@@
 	)
 	(symbol
+		(lib_name "Pressure_Transducer_4")
 		(lib_id "PID_symbols:Pressure_Transducer")
 		(at 38.1 119.38 0)
@@
 	)
 	(symbol
+		(lib_name "Check_Valve_1")
 		(lib_id "PID_symbols:Check_Valve")
 		(at 259.08 140.97 0)
@@
 	)
 	(symbol
+		(lib_name "Check_Valve_2")
 		(lib_id "PID_symbols:Check_Valve")
 		(at 198.12 153.67 0)
@@
 	)
 	(symbol
+		(lib_name "Ball_Valve_1")
 		(lib_id "PID_symbols:Ball_Valve")
 		(at 138.43 99.06 0)
@@
 	)
 	(symbol
+		(lib_name "Pressure_Regulator_1")
 		(lib_id "PID_symbols:Pressure_Regulator")
 		(at 179.07 53.34 0)
@@
 	)
 	(symbol
+		(lib_name "Tank_1")
 		(lib_id "PID_symbols:Tank")
 		(at 154.94 33.02 0)
@@
 	)
 	(symbol
+		(lib_name "Check_Valve_3")
 		(lib_id "PID_symbols:Check_Valve")
 		(at 209.55 53.34 0)
@@
 	)
 	(symbol
+		(lib_name "Needle_Valve_1")
 		(lib_id "PID_symbols:Needle_Valve")
 		(at 93.98 105.41 0)
@@
 	)
 	(symbol
+		(lib_name "Pressure_Transducer_5")
 		(lib_id "PID_symbols:Pressure_Transducer")
 		(at 144.78 106.68 0)
@@
 	)
 	(symbol
+		(lib_name "Pressure_Transducer_6")
 		(lib_id "PID_symbols:Pressure_Transducer")
 		(at 168.91 168.91 0)
@@
 	)
 	(symbol
+		(lib_name "SPRV_1")
 		(lib_id "PID_symbols:SPRV")
 		(at 134.62 119.38 0)
@@
 	)
 	(symbol
+		(lib_name "Ball_Valve_2")
 		(lib_id "PID_symbols:Ball_Valve")
 		(at 34.29 69.85 0)
@@
 	)
 	(symbol
+		(lib_name "Check_Valve_4")
 		(lib_id "PID_symbols:Check_Valve")
 		(at 35.56 91.44 0)
@@
 	)
 	(symbol
+		(lib_name "Burst_Disc_2")
 		(lib_id "PID_symbols:Burst_Disc")
 		(at 146.05 64.77 0)
@@
 	)
 	(symbol
+		(lib_name "Ball_Valve_3")
 		(lib_id "PID_symbols:Ball_Valve")
 		(at 139.7 156.21 0)
@@
 	)
 	(symbol
+		(lib_name "Pressure_Transducer_7")
 		(lib_id "PID_symbols:Pressure_Transducer")
 		(at 135.89 45.72 0)
@@
 	)
 	(symbol
+		(lib_name "SPRV_2")
 		(lib_id "PID_symbols:SPRV")
 		(at 177.8 72.39 0)
@@
 	)
 	(symbol
+		(lib_name "Tank_2")
 		(lib_id "PID_symbols:Tank")
 		(at 154.94 125.73 0)
@@
 	)
 	(symbol
+		(lib_name "Pressure_Transducer_1")
 		(lib_id "PID_symbols:Pressure_Transducer")
 		(at 168.91 162.56 0)
@@
 	)
 	(symbol
+		(lib_name "Quick_Disconnect_1")
 		(lib_id "PID_symbols:Quick_Disconnect")
 		(at 38.1 128.27 0)
@@
 	)
 	(symbol
+		(lib_name "Pressure_Transducer_2")
 		(lib_id "PID_symbols:Pressure_Transducer")
 		(at 166.37 154.94 0)
@@
 	)
 	(symbol
+		(lib_name "Burst_Disc_1")
 		(lib_id "PID_symbols:Burst_Disc")
 		(at 173.99 118.11 0)

Commit message: overwriting babz
Parts:
- renumbered BV5 to BV11, BV6 to BV12, BV8 to BV13, BV7 to BV14, Burst_Disc3 to Burst_Disc5, Burst_Disc5 to Burst_Disc6, CV12 to CV15, CV11 to CV16, CV15 to CV17, CV13 to CV18, Engine2 to Engine4, Needle_Valve2 to Needle_Valve1, Needle_Valve3 to Needle_Valve2, PT17 to PT14, PT23 to PT15, PT19 to PT16, PT18 to PT17, PT16 to PT18, PT20 to PT19, PT21 to PT20, PT22 to PT21, QD8 to QD10, QD7 to QD11, QD6 to QD9, Reg6 to Reg7, Reg5 to Reg8, SPRV5 to SPRV6, SPRV4 to SPRV7, SPRV3 to SPRV8, Solenoid4 to Solenoid1, Solenoid1 to Solenoid4, T1 to T4, T2 to T5, T3 to T6
Connections:
- net at QD11.: now also CV18.
- net at CV18.: now also BV13., T6.; no longer QD11.
- net at PT15.: now also CV14., T6.
- net at CV17.: now also QD10.
- net at QD10.: no longer CV17.
- net at Engine4.: now also BV13., PT19.; no longer BV14.
- net at PT20.: no longer Engine4.
- net at Needle_Valve2.: now also BV14.
- new net: CV14., CV15., Reg7.
- new net: PT14., Reg7., Solenoid1., T4.
- new net: BV14., Engine4.
- new net: Engine4., PT20.
- now unconnected: PT14., PT19., Solenoid1., T4.

Commit message: New year update
Parts:
- renumbered BV11 to BV48, BV12 to BV49, BV14 to BV50, BV13 to BV51, Burst_Disc5 to Burst_Disc19, Burst_Disc4 to Burst_Disc20, Burst_Disc6 to Burst_Disc21, CV16 to CV50, CV15 to CV51, CV18 to CV52, CV14 to CV53, CV17 to CV54, Engine4 to Engine15, Needle_Valve1 to Needle_Valve13, Needle_Valve2 to Needle_Valve14, PT18 to PT78, PT14 to PT79, PT17 to PT80, PT16 to PT81, PT19 to PT82, PT20 to PT83, PT21 to PT84, PT15 to PT85, QD9 to QD32, QD11 to QD33, QD10 to QD34, Reg8 to Reg20, Reg7 to Reg21, SPRV8 to SPRV26, SPRV7 to SPRV27, SPRV6 to SPRV28, Solenoid4 to Solenoid13, Solenoid2 to Solenoid14, Solenoid3 to Solenoid15, Solenoid1 to Solenoid16, T4 to T14, T5 to T15, T6 to T16
Connections:
- net at QD33.: now also CV52.
- net at CV52.: now also BV51., T16.; no longer QD33.
- net at PT85.: now also CV53., T16.
- net at CV54.: now also QD34.
- net at QD34.: no longer CV54.
- net at Engine15.: now also BV51., PT82.; no longer BV50.
- net at PT83.: no longer Engine15.
- net at Needle_Valve14.: now also BV50.
- new net: CV51., CV53., Reg21.
- new net: PT79., Reg21., Solenoid16., T14.
- new net: BV50., Engine15.
- new net: Engine15., PT83.
- now unconnected: PT79., PT82., Solenoid16., T14.

Commit message: j0
Parts:
- renumbered BV48 to BV18, BV49 to BV19, BV51 to BV20, BV50 to BV21, Burst_Disc20 to Burst_Disc7, Burst_Disc19 to Burst_Disc8, Burst_Disc21 to Burst_Disc9, CV53 to CV29, CV51 to CV30, CV50 to CV31, CV54 to CV32, CV52 to CV33, Engine15 to Engine4, Needle_Valve13 to Needle_Valve5, Needle_Valve14 to Needle_Valve6, PT79 to PT24, PT85 to PT25, PT81 to PT26, PT80 to PT27, PT78 to PT28, PT82 to PT29, PT83 to PT30, PT84 to PT31, QD32 to QD5, QD34 to QD6, QD33 to QD7, Reg21 to Reg7, Reg20 to Reg8, SPRV28 to SPRV11, SPRV27 to SPRV12, SPRV26 to SPRV13, Solenoid16 to Solenoid1, Solenoid14 to Solenoid2, Solenoid15 to Solenoid3, Solenoid13 to Solenoid4, T14 to T3, T15 to T4, T16 to T8
Connections:
- net at QD7.: now also CV33.
- net at CV33.: now also BV20., T8.; no longer QD7.
- net at PT25.: now also CV29., T8.
- net at CV32.: now also QD6.
- net at QD6.: no longer CV32.
- net at Engine4.: now also BV20., PT29.; no longer BV21.
- net at PT30.: no longer Engine4.
- net at Needle_Valve6.: now also BV21.
- new net: CV29., CV30., Reg7.
- new net: PT24., Reg7., Solenoid1., T3.
- new net: BV21., Engine4.
- new net: Engine4., PT30.
- now unconnected: PT24., PT29., Solenoid1., T3.

Commit message: more silwood stuff
Parts:
- renumbered BV18 to BV17, BV19 to BV18, BV21 to BV19, Burst_Disc8 to Burst_Disc7, Burst_Disc7 to Burst_Disc8, CV31 to CV29, CV33 to CV31, CV29 to CV32, CV32 to CV33, Engine4 to Engine5, PT28 to PT37, PT24 to PT38, PT27 to PT39, PT26 to PT40, PT29 to PT41, PT30 to PT42, PT31 to PT43, PT25 to PT44, QD5 to QD6, QD6 to QD8, SPRV12 to SPRV14, SPRV11 to SPRV15, Reg8 to Servo_Reg7, Reg7 to Servo_Reg8, Solenoid4 to Solenoid1, Solenoid1 to Solenoid4
Connections:
- net at QD7.: now also CV31.
- net at CV31.: now also BV20., T8.; no longer QD7.
- net at PT44.: now also CV32., T8.
- net at CV33.: now also QD8.
- net at QD8.: no longer CV33.
- net at Engine5.: now also BV20., PT41.
- net at BV19.: now also Needle_Valve6.; no longer Engine5.
- net at PT42.: no longer Engine5.
- new net: CV30., CV32., Servo_Reg8.
- new net: PT38., Servo_Reg8., Solenoid4., T3.
- new net: BV19., Engine5.
- new net: Engine5., PT42.
- now unconnected: PT38., PT41., Solenoid4., T3.

Commit message: Formatiing
Parts:
- renumbered BV17 to BV48, BV18 to BV49, BV19 to BV50, BV20 to BV51, Burst_Disc7 to Burst_Disc19, Burst_Disc8 to Burst_Disc20, Burst_Disc9 to Burst_Disc21, CV29 to CV50, CV30 to CV51, CV31 to CV52, CV32 to CV53, CV33 to CV54, Engine5 to Engine15, Needle_Valve5 to Needle_Valve13, Needle_Valve6 to Needle_Valve14, PT37 to PT78, PT38 to PT79, PT39 to PT80, PT40 to PT81, PT41 to PT82, PT42 to PT83, PT43 to PT84, PT44 to PT85, QD6 to QD32, QD7 to QD33, QD8 to QD34, Servo_Reg7 to Reg20, Servo_Reg8 to Reg21, SPRV13 to SPRV26, SPRV14 to SPRV27, SPRV15 to SPRV28, Solenoid1 to Solenoid13, Solenoid2 to Solenoid14, Solenoid3 to Solenoid15, Solenoid4 to Solenoid16, T3 to T14, T4 to T15, T8 to T16
Connections:
- net at QD33.: now also CV52.
- net at CV52.: now also BV51., T16.; no longer QD33.
- net at PT85.: now also CV53., T16.
- net at CV54.: now also QD34.
- net at QD34.: no longer CV54.
- net at Engine15.: now also BV51., PT82.
- net at BV50.: now also Needle_Valve14.; no longer Engine15.
- net at PT83.: no longer Engine15.
- new net: CV51., CV53., Reg21.
- new net: PT79., Reg21., Solenoid16., T14.
- new net: BV50., Engine15.
- new net: Engine15., PT83.
- now unconnected: PT79., PT82., Solenoid16., T14.
