File: Pluto_Common_Dome.kicad_sch (KiCad schematic)
At the start: 47 parts

Commit message: overwriting babz
Parts:
- renumbered BV11 to BV27, Ball_Valve(ServoControlled)100 to Ball_Valve(ServoControlled)1, BurstDisc123 to BurstDisc1, Burst_Disc7 to Burst_Disc10, Burst_Disc4 to Burst_Disc9, Check_Valve4 to Check_Valve1, Check_Valve3 to Check_Valve2, Check_Valve112 to Check_Valve3, Check_Valve5 to Check_Valve4, Check_Valve2 to Check_Valve5, CommonDomeTank2 to CommonDomeTank1, CommonDomeTank1 to CommonDomeTank2, Engine3 to Engine7, Engine2 to Engine8, Manual_Pressure_Gauge3 to Manual_Pressure_Gauge1, Needle_Valve2 to Needle_Valve4, Needle_Valve3 to Needle_Valve5, PT11 to PT36, PT14 to PT37, PT10 to PT38, PT7 to PT39, PT9 to PT40, PT38 to PT41, PT37 to PT42, PT15 to PT43, Pressure_Regulator123 to Pressure_Regulator1, QD6 to QD13, QD8 to QD14, QD7 to QD15, Reg8 to Reg12, SPRV4 to SPRV12, SPRV5 to SPRV13, SPRV3 to SPRV14, Solenoid2 to Solenoid5, Solenoid3 to Solenoid6, Solenoid1 to Solenoid7, Solenoid4 to Solenoid8, Tank200 to Tank1, U5 to U16, U2 to U17, U3 to U18, U4 to U19
Connections:
- net D: now also Engine8., PT42.
- new net: Needle_Valve5., U19.

Commit message: New year update
Parts:
- renumbered BV27 to BV52, Ball_Valve(ServoControlled)1 to Ball_Valve(ServoControlled)4, Ball_Valve1 to Ball_Valve7, Ball_Valve2 to Ball_Valve8, Ball_Valve3 to Ball_Valve9, BurstDisc1 to BurstDisc4, Burst_Disc9 to Burst_Disc22, Burst_Disc10 to Burst_Disc23, Check_Valve3 to Check_Valve12, Check_Valve5 to Check_Valve13, Check_Valve2 to Check_Valve14, Check_Valve1 to Check_Valve15, Check_Valve4 to Check_Valve16, CommonDomeTank1 to CommonDomeTank5, CommonDomeTank2 to CommonDomeTank6, Engine7 to Engine16, Engine8 to Engine17, Manual_Pressure_Gauge2 to Manual_Pressure_Gauge10, Manual_Pressure_Gauge1 to Manual_Pressure_Gauge9, Needle_Valve4 to Needle_Valve15, Needle_Valve5 to Needle_Valve16, NitrogenTank1 to NitrogenTank3, PT39 to PT86, PT40 to PT87, PT36 to PT88, PT42 to PT89, PT41 to PT90, PT38 to PT91, PT43 to PT92, PT37 to PT93, Pressure_Regulator1 to Pressure_Regulator4, QD13 to QD35, QD14 to QD36, QD15 to QD37, Reg12 to Reg22, SPRV14 to SPRV29, SPRV12 to SPRV30, SPRV13 to SPRV31, Solenoid7 to Solenoid17, Solenoid5 to Solenoid18, Solenoid6 to Solenoid19, Solenoid8 to Solenoid20, Tank1 to Tank4, U18 to U49, U16 to U50, U19 to U51, U17 to U52
Connections:
- new net: Needle_Valve16., U51.

Commit message: Feed System Work
Connections:
- new net: Needle_Valve16., U51.
Changed lines of the file:
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@@
 	(title_block
 		(title "Pluto Propulsion P&ID")
-		(date "2025-02-25")
 		(company "ICLR")
 	)

Commit message: j0
Parts:
- renumbered BV52 to BV26, Ball_Valve(ServoControlled)4 to Ball_Valve(ServoControlled)2, Ball_Valve7 to Ball_Valve1, Ball_Valve8 to Ball_Valve2, Ball_Valve9 to Ball_Valve3, BurstDisc4 to BurstDisc2, Burst_Disc22 to Burst_Disc12, Burst_Disc23 to Burst_Disc13, Check_Valve15 to Check_Valve2, Check_Valve14 to Check_Valve3, Check_Valve12 to Check_Valve4, Check_Valve16 to Check_Valve5, Check_Valve13 to Check_Valve6, CommonDomeTank5 to CommonDomeTank1, CommonDomeTank6 to CommonDomeTank2, Engine16 to Engine7, Engine17 to Engine8, Manual_Pressure_Gauge9 to Manual_Pressure_Gauge8, Manual_Pressure_Gauge10 to Manual_Pressure_Gauge9, Needle_Valve16 to Needle_Valve10, Needle_Valve15 to Needle_Valve9, NitrogenTank3 to NitrogenTank1, PT88 to PT40, PT93 to PT41, PT91 to PT42, PT86 to PT43, PT87 to PT44, PT90 to PT45, PT89 to PT46, PT92 to PT47, Pressure_Regulator4 to Pressure_Regulator2, QD35 to QD11, QD36 to QD12, QD37 to QD13, Reg22 to Reg10, SPRV30 to SPRV17, SPRV31 to SPRV18, SPRV29 to SPRV19, Solenoid18 to Solenoid5, Solenoid19 to Solenoid6, Solenoid17 to Solenoid7, Solenoid20 to Solenoid8, Tank4 to Tank2, U50 to U36, U52 to U37, U49 to U38, U51 to U39
Connections:
- new net: Needle_Valve10., U39.

Commit message: more silwood stuff
Parts:
- renumbered Ball_Valve1 to BV1, Ball_Valve2 to BV2, Ball_Valve(ServoControlled)2 to BV2, BV26 to BV25, Ball_Valve3 to BV3, BurstDisc2 to Burst_Disc2, Check_Valve4 to CV2, Check_Valve6 to CV3, Check_Valve3 to CV4, Check_Valve2 to CV5, Check_Valve5 to CV6, Engine7 to Engine8, Engine8 to Engine9, Manual_Pressure_Gauge8 to Manual_Pressure_Gauge10, Manual_Pressure_Gauge9 to Manual_Pressure_Gauge11, PT43 to PT53, PT44 to PT54, PT40 to PT55, PT46 to PT56, PT45 to PT57, PT42 to PT58, PT47 to PT59, PT41 to PT60, QD11 to QD12, QD12 to QD13, QD13 to QD14, SPRV17 to SPRV20, SPRV18 to SPRV21, Reg10 to Servo_Reg10, Pressure_Regulator2 to Servo_Reg2, Solenoid7 to Solenoid5, Solenoid5 to Solenoid6, Solenoid6 to Solenoid7, NitrogenTank1 to T1, Tank2 to T2, U38 to U51, U36 to U52, U39 to U53, U37 to U54
Connections:
- new net: Needle_Valve10., U53.

Commit message: Formatiing
Parts:
- renumbered BV25 to BV52, BV2 to Ball_Valve(ServoControlled)4, BV1 to Ball_Valve7, BV2 to Ball_Valve8, BV3 to Ball_Valve9, Burst_Disc2 to BurstDisc4, Burst_Disc12 to Burst_Disc22, Burst_Disc13 to Burst_Disc23, CV2 to Check_Valve12, CV3 to Check_Valve13, CV4 to Check_Valve14, CV5 to Check_Valve15, CV6 to Check_Valve16, CommonDomeTank1 to CommonDomeTank5, CommonDomeTank2 to CommonDomeTank6, Engine8 to Engine16, Engine9 to Engine17, Manual_Pressure_Gauge11 to Manual_Pressure_Gauge10, Manual_Pressure_Gauge10 to Manual_Pressure_Gauge9, Needle_Valve9 to Needle_Valve15, Needle_Valve10 to Needle_Valve16, T1 to NitrogenTank3, PT53 to PT86, PT54 to PT87, PT55 to PT88, PT56 to PT89, PT57 to PT90, PT58 to PT91, PT59 to PT92, PT60 to PT93, Servo_Reg2 to Pressure_Regulator4, QD12 to QD35, QD13 to QD36, QD14 to QD37, Servo_Reg10 to Reg22, SPRV19 to SPRV29, SPRV20 to SPRV30, SPRV21 to SPRV31, Solenoid5 to Solenoid17, Solenoid6 to Solenoid18, Solenoid7 to Solenoid19, Solenoid8 to Solenoid20, T2 to Tank4, U51 to U49, U52 to U50, U53 to U51, U54 to U52
Connections:
- new net: Needle_Valve16., U51.
