File: Pluto_GSS.kicad_sch (KiCad schematic)
At the start: 8 parts

Commit message: Big Pluto Commit, baboucarr jeng imperial college london second year aeronautics student.
Connections:
- net at N2QD1.: now also BV_N2_filling_Vent1., BV_N2_servo1.
- net at Needle_Valve_N1filling_vent1.: now also BV_N2_servo1.
- new net: BV_Oxfilling_Servo1., BV_Oxfilling_Vent1., OxQD1.
- now unconnected: BV_N2_filling_Vent1., BV_Oxfilling_Vent1., OxQD1.
Changed lines of the file:
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@@
 		(instances
 			(project "P_IDs"
-				(path "/045f1f05-3134-4b6d-91b6-463031104f1e/9704eb45-91f5-4a31-9f50-e6cb45eec041"
+				(path "/045f1f05-3134-4b6d-91b6-463031104f1e/462f9fab-58b5-4b75-b4d3-2a00576f9247"
 					(reference "BV_Oxfilling_Servo1")
 					(unit 1)
@@
 		(instances
 			(project "P_IDs"
-				(path "/045f1f05-3134-4b6d-91b6-463031104f1e/9704eb45-91f5-4a31-9f50-e6cb45eec041"
+				(path "/045f1f05-3134-4b6d-91b6-463031104f1e/462f9fab-58b5-4b75-b4d3-2a00576f9247"
 					(reference "N2QD1")
 					(unit 1)
@@
 		(instances
 			(project "P_IDs"
-				(path "/045f1f05-3134-4b6d-91b6-463031104f1e/9704eb45-91f5-4a31-9f50-e6cb45eec041"
+				(path "/045f1f05-3134-4b6d-91b6-463031104f1e/462f9fab-58b5-4b75-b4d3-2a00576f9247"
 					(reference "Needle_Valve_N1filling_vent1")
 					(unit 1)
@@
 		(instances
 			(project "P_IDs"
-				(path "/045f1f05-3134-4b6d-91b6-463031104f1e/9704eb45-91f5-4a31-9f50-e6cb45eec041"
+				(path "/045f1f05-3134-4b6d-91b6-463031104f1e/462f9fab-58b5-4b75-b4d3-2a00576f9247"
 					(reference "BV_N2_filling_Vent1")
 					(unit 1)
@@
 		(instances
 			(project "P_IDs"
-				(path "/045f1f05-3134-4b6d-91b6-463031104f1e/9704eb45-91f5-4a31-9f50-e6cb45eec041"
+				(path "/045f1f05-3134-4b6d-91b6-463031104f1e/462f9fab-58b5-4b75-b4d3-2a00576f9247"
 					(reference "BV_Oxfilling_Vent1")
 					(unit 1)
@@
 		(instances
 			(project "P_IDs"
-				(path "/045f1f05-3134-4b6d-91b6-463031104f1e/9704eb45-91f5-4a31-9f50-e6cb45eec041"
+				(path "/045f1f05-3134-4b6d-91b6-463031104f1e/462f9fab-58b5-4b75-b4d3-2a00576f9247"
 					(reference "Needle_Valve_Oxfilling1")
 					(unit 1)
@@
 		(instances
 			(project "P_IDs"
-				(path "/045f1f05-3134-4b6d-91b6-463031104f1e/9704eb45-91f5-4a31-9f50-e6cb45eec041"
+				(path "/045f1f05-3134-4b6d-91b6-463031104f1e/462f9fab-58b5-4b75-b4d3-2a00576f9247"
 					(reference "BV_N2_servo1")
 					(unit 1)
@@
 		(instances
 			(project "P_IDs"
-				(path "/045f1f05-3134-4b6d-91b6-463031104f1e/9704eb45-91f5-4a31-9f50-e6cb45eec041"
+				(path "/045f1f05-3134-4b6d-91b6-463031104f1e/462f9fab-58b5-4b75-b4d3-2a00576f9247"
 					(reference "OxQD1")
 					(unit 1)

Commit message: added universal key
Connections:
- net at N2QD1.: now also BV_N2_filling_Vent1., BV_N2_servo1.
- net at Needle_Valve_N1filling_vent1.: now also BV_N2_servo1.
- new net: BV_Oxfilling_Servo1., BV_Oxfilling_Vent1., OxQD1.
- now unconnected: BV_N2_filling_Vent1., BV_Oxfilling_Vent1., OxQD1.
Changed lines of the file:
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@@
 	)
 	(symbol
+		(lib_name "Ball_Valve_1")
 		(lib_id "PID_symbols:Ball_Valve")
 		(at 199.39 120.65 0)
@@
 	)
 	(symbol
-		(lib_name "Ball_Valve_3")
+		(lib_name "Ball_Valve_2")
 		(lib_id "PID_symbols:Ball_Valve")
 		(at 226.06 31.75 0)
@@
 	)
 	(symbol
-		(lib_name "Ball_Valve_1")
 		(lib_id "PID_symbols:Ball_Valve")
 		(at 226.06 97.79 0)
@@
 	)
 	(symbol
-		(lib_name "Ball_Valve_2")
+		(lib_name "Ball_Valve_3")
 		(lib_id "PID_symbols:Ball_Valve")
 		(at 199.39 50.8 0)

Commit message: overwriting babz
Parts:
- removed BV_N2_filling_Vent1, BV_N2_servo1, BV_Oxfilling_Servo1, BV_Oxfilling_Vent1: ~, symbol PID_symbols:Ball_Valve
- removed N2QD1, OxQD1: ~, symbol PID_symbols:Quick_Disconnect
- removed Needle_Valve_N1filling_vent1, Needle_Valve_Oxfilling1: ~, symbol PID_symbols:Needle_Valve
- added Filter5: ~, symbol PID_symbols:Filter
- added N2O_Hose_1, N2O_Hose_2, N2_Hose3: ~, symbol PID_symbols:Hose
- added N2O_Tank_1, N2O_Tank_2, N2_Cylinder2: ~, symbol PID_symbols:Cylinder
Connections:
- new net: N2O_Hose_1., N2O_Tank_1.
- new net: N2O_Hose_2., N2O_Tank_2.
- new net: Filter5., N2_Hose3.
- new net: N2_Cylinder2., N2_Hose3.

Commit message: New year update
Parts:
- renumbered Filter5 to Filter12, N2O_Hose_1 to N2O_Hose_3, N2O_Hose_2 to N2O_Hose_4, N2O_Tank_1 to N2O_Tank_3, N2O_Tank_2 to N2O_Tank_4, N2_Cylinder2 to N2_Cylinder4, N2_Hose3 to N2_Hose6
Connections:
- net at N2O_Hose_4.: now also N2O_Tank_4.
- net at Filter12.: now also N2_Hose6.
- net at N2_Hose6.: now also N2_Cylinder4.; no longer Filter12.
Changed lines of the file:
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@@
 		(dnp no)
 		(fields_autoplaced yes)
-		(property "Reference" "N2O_Tank_1"
+		(property "Reference" "N2O_Tank_3"
 			(at 77.47 93.98 90)
 			(effects
@@
 		(instances
 			(project "P_IDs"
-				(path "/045f1f05-3134-4b6d-91b6-463031104f1e/462f9fab-58b5-4b75-b4d3-2a00576f9247"
-					(reference "N2O_Tank_1")
+				(path "/045f1f05-3134-4b6d-91b6-463031104f1e/d4c68d07-3148-4b28-9ebc-772298248340/d1c23521-1854-4751-80d3-fa4616e29f0e"
+					(reference "N2O_Tank_3")
 					(unit 1)
 				)
@@
 		(dnp no)
 		(fields_autoplaced yes)
-		(property "Reference" "N2O_Hose_2"
+		(property "Reference" "N2O_Hose_4"
 			(at 100.965 119.38 90)
 			(effects
@@
 		)
 		(instances
-			(project ""
-				(path "/045f1f05-3134-4b6d-91b6-463031104f1e/462f9fab-58b5-4b75-b4d3-2a00576f9247"
-					(reference "N2O_Hose_2")
+			(project "P_IDs"
+				(path "/045f1f05-3134-4b6d-91b6-463031104f1e/d4c68d07-3148-4b28-9ebc-772298248340/d1c23521-1854-4751-80d3-fa4616e29f0e"
+					(reference "N2O_Hose_4")
 					(unit 1)
 				)
@@
 		(on_board yes)
 		(dnp no)
-		(property "Reference" "Filter5"
+		(property "Reference" "Filter12"
 			(at 116.205 60.96 0)
 			(effects
@@
 		)
 		(instances
-			(project ""
-				(path "/045f1f05-3134-4b6d-91b6-463031104f1e/462f9fab-58b5-4b75-b4d3-2a00576f9247"
-					(reference "Filter5")
+			(project "P_IDs"
+				(path "/045f1f05-3134-4b6d-91b6-463031104f1e/d4c68d07-3148-4b28-9ebc-772298248340/d1c23521-1854-4751-80d3-fa4616e29f0e"
+					(reference "Filter12")
 					(unit 1)
 				)
@@
 		(dnp no)
 		(fields_autoplaced yes)
-		(property "Reference" "N2O_Tank_2"
+		(property "Reference" "N2O_Tank_4"
 			(at 77.47 113.03 90)
 			(effects
@@
 		(instances
 			(project "P_IDs"
-				(path "/045f1f05-3134-4b6d-91b6-463031104f1e/462f9fab-58b5-4b75-b4d3-2a00576f9247"
-					(reference "N2O_Tank_2")
+				(path "/045f1f05-3134-4b6d-91b6-463031104f1e/d4c68d07-3148-4b28-9ebc-772298248340/d1c23521-1854-4751-80d3-fa4616e29f0e"
+					(reference "N2O_Tank_4")
 					(unit 1)
 				)
@@
 		(dnp no)
 		(fields_autoplaced yes)
-		(property "Reference" "N2O_Hose_1"
+		(property "Reference" "N2O_Hose_3"
 			(at 100.965 100.33 90)
 			(effects
@@
 		)
 		(instances
-			(project ""
-				(path "/045f1f05-3134-4b6d-91b6-463031104f1e/462f9fab-58b5-4b75-b4d3-2a00576f9247"
-					(reference "N2O_Hose_1")
+			(project "P_IDs"
+				(path "/045f1f05-3134-4b6d-91b6-463031104f1e/d4c68d07-3148-4b28-9ebc-772298248340/d1c23521-1854-4751-80d3-fa4616e29f0e"
+					(reference "N2O_Hose_3")
 					(unit 1)
 				)
@@
 		(dnp no)
 		(fields_autoplaced yes)
-		(property "Reference" "N2_Hose3"
+		(property "Reference" "N2_Hose6"
 			(at 100.965 60.96 90)
 			(effects
@@
 		)
 		(instances
-			(project ""
-				(path "/045f1f05-3134-4b6d-91b6-463031104f1e/462f9fab-58b5-4b75-b4d3-2a00576f9247"
-					(reference "N2_Hose3")
+			(project "P_IDs"
+				(path "/045f1f05-3134-4b6d-91b6-463031104f1e/d4c68d07-3148-4b28-9ebc-772298248340/d1c23521-1854-4751-80d3-fa4616e29f0e"
+					(reference "N2_Hose6")
 					(unit 1)
 				)
@@
 		(dnp no)
 		(fields_autoplaced yes)
-		(property "Reference" "N2_Cylinder2"
+		(property "Reference" "N2_Cylinder4"
 			(at 77.47 55.245 90)
 			(effects
@@
 		)
 		(instances
-			(project ""
-				(path "/045f1f05-3134-4b6d-91b6-463031104f1e/462f9fab-58b5-4b75-b4d3-2a00576f9247"
-					(reference "N2_Cylinder2")
-					(unit 1)
-				)
+			(project "P_IDs"
+				(path "/045f1f05-3134-4b6d-91b6-463031104f1e/d4c68d07-3148-4b28-9ebc-772298248340/d1c23521-1854-4751-80d3-fa4616e29f0e"
+					(reference "N2_Cylinder4")
+					(unit 1)
+				)

Commit message: Feed System Work
Connections:
- net at N2O_Hose_4.: now also N2O_Tank_4.
- net at Filter12.: now also N2_Hose6.
- net at N2_Hose6.: now also N2_Cylinder4.; no longer Filter12.
Changed lines of the file:
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@@
 	(title_block
 		(title "Pluto GSS")
-		(date "2025-02-25")
 		(company "ICLR")
 	)

Commit message: j0
Parts:
- renumbered Filter12 to Filter10, N2O_Hose_3 to N2O_Hose_1, N2O_Hose_4 to N2O_Hose_2, N2O_Tank_3 to N2O_Tank_1, N2O_Tank_4 to N2O_Tank_2, N2_Cylinder4 to N2_Cylinder3, N2_Hose6 to N2_Hose3
Connections:
- net at N2O_Hose_2.: now also N2O_Tank_2.
- net at N2_Hose3.: now also N2_Cylinder3.; no longer Filter10.
Changed lines of the file:
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@@
 		(dnp no)
 		(fields_autoplaced yes)
-		(property "Reference" "N2O_Tank_3"
+		(property "Reference" "N2O_Tank_1"
 			(at 77.47 93.98 90)
 			(effects
@@
 			(project "P_IDs"
 				(path "/045f1f05-3134-4b6d-91b6-463031104f1e/d4c68d07-3148-4b28-9ebc-772298248340/d1c23521-1854-4751-80d3-fa4616e29f0e"
-					(reference "N2O_Tank_3")
+					(reference "N2O_Tank_1")
+					(unit 1)
+				)
+			)
+		)
+	)
+	(symbol
+		(lib_id "PID_symbols:Hose")
+		(at 97.155 122.555 270)
+		(unit 1)
+		(exclude_from_sim no)
+		(in_bom yes)
+		(on_board yes)
+		(dnp no)
+		(fields_autoplaced yes)
+		(property "Reference" "N2O_Hose_2"
+			(at 100.965 119.38 90)
+			(effects
+				(font
+					(size 1.27 1.27)
+				)
+			)
+		)
+		(property "Value" "~"
+			(at 100.965 120.65 90)
+			(effects
+				(font
+					(size 1.27 1.27)
+				)
+			)
+		)
+		(property "Footprint" ""
+			(at 97.155 122.555 0)
+			(effects
+				(font
+					(size 1.27 1.27)
+				)
+				(hide yes)
+			)
+		)
+		(property "Datasheet" ""
+			(at 97.155 122.555 0)
+			(effects
+				(font
+					(size 1.27 1.27)
+				)
+				(hide yes)
+			)
+		)
+		(property "Description" ""
+			(at 97.155 122.555 0)
+			(effects
+				(font
+					(size 1.27 1.27)
+				)
+				(hide yes)
+			)
+		)
+		(pin ""
+		)
+		(pin ""
+		)
+		(instances
+			(project "P_IDs"
+				(path "/045f1f05-3134-4b6d-91b6-463031104f1e/d4c68d07-3148-4b28-9ebc-772298248340/d1c23521-1854-4751-80d3-fa4616e29f0e"
+					(reference "N2O_Hose_2")
+					(unit 1)
+				)
+			)
+		)
+	)
+	(symbol
+		(lib_id "PID_symbols:Filter")
+		(at 116.205 64.77 0)
+		(unit 1)
+		(exclude_from_sim no)
+		(in_bom yes)
+		(on_board yes)
+		(dnp no)
+		(property "Reference" "Filter10"
+			(at 116.205 60.96 0)
+			(effects
+				(font
+					(size 1.27 1.27)
+				)
+			)
+		)
+		(property "Value" "~"
+			(at 116.205 62.23 0)
+			(effects
+				(font
+					(size 1.27 1.27)
+				)
+			)
+		)
+		(property "Footprint" ""
+			(at 116.205 64.77 0)
+			(effects
+				(font
+					(size 1.27 1.27)
+				)
+				(hide yes)
+			)
+		)
+		(property "Datasheet" ""
+			(at 116.205 64.77 0)
+			(effects
+				(font
+					(size 1.27 1.27)
+				)
+				(hide yes)
+			)
+		)
+		(property "Description" ""
+			(at 116.205 64.77 0)
+			(effects
+				(font
+					(size 1.27 1.27)
+				)
+				(hide yes)
+			)
+		)
+		(pin ""
+		)
+		(pin ""
+		)
+		(instances
+			(project "P_IDs"
+				(path "/045f1f05-3134-4b6d-91b6-463031104f1e/d4c68d07-3148-4b28-9ebc-772298248340/d1c23521-1854-4751-80d3-fa4616e29f0e"
+					(reference "Filter10")
+					(unit 1)
+				)
+			)
+		)
+	)
+	(symbol
+		(lib_id "PID_symbols:Cylinder")
+		(at 76.835 122.555 90)
+		(unit 1)
+		(exclude_from_sim no)
+		(in_bom yes)
+		(on_board yes)
+		(dnp no)
+		(fields_autoplaced yes)
+		(property "Reference" "N2O_Tank_2"
+			(at 77.47 113.03 90)
+			(effects
+				(font
+					(size 1.27 1.27)
+				)
+			)
+		)
+		(property "Value" "~"
+			(at 77.47 114.3 90)
+			(effects
+				(font
+					(size 1.27 1.27)
+				)
+			)
+		)
+		(property "Footprint" ""
+			(at 76.835 122.555 0)
+			(effects
+				(font
+					(size 1.27 1.27)
+				)
+				(hide yes)
+			)
+		)
+		(property "Datasheet" ""
+			(at 76.835 122.555 0)
+			(effects
+				(font
+					(size 1.27 1.27)
+				)
+				(hide yes)
+			)
+		)
+		(property "Description" ""
+			(at 76.835 122.555 0)
+			(effects
+				(font
+					(size 1.27 1.27)
+				)
+				(hide yes)
+			)
+		)
+		(pin ""
+		)
+		(instances
+			(project "P_IDs"
+				(path "/045f1f05-3134-4b6d-91b6-463031104f1e/d4c68d07-3148-4b28-9ebc-772298248340/d1c23521-1854-4751-80d3-fa4616e29f0e"
+					(reference "N2O_Tank_2")
 					(unit 1)
 				)
@@
 		(lib_name "Hose_1")
 		(lib_id "PID_symbols:Hose")
-		(at 97.155 122.555 270)
-		(unit 1)
-		(exclude_from_sim no)
-		(in_bom yes)
-		(on_board yes)
-		(dnp no)
-		(fields_autoplaced yes)
-		(property "Reference" "N2O_Hose_4"
-			(at 100.965 119.38 90)
-			(effects
-				(font
-					(size 1.27 1.27)
-				)
-			)
-		)
-		(property "Value" "~"
-			(at 100.965 120.65 90)
-			(effects
-				(font
-					(size 1.27 1.27)
-				)
-			)
-		)
-		(property "Footprint" ""
-			(at 97.155 122.555 0)
-			(effects
-				(font
-					(size 1.27 1.27)
-				)
-				(hide yes)
-			)
-		)
-		(property "Datasheet" ""
-			(at 97.155 122.555 0)
-			(effects
-				(font
-					(size 1.27 1.27)
-				)
-				(hide yes)
-			)
-		)
-		(property "Description" ""
-			(at 97.155 122.555 0)
-			(effects
-				(font
-					(size 1.27 1.27)
-				)
-				(hide yes)
-			)
-		)
-		(pin ""
-		)
-		(pin ""
-		)
-		(instances
-			(project "P_IDs"
-				(path "/045f1f05-3134-4b6d-91b6-463031104f1e/d4c68d07-3148-4b28-9ebc-772298248340/d1c23521-1854-4751-80d3-fa4616e29f0e"
-					(reference "N2O_Hose_4")
-					(unit 1)
-				)
-			)
-		)
-	)
-	(symbol
-		(lib_id "PID_symbols:Filter")
-		(at 116.205 64.77 0)
-		(unit 1)
-		(exclude_from_sim no)
-		(in_bom yes)
-		(on_board yes)
-		(dnp no)
-		(property "Reference" "Filter12"
-			(at 116.205 60.96 0)
-			(effects
-				(font
-					(size 1.27 1.27)
-				)
-			)
-		)
-		(property "Value" "~"
-			(at 116.205 62.23 0)
-			(effects
-				(font
-					(size 1.27 1.27)
-				)
-			)
-		)
-		(property "Footprint" ""
-			(at 116.205 64.77 0)
-			(effects
-				(font
-					(size 1.27 1.27)
-				)
-				(hide yes)
-			)
-		)
-		(property "Datasheet" ""
-			(at 116.205 64.77 0)
-			(effects
-				(font
-					(size 1.27 1.27)
-				)
-				(hide yes)
-			)
-		)
-		(property "Description" ""
-			(at 116.205 64.77 0)
-			(effects
-				(font
-					(size 1.27 1.27)
-				)
-				(hide yes)
-			)
-		)
-		(pin ""
-		)
-		(pin ""
-		)
-		(instances
-			(project "P_IDs"
-				(path "/045f1f05-3134-4b6d-91b6-463031104f1e/d4c68d07-3148-4b28-9ebc-772298248340/d1c23521-1854-4751-80d3-fa4616e29f0e"
-					(reference "Filter12")
-					(unit 1)
-				)
-			)
-		)
-	)
-	(symbol
-		(lib_id "PID_symbols:Cylinder")
-		(at 76.835 122.555 90)
-		(unit 1)
-		(exclude_from_sim no)
-		(in_bom yes)
-		(on_board yes)
-		(dnp no)
-		(fields_autoplaced yes)
-		(property "Reference" "N2O_Tank_4"
-			(at 77.47 113.03 90)
-			(effects
-				(font
-					(size 1.27 1.27)
-				)
-			)
-		)
-		(property "Value" "~"
-			(at 77.47 114.3 90)
-			(effects
-				(font
-					(size 1.27 1.27)
-				)
-			)
-		)
-		(property "Footprint" ""
-			(at 76.835 122.555 0)
-			(effects
-				(font
-					(size 1.27 1.27)
-				)
-				(hide yes)
-			)
-		)
-		(property "Datasheet" ""
-			(at 76.835 122.555 0)
-			(effects
-				(font
-					(size 1.27 1.27)
-				)
-				(hide yes)
-			)
-		)
-		(property "Description" ""
-			(at 76.835 122.555 0)
-			(effects
-				(font
-					(size 1.27 1.27)
-				)
-				(hide yes)
-			)
-		)
-		(pin ""
-		)
-		(instances
-			(project "P_IDs"
-				(path "/045f1f05-3134-4b6d-91b6-463031104f1e/d4c68d07-3148-4b28-9ebc-772298248340/d1c23521-1854-4751-80d3-fa4616e29f0e"
-					(reference "N2O_Tank_4")
-					(unit 1)
-				)
-			)
-		)
-	)
-	(symbol
-		(lib_id "PID_symbols:Hose")
 		(at 97.155 104.14 270)
 		(unit 1)
@@
 		(dnp no)
 		(fields_autoplaced yes)
-		(property "Reference" "N2O_Hose_3"
+		(property "Reference" "N2O_Hose_1"
 			(at 100.965 100.33 90)
 			(effects
@@
 			(project "P_IDs"
 				(path "/045f1f05-3134-4b6d-91b6-463031104f1e/d4c68d07-3148-4b28-9ebc-772298248340/d1c23521-1854-4751-80d3-fa4616e29f0e"
-					(reference "N2O_Hose_3")
+					(reference "N2O_Hose_1")
 					(unit 1)
 				)
@@
 		(dnp no)
 		(fields_autoplaced yes)
-		(property "Reference" "N2_Hose6"
+		(property "Reference" "N2_Hose3"
 			(at 100.965 60.96 90)
 			(effects
@@
 			(project "P_IDs"
 				(path "/045f1f05-3134-4b6d-91b6-463031104f1e/d4c68d07-3148-4b28-9ebc-772298248340/d1c23521-1854-4751-80d3-fa4616e29f0e"
-					(reference "N2_Hose6")
+					(reference "N2_Hose3")
 					(unit 1)
 				)
@@
 		(dnp no)
 		(fields_autoplaced yes)
-		(property "Reference" "N2_Cylinder4"
+		(property "Reference" "N2_Cylinder3"
 			(at 77.47 55.245 90)
 			(effects
@@
 			(project "P_IDs"
 				(path "/045f1f05-3134-4b6d-91b6-463031104f1e/d4c68d07-3148-4b28-9ebc-772298248340/d1c23521-1854-4751-80d3-fa4616e29f0e"
-					(reference "N2_Cylinder4")
-					(unit 1)
-				)
+					(reference "N2_Cylinder3")
+					(unit 1)
+				)

Commit message: more silwood stuff
Parts:
- renumbered N2O_Tank_1 to C?, N2O_Tank_2 to C?, N2_Cylinder3 to C?, N2O_Hose_2 to Hose?, N2O_Hose_1 to Hose?, N2_Hose3 to Hose?
Connections:
- net at Hose?.: now also C?. (x2)
Changed lines of the file:
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@@
 		(dnp no)
 		(fields_autoplaced yes)
-		(property "Reference" "N2O_Tank_1"
+		(property "Reference" "C?"
 			(at 77.47 93.98 90)
 			(effects
@@
 					(size 1.27 1.27)
 				)
+				(hide yes)
 			)
 		)
@@
 					(size 1.27 1.27)
 				)
-				(hide yes)
-			)
-		)
-		(pin ""
-		)
-		(instances
-			(project "P_IDs"
-				(path "/045f1f05-3134-4b6d-91b6-463031104f1e/d4c68d07-3148-4b28-9ebc-772298248340/d1c23521-1854-4751-80d3-fa4616e29f0e"
-					(reference "N2O_Tank_1")
+			)
+		)
+		(pin ""
+		)
+		(instances
+			(project "P_IDs"
+				(path "/045f1f05-3134-4b6d-91b6-463031104f1e/d4c68d07-3148-4b28-9ebc-772298248340/d1c23521-1854-4751-80d3-fa4616e29f0e"
+					(reference "C?")
 					(unit 1)
 				)
@@
 		(dnp no)
 		(fields_autoplaced yes)
-		(property "Reference" "N2O_Hose_2"
+		(property "Reference" "Hose?"
 			(at 100.965 119.38 90)
 			(effects
@@
 					(size 1.27 1.27)
 				)
+				(hide yes)
 			)
 		)
@@
 					(size 1.27 1.27)
 				)
-				(hide yes)
-			)
-		)
-		(pin ""
-		)
-		(pin ""
-		)
-		(instances
-			(project "P_IDs"
-				(path "/045f1f05-3134-4b6d-91b6-463031104f1e/d4c68d07-3148-4b28-9ebc-772298248340/d1c23521-1854-4751-80d3-fa4616e29f0e"
-					(reference "N2O_Hose_2")
+			)
+		)
+		(pin ""
+		)
+		(pin ""
+		)
+		(instances
+			(project "P_IDs"
+				(path "/045f1f05-3134-4b6d-91b6-463031104f1e/d4c68d07-3148-4b28-9ebc-772298248340/d1c23521-1854-4751-80d3-fa4616e29f0e"
+					(reference "Hose?")
 					(unit 1)
 				)
@@
 					(size 1.27 1.27)
 				)
+				(hide yes)
 			)
 		)
@@
 					(size 1.27 1.27)
 				)
-				(hide yes)
 			)
 		)
@@
 		(dnp no)
 		(fields_autoplaced yes)
-		(property "Reference" "N2O_Tank_2"
+		(property "Reference" "C?"
 			(at 77.47 113.03 90)
 			(effects
@@
 					(size 1.27 1.27)
 				)
+				(hide yes)
 			)
 		)
@@
 					(size 1.27 1.27)
 				)
-				(hide yes)
-			)
-		)
-		(pin ""
-		)
-		(instances
-			(project "P_IDs"
-				(path "/045f1f05-3134-4b6d-91b6-463031104f1e/d4c68d07-3148-4b28-9ebc-772298248340/d1c23521-1854-4751-80d3-fa4616e29f0e"
-					(reference "N2O_Tank_2")
+			)
+		)
+		(pin ""
+		)
+		(instances
+			(project "P_IDs"
+				(path "/045f1f05-3134-4b6d-91b6-463031104f1e/d4c68d07-3148-4b28-9ebc-772298248340/d1c23521-1854-4751-80d3-fa4616e29f0e"
+					(reference "C?")
 					(unit 1)
 				)
@@
 		(dnp no)
 		(fields_autoplaced yes)
-		(property "Reference" "N2O_Hose_1"
+		(property "Reference" "Hose?"
 			(at 100.965 100.33 90)
 			(effects
@@
 					(size 1.27 1.27)
 				)
+				(hide yes)
 			)
 		)
@@
 					(size 1.27 1.27)
 				)
-				(hide yes)
-			)
-		)
-		(pin ""
-		)
-		(pin ""
-		)
-		(instances
-			(project "P_IDs"
-				(path "/045f1f05-3134-4b6d-91b6-463031104f1e/d4c68d07-3148-4b28-9ebc-772298248340/d1c23521-1854-4751-80d3-fa4616e29f0e"
-					(reference "N2O_Hose_1")
+			)
+		)
+		(pin ""
+		)
+		(pin ""
+		)
+		(instances
+			(project "P_IDs"
+				(path "/045f1f05-3134-4b6d-91b6-463031104f1e/d4c68d07-3148-4b28-9ebc-772298248340/d1c23521-1854-4751-80d3-fa4616e29f0e"
+					(reference "Hose?")
 					(unit 1)
 				)
@@
 		(dnp no)
 		(fields_autoplaced yes)
-		(property "Reference" "N2_Hose3"
+		(property "Reference" "Hose?"
 			(at 100.965 60.96 90)
 			(effects
@@
 					(size 1.27 1.27)
 				)
+				(hide yes)
 			)
 		)
@@
 					(size 1.27 1.27)
 				)
-				(hide yes)
-			)
-		)
-		(pin ""
-		)
-		(pin ""
-		)
-		(instances
-			(project "P_IDs"
-				(path "/045f1f05-3134-4b6d-91b6-463031104f1e/d4c68d07-3148-4b28-9ebc-772298248340/d1c23521-1854-4751-80d3-fa4616e29f0e"
-					(reference "N2_Hose3")
+			)
+		)
+		(pin ""
+		)
+		(pin ""
+		)
+		(instances
+			(project "P_IDs"
+				(path "/045f1f05-3134-4b6d-91b6-463031104f1e/d4c68d07-3148-4b28-9ebc-772298248340/d1c23521-1854-4751-80d3-fa4616e29f0e"
+					(reference "Hose?")
 					(unit 1)
 				)
@@
 		(dnp no)
 		(fields_autoplaced yes)
-		(property "Reference" "N2_Cylinder3"
+		(property "Reference" "C?"
 			(at 77.47 55.245 90)
 			(effects
@@
 					(size 1.27 1.27)
 				)
+				(hide yes)
 			)
 		)
@@
 					(size 1.27 1.27)
 				)
-				(hide yes)
-			)
-		)
-		(pin ""
-		)
-		(instances
-			(project "P_IDs"
-				(path "/045f1f05-3134-4b6d-91b6-463031104f1e/d4c68d07-3148-4b28-9ebc-772298248340/d1c23521-1854-4751-80d3-fa4616e29f0e"
-					(reference "N2_Cylinder3")
-					(unit 1)
-				)
+			)
+		)
+		(pin ""
+		)
+		(instances
+			(project "P_IDs"
+				(path "/045f1f05-3134-4b6d-91b6-463031104f1e/d4c68d07-3148-4b28-9ebc-772298248340/d1c23521-1854-4751-80d3-fa4616e29f0e"
+					(reference "C?")
+					(unit 1)
+				)
