File: Silwood/J-0_N2O_Bottles.kicad_sch (KiCad schematic)
At the start: 19 parts

Commit message: Formatiing
Parts:
- renumbered BV8 to BV2, BV9 to BV3, BV10 to BV4, BV7 to BV?, C4 to C3, C3 to C4, C2 to C5, C5 to C?, CV8 to CV4, CV9 to CV5, CV10 to CV6, CV7 to CV?, Filter1 to Filter?, Hose4 to Hose2, Hose5 to Hose3, Hose6 to Hose4, Hose3 to Hose?, Hose7 to Hose?, SPRV5 to SPRV?
Connections:
- net 3-8 is gone; now on net N2O_FILL: Filter?., SPRV?.
- net at Hose3.: now also CV5.; no longer BV3.
- net at Hose?.: now also CV?.; no longer BV?.
- net N2O_FILL: now reaches SPRV?.
- removed net 1-4: CV4., CV5., CV6., CV?., Hose2., Hose3., Hose4., Hose?., Hose?.
- new net: BV3., Hose3.
- new net: BV?., Hose?.
- new net: CV4., CV5., CV6., CV?., Hose?.
- new net: CV6., Hose4.
- new net: CV4., Hose2.
Other:
- moved on the sheet: Hose?
