File: Silwood/J-0_N2O_Bottles.kicad_sch (KiCad schematic)
At the start: 19 parts

Commit message: update
Parts:
- gave numbers to parts that had none: 12
Connections:
- net at Hose3.: now also CV5.; no longer BV3.
- net at CV5.: now also CV4., CV6., CV?., Hose?.; no longer Hose3.
- net at Hose?.: now also CV?.; no longer BV?.
- new net: BV3., Hose3.
- new net: BV?., Hose?.
Changed lines of the file:
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@@
 		(dnp no)
 		(fields_autoplaced yes)
-		(property "Reference" "Hose?"
+		(property "Reference" "Hose3"
 			(at 127 95.885 90)
 			(effects
@@
 			(project "P_IDs"
 				(path "/045f1f05-3134-4b6d-91b6-463031104f1e/a0b6300e-76e9-4a18-afd6-e2d656b0d8f9/d375e00a-1ce3-4f93-9279-82acf09c7292/4f024983-2e1e-4582-8230-72c25523eed0"
-					(reference "Hose?")
+					(reference "Hose3")
 					(unit 1)
 				)
@@
 		(dnp no)
 		(fields_autoplaced yes)
-		(property "Reference" "BV?"
+		(property "Reference" "BV3"
 			(at 116.84 93.98 0)
 			(effects
@@
 			(project "P_IDs"
 				(path "/045f1f05-3134-4b6d-91b6-463031104f1e/a0b6300e-76e9-4a18-afd6-e2d656b0d8f9/d375e00a-1ce3-4f93-9279-82acf09c7292/4f024983-2e1e-4582-8230-72c25523eed0"
-					(reference "BV?")
+					(reference "BV3")
 					(unit 1)
 				)
@@
 		(on_board yes)
 		(dnp no)
-		(property "Reference" "C?"
+		(property "Reference" "C4"
 			(at 95.25 73.66 90)
 			(effects
@@
 			(project "P_IDs"
 				(path "/045f1f05-3134-4b6d-91b6-463031104f1e/a0b6300e-76e9-4a18-afd6-e2d656b0d8f9/d375e00a-1ce3-4f93-9279-82acf09c7292/4f024983-2e1e-4582-8230-72c25523eed0"
-					(reference "C?")
+					(reference "C4")
 					(unit 1)
 				)
@@
 		(dnp no)
 		(fields_autoplaced yes)
-		(property "Reference" "CV?"
+		(property "Reference" "CV6"
 			(at 143.383 113.03 0)
 			(effects
@@
 			(project "P_IDs"
 				(path "/045f1f05-3134-4b6d-91b6-463031104f1e/a0b6300e-76e9-4a18-afd6-e2d656b0d8f9/d375e00a-1ce3-4f93-9279-82acf09c7292/4f024983-2e1e-4582-8230-72c25523eed0"
-					(reference "CV?")
+					(reference "CV6")
 					(unit 1)
 				)
@@
 		(dnp no)
 		(fields_autoplaced yes)
-		(property "Reference" "CV?"
+		(property "Reference" "CV5"
 			(at 143.383 93.98 0)
 			(effects
@@
 			(project "P_IDs"
 				(path "/045f1f05-3134-4b6d-91b6-463031104f1e/a0b6300e-76e9-4a18-afd6-e2d656b0d8f9/d375e00a-1ce3-4f93-9279-82acf09c7292/4f024983-2e1e-4582-8230-72c25523eed0"
-					(reference "CV?")
+					(reference "CV5")
 					(unit 1)
 				)
@@
 		(dnp no)
 		(fields_autoplaced yes)
-		(property "Reference" "BV?"
+		(property "Reference" "BV2"
 			(at 116.84 74.93 0)
 			(effects
@@
 			(project "P_IDs"
 				(path "/045f1f05-3134-4b6d-91b6-463031104f1e/a0b6300e-76e9-4a18-afd6-e2d656b0d8f9/d375e00a-1ce3-4f93-9279-82acf09c7292/4f024983-2e1e-4582-8230-72c25523eed0"
-					(reference "BV?")
+					(reference "BV2")
 					(unit 1)
 				)
@@
 		(dnp no)
 		(fields_autoplaced yes)
-		(property "Reference" "CV?"
+		(property "Reference" "CV4"
 			(at 143.383 74.93 0)
 			(effects
@@
 			(project "P_IDs"
 				(path "/045f1f05-3134-4b6d-91b6-463031104f1e/a0b6300e-76e9-4a18-afd6-e2d656b0d8f9/d375e00a-1ce3-4f93-9279-82acf09c7292/4f024983-2e1e-4582-8230-72c25523eed0"
-					(reference "CV?")
+					(reference "CV4")
 					(unit 1)
 				)
@@
 		(dnp no)
 		(fields_autoplaced yes)
-		(property "Reference" "BV?"
+		(property "Reference" "BV4"
 			(at 116.84 113.03 0)
 			(effects
@@
 			(project "P_IDs"
 				(path "/045f1f05-3134-4b6d-91b6-463031104f1e/a0b6300e-76e9-4a18-afd6-e2d656b0d8f9/d375e00a-1ce3-4f93-9279-82acf09c7292/4f024983-2e1e-4582-8230-72c25523eed0"
-					(reference "BV?")
+					(reference "BV4")
 					(unit 1)
 				)
@@
 		(dnp no)
 		(fields_autoplaced yes)
-		(property "Reference" "Hose?"
+		(property "Reference" "Hose4"
 			(at 127 114.935 90)
 			(effects
@@
 			(project "P_IDs"
 				(path "/045f1f05-3134-4b6d-91b6-463031104f1e/a0b6300e-76e9-4a18-afd6-e2d656b0d8f9/d375e00a-1ce3-4f93-9279-82acf09c7292/4f024983-2e1e-4582-8230-72c25523eed0"
-					(reference "Hose?")
+					(reference "Hose4")
 					(unit 1)
 				)
@@
 		(dnp no)
 		(fields_autoplaced yes)
-		(property "Reference" "Hose?"
+		(property "Reference" "Hose2"
 			(at 127 76.835 90)
 			(effects
@@
 			(project "P_IDs"
 				(path "/045f1f05-3134-4b6d-91b6-463031104f1e/a0b6300e-76e9-4a18-afd6-e2d656b0d8f9/d375e00a-1ce3-4f93-9279-82acf09c7292/4f024983-2e1e-4582-8230-72c25523eed0"
-					(reference "Hose?")
+					(reference "Hose2")
 					(unit 1)
 				)
@@
 		(on_board yes)
 		(dnp no)
-		(property "Reference" "C?"
+		(property "Reference" "C3"
 			(at 95.25 92.71 90)
 			(effects
@@
 			(project "P_IDs"
 				(path "/045f1f05-3134-4b6d-91b6-463031104f1e/a0b6300e-76e9-4a18-afd6-e2d656b0d8f9/d375e00a-1ce3-4f93-9279-82acf09c7292/4f024983-2e1e-4582-8230-72c25523eed0"
-					(reference "C?")
+					(reference "C3")
 					(unit 1)
 				)
@@
 		(on_board yes)
 		(dnp no)
-		(property "Reference" "C?"
+		(property "Reference" "C5"
 			(at 95.25 52.705 90)
 			(effects
@@
 			(project "P_IDs"
 				(path "/045f1f05-3134-4b6d-91b6-463031104f1e/a0b6300e-76e9-4a18-afd6-e2d656b0d8f9/d375e00a-1ce3-4f93-9279-82acf09c7292/4f024983-2e1e-4582-8230-72c25523eed0"
-					(reference "C?")
-					(unit 1)
-				)
+					(reference "C5")
+					(unit 1)
+				)

Commit message: j0
Parts:
- gave numbers to parts that had none: 7
- renumbered BV4 to BV10, BV2 to BV8, BV3 to BV9, C5 to C2, C4 to C3, C3 to C4, CV6 to CV10, CV4 to CV8, CV5 to CV9, Hose3 to Hose4, Hose4 to Hose5
Connections:
- net N2O_FILL is gone; now on net 3-8: Filter1., SPRV4.
- net at BV9.: now also C4.; no longer Hose4.
- net 1-4: now reaches CV9., Hose4.
- net 1-4: now also CV10., CV7., CV8., Hose1., Hose2., Hose3., Hose5.
- net at BV7.: now also C2.; no longer Hose1.
- net 3-8: now reaches Filter1.
- net 3-8: no longer Hose3.
- net at BV10.: now also C5.; no longer Hose5.
- new net: BV9., Hose4.
- new net: BV7., Hose1.
- new net: Filter1., Hose3.
- new net: BV10., Hose5.
Other:
- moved on the sheet: Hose3

Commit message: more silwood stuff
Parts:
- renumbered Hose1 to Hose3, Hose2 to Hose4, Hose4 to Hose5, Hose5 to Hose6, Hose3 to Hose7, SPRV4 to SPRV5
Connections:
- net at BV9.: now also C4.; no longer Hose5.
- net at BV7.: now also C2.; no longer Hose3.
- net at BV10.: now also C5.; no longer Hose6.
- new net: BV9., Hose5.
- new net: BV7., Hose3.
- new net: Filter1., Hose7.
- new net: BV10., Hose6.

Commit message: silwood upgrade
Parts:
- removed BV10, BV7, BV8, BV9: ~, symbol PID_symbols:Ball_Valve
- removed C3, C4, C5: ~, symbol PID_symbols:Cylinder
- removed CV10, CV8, CV9: ~, symbol PID_symbols:Check_Valve
- removed Hose4, Hose5, Hose6: ~, symbol PID_symbols:Hose
- added MB_V16: ~, symbol PID_symbols:MBallValve
Connections:
- net 1-4: no longer Hose3.
- net 3-8: now also Hose7.; no longer Filter1.
- net at Hose3.: now also MB_V16.
- net at C2.: now also MB_V16.
- net at Filter1.: now also CV7.; no longer Hose7.
- new net: Filter1., Hose3.
Other:
- moved on the sheet: C2, CV7, Filter1, Hose3, Hose7

Commit message: big silwood update
Parts:
- removed Hose7: ~, symbol PID_symbols:Hose
- removed MB_V16: ~, symbol PID_symbols:MBallValve
- added BV8: ~, symbol PID_symbols:Ball_Valve
- added Burst_Disc19: ~, symbol PID_symbols:Burst_Disc
- added C3, C4: ~, symbol PID_symbols:Cylinder
- added CF4: ~, symbol PID_symbols:Coriolis_Flow
- added CV18, CV8, CV9: ~, symbol PID_symbols:Check_Valve
- added DP4: ~, symbol PID_symbols:DP_Sensor
- added Dome4: ~, symbol PID_symbols:Dome_Reg
- added Filter15, Filter16, Filter18: ~, symbol PID_symbols:Filter
- added Hose31, Hose32: ~, symbol PID_symbols:Hose
- added MB_V7, MB_V8: ~, symbol PID_symbols:MBallValve
- added Manual_Pressure_Gauge20, Manual_Pressure_Gauge22: ~, symbol PID_symbols:Manual_Pressure_Gauge
- added PT84: ~, symbol PID_symbols:Pressure_Transducer
- added Pmatic_B_Valve12: ~, symbol PID_symbols:Pneumatic_Rotary_Ball_Valve
- added QD25: ~, symbol PID_symbols:Quick_Disconnect
- added SPRV29: ~, symbol PID_symbols:SPRV
- added Servo_Reg18, Servo_Reg4: ~, symbol PID_symbols:Pressure_Regulator
- added TC10: ~, symbol PID_symbols:Thermocouple
- added nC_Sol9: ~, symbol PID_symbols:Normally_Closed_Solenoid
- added nO_Sol27: ~, symbol PID_symbols:Normally Open Solenoid
Connections:
- net 1-4: now also Filter1., CV8., CV9., Filter15., Filter16., MB_V7.
- net 3-8: now also CV7., CV8., CV9., MB_V7., Manual_Pressure_Gauge20.
- net at Hose3.: now also C2.; no longer Filter1.
- new net: Filter1., Hose3.
- new net: Filter15., Hose31.
- new net: Filter16., Hose32.
- new net: C3., Hose31.
- new net: C4., Hose32.
Other:
- note added: "(4): Optional Numbering if multiple sensors in same local feed line Smaller number is upstream."
- note added: "1 INCH"
- note added: "1-2 INCH"
- note added: "1-4 INCH"
- note added: "1-8 INCH"
- note added: "1: Macro location of component KEY: O: Oxidiser panel F: Fuel panel N: Outer N2 System I: Igniter PP: Pressure Panel OB: Oxidiser outside bottles"
- note added: "2: Component Type KEY: Bv: Ball Valve (servo actuated) Mbv: Manual Ball Valve Mf: Massflow control Ball Valve Pn: Pneumatic Actuated Valves Sol: Solenoid Valves PT: Pressure Transducer Tc: Thermocouple Reg: Pressure Regulator CFM: Coriolis Flow Meter PG: Pressure Gauge Tk: Tank Prv: Pressure Relief Valve BD: Burst Disk DP: Differential Pressure Sensor"
- note added: "3-4 INCH"
- note added: "3-8 INCH"
- note added: "3: Local Location feed system of Component KEY: Ref: Dome reference pressure system M: Main run line V: Venting Line T: Tank Pressurisation Line N: Nitrogen High Pressure Source Line O: Oxidiser Source Line F: Fill Line D: Drain Line P: Purge Line LP: Low Pressure Impulse Air Line"
- note added: "Burst Disk"
- note added: "Check-Valve"
- note added: "Component Naming Scheme: 1_2_3(4)"
- note added: "Coriolis Flow Meter"
- note added: "Deployment Line 1: 'D1' Run Valves on N2 lines to tanks, and main lines."
- note added: "Deployment Line 2: 'D2' All venting valves."
- note added: "Differential Pressure Transducer"
- note added: "Direct Connection"
- note added: "Dome-Loaded Regulator"
- note added: "Filter"
- note added: "Low Pressure Pneumatics"
- note added: "Manual Ball Valve"
- note added: "Normally Closed Solenoid"
- note added: "Normally Open Solenoid"
- note added: "Pneumatic Actuated Valve, NO/NC (Normally Open/Closed)"
- note added: "Pressure Gauge"
- note added: "Pressure Regulator"
- note added: "Pressure Relief Valve"
- note added: "Pressure Transducer"
- note added: "Quick-Disconnect"
- note added: "Servo Ball Valve"
- note added: "Servo-Actuated Pressure Regulator"
- note added: "Thermocouple"
- note added: "Torch Igniter High Pressure Line"
- note added: "Torch Igniter Pneumatics Line"
- moved on the sheet: C2, CV7, Filter1, Hose3
