File: Silwood/J0.kicad_sch (KiCad schematic)
At the start: 21 parts

Commit message: Formatiing
Parts:
- removed Engine1: ~, symbol PID_symbols:Engine
- removed Hose1, Hose2: ~, symbol PID_symbols:Hose
- removed PT1, PT2, PT3, PT4: ~, symbol PID_symbols:Pressure_Transducer
- removed Pmatic_B_Valve1, Pmatic_B_Valve10: ~, symbol PID_symbols:Pneumatic_Rotary_Ball_Valve
- removed TC1, TC2: ~, symbol PID_symbols:Thermocouple
- removed U10, U11, U12, U13, U14, U5, U6, U7, U8, U9: ~, symbol PID_symbols:stop
Connections:
- no-connect marks 3 -> 0
Other:
- sheet Fuel Bay ports: added none; removed Fuel_Delivery, Fuel_External_Vent, N2_HP, N2_LP, N2_Purge_Fuel
- sheet N2O Bay ports: added none; removed N20_Delivery, N2_Purge_Ox, Ox_External_Vent
- note removed: "1 INCH"
- note removed: "1-2 INCH"
- note removed: "1-4 INCH"
- note removed: "1-8 INCH"
- note removed: "3-4 INCH"
- note removed: "3-8 INCH"
- note removed: "Container Wall"
- note removed: "Direct Connection"
- note removed: "Low Pressure Pneumatics"
- note removed: "Torch Igniter High Pressure Line"
- note removed: "Torch Igniter Pneumatics Line"
