File: Silwood/J0_Fuel.kicad_sch (KiCad schematic)
At the start: 39 parts

Commit message: Formatiing
Parts:
- removed BV2: ~, symbol PID_symbols:Ball_Valve
- removed Burst_Disc4: ~, symbol PID_symbols:Burst_Disc
- removed CF2: ~, symbol PID_symbols:Coriolis_Flow
- removed CV18, CV19, CV20: ~, symbol PID_symbols:Check_Valve
- removed DP2: ~, symbol PID_symbols:DP_Sensor
- removed Dome2: ~, symbol PID_symbols:Dome_Reg
- removed MB_V6: ~, symbol PID_symbols:MBallValve
- removed Manual_Pressure_Gauge7: ~, symbol PID_symbols:Manual_Pressure_Gauge
- removed PT29, PT30, PT31, PT32, PT33: ~, symbol PID_symbols:Pressure_Transducer
- removed Pmatic_B_Valve3, Pmatic_B_Valve4, Pmatic_B_Valve8, Pmatic_B_Valve9: ~, symbol PID_symbols:Pneumatic_Rotary_Ball_Valve
- removed QD5: ~, symbol PID_symbols:Quick_Disconnect
- removed SPRV8, SPRV9: ~, symbol PID_symbols:SPRV
- removed Servo_Reg2, Servo_Reg5: ~, symbol PID_symbols:Pressure_Regulator
- removed T4: ~, symbol PID_symbols:Tank
- removed TC6, TC7, TC8: ~, symbol PID_symbols:Thermocouple
- removed U27, U28, U29, U30, U31, U32, U33, U34, U35, U36: ~, symbol PID_symbols:stop
- removed nO_Sol6: ~, symbol PID_symbols:Normally Open Solenoid
Connections:
- no-connect marks 2 -> 0
Other:
- note removed: "Manifold"
