File: Silwood/J0_Fuel.kicad_sch (KiCad schematic)
At the start: 0 parts

Commit message: j0
Parts:
- added BV17, Throttle_2: ~, symbol PID_symbols:Ball_Valve
- added Burst_Disc4: ~, symbol PID_symbols:Burst_Disc
- added CV18, CV19, CV20: ~, symbol PID_symbols:Check_Valve
- added Coriolis_2: ~, symbol PID_symbols:Coriolis_Flow
- added DP2: ~, symbol PID_symbols:DP_Sensor
- added Dome2: ~, symbol PID_symbols:Dome_Reg
- added PBV2, Pmatic_B_Valve7, Pmatic_B_Valve8, Pmatic_B_Valve9: ~, symbol PID_symbols:Pneumatic_Rotary_Ball_Valve
- added PT20: ~, symbol PID_symbols:Pressure_Transducer
- added Reg5, Servo_Reg2: ~, symbol PID_symbols:Pressure_Regulator
- added SPRV7: ~, symbol PID_symbols:SPRV
- added T4: ~, symbol PID_symbols:Tank
- added U18, U19, U20, U21: ~, symbol PID_symbols:stop
Connections:
- new net: Dome2., Reg5., Servo_Reg2.
- new net: BV17., Burst_Disc4., PBV2., SPRV7., U18.
- new net 1-2: U18.
- new net 1-4: BV17., DP2., Dome2., PBV2., PT20., Servo_Reg2., U19., U20., U21.
- new net 3-4: CV20., Pmatic_B_Valve9., T4., Throttle_2., U21.
- new net 3-8: Burst_Disc4., CV18., CV19., CV20., Dome2., Pmatic_B_Valve7., Pmatic_B_Valve8., Reg5., SPRV7., T4., U19., U20.
- new net LP: PBV2., Pmatic_B_Valve7., Pmatic_B_Valve8., Pmatic_B_Valve9.
- no-connect marks 0 -> 2
Other:
- note added: "Manifold"

Commit message: more silwood stuff
Parts:
- removed BV17, Throttle_2: ~, symbol PID_symbols:Ball_Valve
- removed Coriolis_2: ~, symbol PID_symbols:Coriolis_Flow
- removed PBV2, Pmatic_B_Valve7: ~, symbol PID_symbols:Pneumatic_Rotary_Ball_Valve
- removed PT20: ~, symbol PID_symbols:Pressure_Transducer
- removed Reg5: ~, symbol PID_symbols:Pressure_Regulator
- removed SPRV7: ~, symbol PID_symbols:SPRV
- removed U18, U19, U20, U21: ~, symbol PID_symbols:stop
- added BV2: ~, symbol PID_symbols:Ball_Valve
- added CF2: ~, symbol PID_symbols:Coriolis_Flow
- added MB_V6: ~, symbol PID_symbols:MBallValve
- added Manual_Pressure_Gauge7: ~, symbol PID_symbols:Manual_Pressure_Gauge
- added PT29, PT30, PT31, PT32, PT33: ~, symbol PID_symbols:Pressure_Transducer
- added Pmatic_B_Valve3, Pmatic_B_Valve4: ~, symbol PID_symbols:Pneumatic_Rotary_Ball_Valve
- added QD5: ~, symbol PID_symbols:Quick_Disconnect
- added SPRV8, SPRV9: ~, symbol PID_symbols:SPRV
- added Servo_Reg5: ~, symbol PID_symbols:Pressure_Regulator
- added TC6, TC7, TC8: ~, symbol PID_symbols:Thermocouple
- added U27, U28, U29, U30, U31, U32, U33, U34, U35, U36: ~, symbol PID_symbols:stop
- added nO_Sol6: ~, symbol PID_symbols:Normally Open Solenoid
Connections:
- net LP is gone; now on net N2_LP: Pmatic_B_Valve8., Pmatic_B_Valve9.
- net 1-2: now also Pmatic_B_Valve4., SPRV8., U27.
- net 1-4: now also MB_V6., Manual_Pressure_Gauge7., PT29., PT30., PT31., PT32., PT33., SPRV9., TC6., TC7., TC8., U27., U28., U29., U30., U31., U33., U34., U35., U36., nO_Sol6.
- net 3-4: now also Pmatic_B_Valve8., BV2., CF2., U31., U32., U33., U35., U36.; no longer CV20., Pmatic_B_Valve9.
- net 3-8: now also Pmatic_B_Valve9., Pmatic_B_Valve3., Pmatic_B_Valve4., SPRV8., Servo_Reg5., U28., U29., U30., U32., U34.; no longer Pmatic_B_Valve8.
- net N2_HP: now reaches Servo_Reg2.
- net N2_HP: now also Pmatic_B_Valve3., Servo_Reg5.; no longer Dome2.
- net N2_LP: now reaches Pmatic_B_Valve9.
- net N2_LP: now also Pmatic_B_Valve3., Pmatic_B_Valve4.
- new net D: CV18., QD5.
- new net Fuel_Fill: QD5.
- new net Fuel_Fill_Vent: MB_V6.

Commit message: silwood upgrade
Parts:
- removed CV18: ~, symbol PID_symbols:Check_Valve
- added MB_V15, MB_V17, MB_V18: ~, symbol PID_symbols:MBallValve
- added Manual_Pressure_Gauge14, Manual_Pressure_Gauge15: ~, symbol PID_symbols:Manual_Pressure_Gauge
- added PT82: ~, symbol PID_symbols:Pressure_Transducer
- added U19, U69, U70, U9: ~, symbol PID_symbols:stop
Connections:
- net 1-4: now also MB_V17., PT82., U19., U9.
- net 3-4: now also MB_V18., U69., U70., U9.
- net 3-8: now also MB_V15., Manual_Pressure_Gauge15., U19.
- net D: now also MB_V15., Manual_Pressure_Gauge14.
- new net: MB_V17., U70.
Other:
- moved on the sheet: BV2, PT32, TC7

Commit message: big silwood update
Parts:
- removed U69: ~, symbol PID_symbols:stop
- added BV10: ~, symbol PID_symbols:Ball_Valve
- added Burst_Disc21: ~, symbol PID_symbols:Burst_Disc
- added CF6: ~, symbol PID_symbols:Coriolis_Flow
- added CV23: ~, symbol PID_symbols:Check_Valve
- added DP6: ~, symbol PID_symbols:DP_Sensor
- added Dome6: ~, symbol PID_symbols:Dome_Reg
- added Filter20: ~, symbol PID_symbols:Filter
- added MB_V10: ~, symbol PID_symbols:MBallValve
- added Manual_Pressure_Gauge24: ~, symbol PID_symbols:Manual_Pressure_Gauge
- added PT86: ~, symbol PID_symbols:Pressure_Transducer
- added Pmatic_B_Valve14: ~, symbol PID_symbols:Pneumatic_Rotary_Ball_Valve
- added QD27: ~, symbol PID_symbols:Quick_Disconnect
- added SPRV31: ~, symbol PID_symbols:SPRV
- added Servo_Reg20, Servo_Reg6: ~, symbol PID_symbols:Pressure_Regulator
- added TC12: ~, symbol PID_symbols:Thermocouple
- added nC_Sol11: ~, symbol PID_symbols:Normally_Closed_Solenoid
- added nO_Sol29: ~, symbol PID_symbols:Normally Open Solenoid
- BV2, Pmatic_B_Valve3, Pmatic_B_Valve8, Pmatic_B_Valve9, Servo_Reg2: value ~ -> D1
- Pmatic_B_Valve4, nO_Sol6: value ~ -> D2
Connections:
- net 1-4: now also U70.
Other:
- note added: "(4): Optional Numbering if multiple sensors in same local feed line Smaller number is upstream."
- note added: "1 INCH"
- note added: "1-2 INCH"
- note added: "1-4 INCH"
- note added: "1-8 INCH"
- note added: "1: Macro location of component KEY: O: Oxidiser panel F: Fuel panel N: Outer N2 System I: Igniter PP: Pressure Panel OB: Oxidiser outside bottles"
- note added: "2: Component Type KEY: Bv: Ball Valve (servo actuated) Mbv: Manual Ball Valve Mf: Massflow control Ball Valve Pn: Pneumatic Actuated Valves Sol: Solenoid Valves PT: Pressure Transducer Tc: Thermocouple Reg: Pressure Regulator CFM: Coriolis Flow Meter PG: Pressure Gauge Tk: Tank Prv: Pressure Relief Valve BD: Burst Disk DP: Differential Pressure Sensor"
- note added: "3-4 INCH"
- note added: "3-8 INCH"
- note added: "3: Local Location feed system of Component KEY: Ref: Dome reference pressure system M: Main run line V: Venting Line T: Tank Pressurisation Line N: Nitrogen High Pressure Source Line O: Oxidiser Source Line F: Fill Line D: Drain Line P: Purge Line LP: Low Pressure Impulse Air Line"
- note added: "Burst Disk"
- note added: "Check-Valve"
- note added: "Component Naming Scheme: 1_2_3(4)"
- note added: "Coriolis Flow Meter"
- note added: "Deployment Line 1: 'D1' Run Valves on N2 lines to tanks, and main lines."
- note added: "Deployment Line 2: 'D2' All venting valves."
- note added: "Differential Pressure Transducer"
- note added: "Direct Connection"
- note added: "Dome-Loaded Regulator"
- note added: "Filter"
- note added: "Low Pressure Pneumatics"
- note added: "Manual Ball Valve"
- note added: "Normally Closed Solenoid"
- note added: "Normally Open Solenoid"
- note added: "Pneumatic Actuated Valve, NO/NC (Normally Open/Closed)"
- note added: "Pressure Gauge"
- note added: "Pressure Regulator"
- note added: "Pressure Relief Valve"
- note added: "Pressure Transducer"
- note added: "Quick-Disconnect"
- note added: "Servo Ball Valve"
- note added: "Servo-Actuated Pressure Regulator"
- note added: "Thermocouple"
- note added: "Torch Igniter High Pressure Line"
- note added: "Torch Igniter Pneumatics Line"
- moved on the sheet: QD5, T4B

Commit message: update
Parts:
- renumbered T4 to TANK_
Connections:
- net 1-2: now also Burst_Disc4., CV19., Dome2., Manual_Pressure_Gauge15., Pmatic_B_Valve3., TANK_., U28., U29., U30.
- net 3-8: no longer Burst_Disc4., CV19., Dome2., Manual_Pressure_Gauge15., Pmatic_B_Valve3., Pmatic_B_Valve4., SPRV8., TANK_., U28., U29., U30.
Other:
- note added: "3: Local Location feed line of Component KEY: Ref: Dome reference pressure system M: Main run line V: Venting Line T: Tank Pressurisation Line N: Nitrogen High Pressure Source Line O: Oxidiser Source Line F: Fill Line D: Drain Line P: Purge Line LP: Low Pressure Impulse Air Line"
- note added: "TANK"
- note removed: "3: Local Location feed system of Component KEY: Ref: Dome reference pressure system M: Main run line V: Venting Line T: Tank Pressurisation Line N: Nitrogen High Pressure Source Line O: Oxidiser Source Line F: Fill Line D: Drain Line P: Purge Line LP: Low Pressure Impulse Air Line"
Changed lines of the file:
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@@
 		)
 	)
-	(text "3: Local Location feed system of Component\n\nKEY:\nRef: Dome reference pressure system\nM: Main run line\nV: Venting Line\nT: Tank Pressurisation Line\nN: Nitrogen High Pressure Source Line\nO: Oxidiser Source Line\nF: Fill Line\nD: Drain Line\nP: Purge Line\nLP: Low Pressure Impulse Air Line"
+	(text "3: Local Location feed line of Component\n\nKEY:\nRef: Dome reference pressure system\nM: Main run line\nV: Venting Line\nT: Tank Pressurisation Line\nN: Nitrogen High Pressure Source Line\nO: Oxidiser Source Line\nF: Fill Line\nD: Drain Line\nP: Purge Line\nLP: Low Pressure Impulse Air Line"
 		(exclude_from_sim no)
 		(at 334.01 111.76 0)
@@
 		)
 	)
+	(text "TANK"
+		(exclude_from_sim no)
+		(at 200.025 140.335 0)
+		(effects
+			(font
+				(size 1.27 1.27)
+			)
+			(justify left)
+		)
+	)
 	(text "Quick-Disconnect"
 		(exclude_from_sim no)
@@
 		)
 	)
-	(global_label "3-8"
+	(global_label "1-2"
 		(shape input)
 		(at 127 125.73 180)
@@
 		)
 	)
-	(global_label "3-8"
+	(global_label "1-2"
 		(shape input)
 		(at 84.455 125.73 0)
@@
 		)
 	)
-	(global_label "3-8"
+	(global_label "1-2"
 		(shape input)
 		(at 146.685 155.575 270)
@@
 		(on_board yes)
 		(dnp no)
-		(property "Reference" "T4"
-			(at 200.66 140.335 0)
+		(property "Reference" "TANK_"
+			(at 199.39 140.335 0)
 			(effects
 				(font
@@
 				)
 				(justify left)
+				(hide yes)
 			)
 		)
@@
 			(project "P_IDs"
 				(path "/045f1f05-3134-4b6d-91b6-463031104f1e/a0b6300e-76e9-4a18-afd6-e2d656b0d8f9/d375e00a-1ce3-4f93-9279-82acf09c7292/2a11f1f0-1db0-4a3b-bc44-4a76b750bc36"
-					(reference "T4")
+					(reference "TANK_")
 					(unit 2)
 				)
