File: Silwood/J0_N2.kicad_sch (KiCad schematic)
At the start: 17 parts

Commit message: Formatiing
Parts:
- removed U37: ~, symbol PID_symbols:stop
- renumbered C6 to C10, C7 to C11, C8 to C12, C9 to C13, CV22 to CV12, CV23 to CV13, CV24 to CV14, CV25 to CV15, Hose15 to Hose10, Hose16 to Hose11, Hose17 to Hose12, Hose18 to Hose13, MB_V8 to MB_V11, MB_V9 to MB_V12, MB_V10 to MB_V13, MB_V7 to MB_V5
Connections:
- net 1-4 is gone; now on net N2_HP: CV12., CV13., CV14., CV15.
- net at Hose12.: now also MB_V12.; no longer CV14.
- net at Hose11.: now also CV13.; no longer MB_V11.
- net N2_HP: now reaches CV13.
- net N2_HP: no longer Hose11.
- net at Hose13.: now also MB_V13.; no longer CV15.
- net at MB_V13.: now also C13.; no longer Hose13.
- new net: CV14., Hose12.
- new net: Hose11., MB_V11.
- new net: CV15., Hose13.
