File: Silwood/J0_N2O.kicad_sch (KiCad schematic)
At the start: 12 parts

Commit message: update
Parts:
- gave numbers to parts that had none: 6
Connections:
- net at CV?.: now also T?.; no longer Dome4.
- net at T?.: now also Coriolis_?., Pmatic_B_Valve?.; no longer CV?.
- net at PT9.: now also Dome4., Servo_Reg4.
- net at CV22.: now also Throttle_?.; no longer Pmatic_B_Valve3.
- net at Throttle_?.: now also Pmatic_B_Valve?.; no longer CV22.
- new net: CV?., Dome4.
- new net: CV22., Pmatic_B_Valve3.
- new net: Pmatic_B_Valve3., Reg4.
Changed lines of the file:
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@@
 		(dnp no)
 		(fields_autoplaced yes)
-		(property "Reference" "PT?"
+		(property "Reference" "PT9"
 			(at 79.375 62.865 0)
 			(effects
@@
 			(project "P_IDs"
 				(path "/045f1f05-3134-4b6d-91b6-463031104f1e/a0b6300e-76e9-4a18-afd6-e2d656b0d8f9/d375e00a-1ce3-4f93-9279-82acf09c7292/343346ed-3011-4de4-9739-8cfc7e2486c8"
-					(reference "PT?")
+					(reference "PT9")
 					(unit 1)
 				)
@@
 		(dnp no)
 		(fields_autoplaced yes)
-		(property "Reference" "CV?"
+		(property "Reference" "CV22"
 			(at 250.19 122.4279 90)
 			(effects
@@
 		)
 		(instances
-			(project "P_IDs"
-				(path "/045f1f05-3134-4b6d-91b6-463031104f1e/a0b6300e-76e9-4a18-afd6-e2d656b0d8f9/d375e00a-1ce3-4f93-9279-82acf09c7292/343346ed-3011-4de4-9739-8cfc7e2486c8"
-					(reference "CV?")
+			(project ""
+				(path "/045f1f05-3134-4b6d-91b6-463031104f1e/a0b6300e-76e9-4a18-afd6-e2d656b0d8f9/d375e00a-1ce3-4f93-9279-82acf09c7292/343346ed-3011-4de4-9739-8cfc7e2486c8"
+					(reference "CV22")
 					(unit 1)
 				)
@@
 		(dnp no)
 		(fields_autoplaced yes)
-		(property "Reference" "Pmatic_B_Valve?"
+		(property "Reference" "Pmatic_B_Valve3"
 			(at 232.41 96.6468 0)
 			(effects
@@
 			(project "P_IDs"
 				(path "/045f1f05-3134-4b6d-91b6-463031104f1e/a0b6300e-76e9-4a18-afd6-e2d656b0d8f9/d375e00a-1ce3-4f93-9279-82acf09c7292/343346ed-3011-4de4-9739-8cfc7e2486c8"
-					(reference "Pmatic_B_Valve?")
+					(reference "Pmatic_B_Valve3")
 					(unit 1)
 				)
@@
 		(on_board yes)
 		(dnp no)
-		(property "Reference" "Reg?"
+		(property "Reference" "Reg4"
 			(at 194.31 104.14 0)
 			(effects
@@
 			(project "P_IDs"
 				(path "/045f1f05-3134-4b6d-91b6-463031104f1e/a0b6300e-76e9-4a18-afd6-e2d656b0d8f9/d375e00a-1ce3-4f93-9279-82acf09c7292/343346ed-3011-4de4-9739-8cfc7e2486c8"
-					(reference "Reg?")
+					(reference "Reg4")
 					(unit 1)
 				)
@@
 		(dnp no)
 		(fields_autoplaced yes)
-		(property "Reference" "Servo_Reg?"
+		(property "Reference" "Servo_Reg4"
 			(at 59.7525 52.705 0)
 			(effects
@@
 			(project "P_IDs"
 				(path "/045f1f05-3134-4b6d-91b6-463031104f1e/a0b6300e-76e9-4a18-afd6-e2d656b0d8f9/d375e00a-1ce3-4f93-9279-82acf09c7292/343346ed-3011-4de4-9739-8cfc7e2486c8"
-					(reference "Servo_Reg?")
+					(reference "Servo_Reg4")
 					(unit 2)
 				)
@@
 		(dnp no)
 		(fields_autoplaced yes)
-		(property "Reference" "Dome?"
+		(property "Reference" "Dome4"
 			(at 71.8004 97.155 0)
 			(effects
@@
 			(project "P_IDs"
 				(path "/045f1f05-3134-4b6d-91b6-463031104f1e/a0b6300e-76e9-4a18-afd6-e2d656b0d8f9/d375e00a-1ce3-4f93-9279-82acf09c7292/343346ed-3011-4de4-9739-8cfc7e2486c8"
-					(reference "Dome?")
-					(unit 1)
-				)
+					(reference "Dome4")
+					(unit 1)
+				)

Commit message: j0
Parts:
- removed Coriolis_?: ~, symbol PID_symbols:Coriolis_Flow
- removed PT9: ~, symbol PID_symbols:Pressure_Transducer
- added BV4: ~, symbol PID_symbols:Ball_Valve
- added Burst_Disc2: ~, symbol PID_symbols:Burst_Disc
- added CF1: ~, symbol PID_symbols:Coriolis_Flow
- added CV4: ~, symbol PID_symbols:Check_Valve
- added DP1: ~, symbol PID_symbols:DP_Sensor
- added PBV1, PBV3: ~, symbol PID_symbols:Pneumatic_Rotary_Ball_Valve
- added PT5, PT68, PT69, PT70, PT71: ~, symbol PID_symbols:Pressure_Transducer
- added SPRV25, SPRV3: ~, symbol PID_symbols:SPRV
- added TC1, TC2, TC3: ~, symbol PID_symbols:Thermocouple
- added U11, U12, U13, U14, U52, U53, U54, U55, U56: ~, symbol PID_symbols:stop
- added nO_Sol24: ~, symbol PID_symbols:Normally Open Solenoid
- gave numbers to parts that had none: 5
- renumbered CV22 to CV3, Dome4 to Dome1, Pmatic_B_Valve3 to Pmatic_B_Valve2, Reg4 to Reg2, Servo_Reg4 to Servo_Reg1
Connections:
- net N2_HP: now also PBV3.; no longer Dome1.
- net N2_LP: now also PBV1., PBV3.
- net 3-8: now reaches CV2., Dome1.
- net 3-8: now also CV3., Pmatic_B_Valve2., Pmatic_B_Valve3., Reg2., T3., BV4., Burst_Disc2., CV4., PBV1., SPRV3., U12., U14., U56.
- net N2_Purge_Ox: now reaches CV3.
- net N2_Purge_Ox: no longer Pmatic_B_Valve2.
- net 1: now reaches Throttle_1.
- net 1: now also Pmatic_B_Valve4., T3., CF1., U13., U14., U52., U53., U54.; no longer CV3.
- new net: Dome1., PBV3.
- new net: BV4., PBV1., U11., U55.
- new net 1-2: U11.
- new net 1-4: DP1., Dome1., PT5., PT68., PT69., PT70., PT71., SPRV25., Servo_Reg1., TC1., TC2., TC3., U12., U13., U52., U53., U54., U55., U56., nO_Sol24.
- no-connect marks 0 -> 2
Other:
- note added: "1 INCH"
- note added: "1-2 INCH"
- note added: "1-4 INCH"
- note added: "1-8 INCH"
- note added: "3-4 INCH"
- note added: "3-8 INCH"
- note added: "Direct Connection"
- note added: "Low Pressure Pneumatics"
- note added: "Manifold"
- note added: "Torch Igniter High Pressure Line"
- note added: "Torch Igniter Pneumatics Line"
- note removed: "Top Panel"
- moved on the sheet: CV2, CV3, Pmatic_B_Valve2, Pmatic_B_Valve3, Pmatic_B_Valve4, Reg2A, Servo_Reg1B, T3B, Throttle_1

Commit message: more silwood stuff
Parts:
- removed U11, U12, U14: ~, symbol PID_symbols:stop
- added Manual_Pressure_Gauge4: ~, symbol PID_symbols:Manual_Pressure_Gauge
- added PT10: ~, symbol PID_symbols:Pressure_Transducer
- added U21, U67: ~, symbol PID_symbols:stop
- renumbered Throttle_1 to BV1, CV4 to CV2, CV2 to CV3, CV3 to CV4, PT71 to PT11, PT68 to PT12, PT69 to PT13, PT70 to PT14, PT5 to PT9, PBV3 to Pmatic_B_Valve1, PBV1 to Pmatic_B_Valve2, Pmatic_B_Valve2 to Pmatic_B_Valve5, SPRV25 to SPRV4, Reg2 to Servo_Reg2, TC1 to TC3, TC2 to TC4, TC3 to TC5, U55 to U15, U56 to U16, U13 to U18, U52 to U20, U53 to U22, U54 to U23, nO_Sol24 to nO_Sol3
Connections:
- net N2_Purge_Ox is gone; now on net 3-8: CV4.
- net 1: now also CV2.
- net 1-2: now also BV4., Pmatic_B_Valve2., SPRV3., U15.
- net 1-4: now also Manual_Pressure_Gauge4., U21., U67.
- net 3-8: now also Pmatic_B_Valve1., U21., U67.
- net N2O_Fill: now also PT10.
Other:
- moved on the sheet: Burst_Disc2, CV2, CV3, DP1, PT9, SPRV3, T3B, TC3

Commit message: bit more
Changed lines of the file:
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@@
-	(wire
-		(pts
-			(xy 193.04 169.545) (xy 194.31 169.545)
-		)
-		(stroke
-			(width 0)
-			(type default)
-		)
-	)
 	(wire
 		(pts

Commit message: Formatiing
Parts:
- removed BV4: ~, symbol PID_symbols:Ball_Valve
- removed Burst_Disc2: ~, symbol PID_symbols:Burst_Disc
- removed CF1: ~, symbol PID_symbols:Coriolis_Flow
- removed CV2: ~, symbol PID_symbols:Check_Valve
- removed DP1: ~, symbol PID_symbols:DP_Sensor
- removed Manual_Pressure_Gauge4: ~, symbol PID_symbols:Manual_Pressure_Gauge
- removed PT10, PT11, PT12, PT13, PT14: ~, symbol PID_symbols:Pressure_Transducer
- removed Pmatic_B_Valve1, Pmatic_B_Valve2: ~, symbol PID_symbols:Pneumatic_Rotary_Ball_Valve
- removed SPRV3, SPRV4: ~, symbol PID_symbols:SPRV
- removed TC3, TC4, TC5: ~, symbol PID_symbols:Thermocouple
- removed U15, U16, U18, U20, U21, U22, U23, U67: ~, symbol PID_symbols:stop
- removed nO_Sol3: ~, symbol PID_symbols:Normally Open Solenoid
- added Coriolis_?: ~, symbol PID_symbols:Coriolis_Flow
- renumbered CV4 to CV22, CV3 to CV?, Dome1 to Dome4, Pmatic_B_Valve5 to Pmatic_B_Valve3, Pmatic_B_Valve3 to Pmatic_B_Valve?, Pmatic_B_Valve4 to Pmatic_B_Valve?, Servo_Reg2 to Reg4, Servo_Reg1 to Servo_Reg4, T3 to T?, BV1 to Throttle_?
Connections:
- net N2_HP: now also Dome4.
- net at PT9.: now also Dome4., Servo_Reg4.
- removed net 1: Pmatic_B_Valve?., T?., Throttle_?.
- removed net 1-4: Dome4., PT9., Servo_Reg4.
- removed net 3-8: CV22., CV?., Dome4., Pmatic_B_Valve3., Pmatic_B_Valve?., Reg4., T?.
- new net: CV?., Dome4.
- new net: CV?., T?.
- new net: CV22., Pmatic_B_Valve3.
- new net: CV22., Throttle_?.
- new net: Coriolis_?., Pmatic_B_Valve?., T?.
- new net: Coriolis_?., Pmatic_B_Valve?.
- new net: Pmatic_B_Valve3., Reg4.
- new net: Pmatic_B_Valve?., Throttle_?.
- no-connect marks 2 -> 0
Other:
- note added: "Top Panel"
- note removed: "1 INCH"
- note removed: "1-2 INCH"
- note removed: "1-4 INCH"
- note removed: "1-8 INCH"
- note removed: "3-4 INCH"
- note removed: "3-8 INCH"
- note removed: "Direct Connection"
- note removed: "Low Pressure Pneumatics"
- note removed: "Manifold"
- note removed: "Torch Igniter High Pressure Line"
- note removed: "Torch Igniter Pneumatics Line"
- moved on the sheet: CV22, CV?, Pmatic_B_Valve3, Pmatic_B_Valve?, Reg4A, T?B, Throttle_?
