File: Silwood/J0_N2O.kicad_sch (KiCad schematic)
At the start: 38 parts

Commit message: silwood upgrade
Parts:
- added PT81: ~, symbol PID_symbols:Pressure_Transducer
- added SPRV27: ~, symbol PID_symbols:SPRV
- renumbered Burst_Disc2 to Ox_Burst_Disk
Connections:
- net 1: now also SPRV27.
- net 3-8: now also PT81.
Other:
- note added: "1_2_3 1. panel 2. component type 3. line name"
- moved on the sheet: Manual_Pressure_Gauge4

Commit message: big silwood update
Parts:
- added BV9: ~, symbol PID_symbols:Ball_Valve
- added Burst_Disc20: ~, symbol PID_symbols:Burst_Disc
- added CF5: ~, symbol PID_symbols:Coriolis_Flow
- added CV22: ~, symbol PID_symbols:Check_Valve
- added DP5: ~, symbol PID_symbols:DP_Sensor
- added Dome5: ~, symbol PID_symbols:Dome_Reg
- added Filter19: ~, symbol PID_symbols:Filter
- added MB_V9: ~, symbol PID_symbols:MBallValve
- added Manual_Pressure_Gauge17, Manual_Pressure_Gauge18, Manual_Pressure_Gauge19, Manual_Pressure_Gauge23: ~, symbol PID_symbols:Manual_Pressure_Gauge
- added PT85: ~, symbol PID_symbols:Pressure_Transducer
- added Pmatic_B_Valve13: ~, symbol PID_symbols:Pneumatic_Rotary_Ball_Valve
- added QD26: ~, symbol PID_symbols:Quick_Disconnect
- added SPRV30: ~, symbol PID_symbols:SPRV
- added Servo_Reg19, Servo_Reg5: ~, symbol PID_symbols:Pressure_Regulator
- added TC11: ~, symbol PID_symbols:Thermocouple
- added U17, U68, U71: ~, symbol PID_symbols:stop
- added nC_Sol10: ~, symbol PID_symbols:Normally_Closed_Solenoid
- added nO_Sol28: ~, symbol PID_symbols:Normally Open Solenoid
- BV1, Pmatic_B_Valve1, Pmatic_B_Valve3, Pmatic_B_Valve4, Pmatic_B_Valve5, Servo_Reg2: value ~ -> D1
- BV4, Pmatic_B_Valve2, nO_Sol3: value ~ -> D2
- renumbered SPRV27 to O_Prv_M
Connections:
- net 1: now also U17., U71.
- net 1-4: now also Manual_Pressure_Gauge17., Manual_Pressure_Gauge18., Manual_Pressure_Gauge19., U17., U68., U71.
- net 3-8: now also U68.
Other:
- note added: "(4): Optional Numbering if multiple sensors in same local feed line Smaller number is upstream."
- note added: "1: Macro location of component KEY: O: Oxidiser panel F: Fuel panel N: Outer N2 System I: Igniter PP: Pressure Panel OB: Oxidiser outside bottles"
- note added: "2: Component Type KEY: Bv: Ball Valve (servo actuated) Mbv: Manual Ball Valve Mf: Massflow control Ball Valve Pn: Pneumatic Actuated Valves Sol: Solenoid Valves PT: Pressure Transducer Tc: Thermocouple Reg: Pressure Regulator CFM: Coriolis Flow Meter PG: Pressure Gauge Tk: Tank Prv: Pressure Relief Valve BD: Burst Disk DP: Differential Pressure Sensor"
- note added: "3: Local Location feed system of Component KEY: Ref: Dome reference pressure system M: Main run line V: Venting Line T: Tank Pressurisation Line N: Nitrogen High Pressure Source Line O: Oxidiser Source Line F: Fill Line D: Drain Line P: Purge Line LP: Low Pressure Impulse Air Line"
- note added: "Burst Disk"
- note added: "Check-Valve"
- note added: "Component Naming Scheme: 1_2_3(4)"
- note added: "Coriolis Flow Meter"
- note added: "Deployment Line 1: 'D1' Run Valves on N2 lines to tanks, and main lines."
- note added: "Deployment Line 2: 'D2' All venting valves."
- note added: "Differential Pressure Transducer"
- note added: "Dome-Loaded Regulator"
- note added: "Filter"
- note added: "Manual Ball Valve"
- note added: "Normally Closed Solenoid"
- note added: "Normally Open Solenoid"
- note added: "Pneumatic Actuated Valve, NO/NC (Normally Open/Closed)"
- note added: "Pressure Gauge"
- note added: "Pressure Regulator"
- note added: "Pressure Relief Valve"
- note added: "Pressure Transducer"
- note added: "Quick-Disconnect"
- note added: "Servo Ball Valve"
- note added: "Servo-Actuated Pressure Regulator"
- note added: "Thermocouple"
- note removed: "1_2_3 1. panel 2. component type 3. line name"

Commit message: update
Parts:
- renumbered T3 to TANK
Connections:
- net 1-2: now also CV3., Dome1., Ox_Burst_Disk., Pmatic_B_Valve1., TANK., U16., U67.
- net 3-8: no longer BV4., CV3., Dome1., Ox_Burst_Disk., Pmatic_B_Valve1., Pmatic_B_Valve2., SPRV3., TANK., U16., U67.
Other:
- note added: "TANK"
Changed lines of the file:
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@@
 		)
 	)
+	(text "TANK"
+		(exclude_from_sim no)
+		(at 196.85 137.795 0)
+		(effects
+			(font
+				(size 1.27 1.27)
+			)
+			(justify left)
+		)
+	)
 	(text "Dome-Loaded \nRegulator"
 		(exclude_from_sim no)
@@
 		)
 	)
-	(global_label "3-8"
+	(global_label "1-2"
 		(shape input)
 		(at 85.725 118.11 0)
@@
 	(global_label "1"
 		(shape input)
-		(at 200.66 168.275 180)
+		(at 200.66 168.91 180)
 		(fields_autoplaced yes)
 		(effects
@@
 		)
 		(property "Intersheetrefs" "${INTERSHEET_REFS}"
-			(at 199.9515 168.275 0)
+			(at 199.9515 168.91 0)
 			(effects
 				(font
@@
 		)
 	)
-	(global_label "3-8"
+	(global_label "1-2"
 		(shape input)
 		(at 144.78 147.955 270)
@@
 		)
 	)
-	(global_label "3-8"
+	(global_label "1-2"
 		(shape input)
 		(at 125.095 118.11 180)
@@
 		(on_board yes)
 		(dnp no)
-		(property "Reference" "T3"
+		(property "Reference" "TANK"
 			(at 197.485 137.16 0)
 			(effects
@@
 			(project "P_IDs"
 				(path "/045f1f05-3134-4b6d-91b6-463031104f1e/a0b6300e-76e9-4a18-afd6-e2d656b0d8f9/d375e00a-1ce3-4f93-9279-82acf09c7292/343346ed-3011-4de4-9739-8cfc7e2486c8"
-					(reference "T3")
+					(reference "TANK")
 					(unit 2)
 				)
