File: Silwood/PressurePanel.kicad_sch (KiCad schematic)
At the start: 10 parts

Commit message: update
Parts:
- gave numbers to parts that had none: 10
Connections:
- net at QD4.: now also MB_V16., MB_V17., Manual_Pressure_Gauge8., Servo_Reg2.
- new net: MB_V14., MB_V15., Manual_Pressure_Gauge7., QD3., Servo_Reg2.
- now unconnected: MB_V15., MB_V16., Manual_Pressure_Gauge7., Manual_Pressure_Gauge8., QD3.
Changed lines of the file:
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@@
 		(dnp no)
 		(fields_autoplaced yes)
-		(property "Reference" "MB_V?"
+		(property "Reference" "MB_V14"
 			(at 65.405 76.835 0)
 			(effects
@@
 			(project "P_IDs"
 				(path "/045f1f05-3134-4b6d-91b6-463031104f1e/a0b6300e-76e9-4a18-afd6-e2d656b0d8f9/d375e00a-1ce3-4f93-9279-82acf09c7292/4035a438-db16-4119-8b4d-f938f5ee1d69"
-					(reference "MB_V?")
+					(reference "MB_V14")
 					(unit 1)
 				)
@@
 		(on_board yes)
 		(dnp no)
-		(property "Reference" "QD?"
+		(property "Reference" "QD4"
 			(at 162.56 97.155 90)
 			(effects
@@
 			(project "P_IDs"
 				(path "/045f1f05-3134-4b6d-91b6-463031104f1e/a0b6300e-76e9-4a18-afd6-e2d656b0d8f9/d375e00a-1ce3-4f93-9279-82acf09c7292/4035a438-db16-4119-8b4d-f938f5ee1d69"
-					(reference "QD?")
+					(reference "QD4")
 					(unit 1)
 				)
@@
 		(on_board yes)
 		(dnp no)
-		(property "Reference" "Manual_Pressure_Gauge?"
+		(property "Reference" "Manual_Pressure_Gauge8"
 			(at 123.19 66.04 90)
 			(effects
@@
 			(project "P_IDs"
 				(path "/045f1f05-3134-4b6d-91b6-463031104f1e/a0b6300e-76e9-4a18-afd6-e2d656b0d8f9/d375e00a-1ce3-4f93-9279-82acf09c7292/4035a438-db16-4119-8b4d-f938f5ee1d69"
-					(reference "Manual_Pressure_Gauge?")
+					(reference "Manual_Pressure_Gauge8")
 					(unit 1)
 				)
@@
 		(dnp no)
 		(fields_autoplaced yes)
-		(property "Reference" "Servo_Reg?"
+		(property "Reference" "Servo_Reg2"
 			(at 118.1725 74.93 0)
 			(effects
@@
 			(project "P_IDs"
 				(path "/045f1f05-3134-4b6d-91b6-463031104f1e/a0b6300e-76e9-4a18-afd6-e2d656b0d8f9/d375e00a-1ce3-4f93-9279-82acf09c7292/4035a438-db16-4119-8b4d-f938f5ee1d69"
-					(reference "Servo_Reg?")
+					(reference "Servo_Reg2")
 					(unit 1)
 				)
@@
 		(dnp no)
 		(fields_autoplaced yes)
-		(property "Reference" "MB_V?"
+		(property "Reference" "MB_V17"
 			(at 167.005 77.47 0)
 			(effects
@@
 			(project "P_IDs"
 				(path "/045f1f05-3134-4b6d-91b6-463031104f1e/a0b6300e-76e9-4a18-afd6-e2d656b0d8f9/d375e00a-1ce3-4f93-9279-82acf09c7292/4035a438-db16-4119-8b4d-f938f5ee1d69"
-					(reference "MB_V?")
+					(reference "MB_V17")
 					(unit 1)
 				)
@@
 		(dnp no)
 		(fields_autoplaced yes)
-		(property "Reference" "SPRV?"
+		(property "Reference" "SPRV3"
 			(at 185.42 66.6749 90)
 			(effects
@@
 			(project "P_IDs"
 				(path "/045f1f05-3134-4b6d-91b6-463031104f1e/a0b6300e-76e9-4a18-afd6-e2d656b0d8f9/d375e00a-1ce3-4f93-9279-82acf09c7292/4035a438-db16-4119-8b4d-f938f5ee1d69"
-					(reference "SPRV?")
+					(reference "SPRV3")
 					(unit 1)
 				)
@@
 		(dnp no)
 		(fields_autoplaced yes)
-		(property "Reference" "MB_V?"
+		(property "Reference" "MB_V16"
 			(at 138.43 94.6149 90)
 			(effects
@@
 			(project "P_IDs"
 				(path "/045f1f05-3134-4b6d-91b6-463031104f1e/a0b6300e-76e9-4a18-afd6-e2d656b0d8f9/d375e00a-1ce3-4f93-9279-82acf09c7292/4035a438-db16-4119-8b4d-f938f5ee1d69"
-					(reference "MB_V?")
+					(reference "MB_V16")
 					(unit 1)
 				)
@@
 		(on_board yes)
 		(dnp no)
-		(property "Reference" "Manual_Pressure_Gauge?"
+		(property "Reference" "Manual_Pressure_Gauge7"
 			(at 73.025 69.215 90)
 			(effects
@@
 			(project "P_IDs"
 				(path "/045f1f05-3134-4b6d-91b6-463031104f1e/a0b6300e-76e9-4a18-afd6-e2d656b0d8f9/d375e00a-1ce3-4f93-9279-82acf09c7292/4035a438-db16-4119-8b4d-f938f5ee1d69"
-					(reference "Manual_Pressure_Gauge?")
+					(reference "Manual_Pressure_Gauge7")
 					(unit 1)
 				)
@@
 		(dnp no)
 		(fields_autoplaced yes)
-		(property "Reference" "QD?"
+		(property "Reference" "QD3"
 			(at 81.28 90.8049 90)
 			(effects
@@
 			(project "P_IDs"
 				(path "/045f1f05-3134-4b6d-91b6-463031104f1e/a0b6300e-76e9-4a18-afd6-e2d656b0d8f9/d375e00a-1ce3-4f93-9279-82acf09c7292/4035a438-db16-4119-8b4d-f938f5ee1d69"
-					(reference "QD?")
+					(reference "QD3")
 					(unit 1)
 				)
@@
 		(dnp no)
 		(fields_autoplaced yes)
-		(property "Reference" "MB_V?"
+		(property "Reference" "MB_V15"
 			(at 104.14 93.9799 90)
 			(effects
@@
 			(project "P_IDs"
 				(path "/045f1f05-3134-4b6d-91b6-463031104f1e/a0b6300e-76e9-4a18-afd6-e2d656b0d8f9/d375e00a-1ce3-4f93-9279-82acf09c7292/4035a438-db16-4119-8b4d-f938f5ee1d69"
-					(reference "MB_V?")
-					(unit 1)
-				)
+					(reference "MB_V15")
+					(unit 1)
+				)

Commit message: j0
Parts:
- renumbered MB_V14 to MB_V1, MB_V17 to MB_V2, MB_V15 to MB_V3, MB_V16 to MB_V4, Manual_Pressure_Gauge8 to Manual_Pressure_Gauge1, Manual_Pressure_Gauge7 to Manual_Pressure_Gauge2, QD3 to QD1, QD4 to QD2, SPRV3 to SPRV1, Servo_Reg2 to Servo_Reg1
Connections:
- net N2_LP is gone; now on net 3-8: MB_V2., SPRV1.
- net 1-4: now reaches MB_V1., MB_V3., Manual_Pressure_Gauge2., QD1., Servo_Reg1.
- net 1-4: now also MB_V2., MB_V4., Manual_Pressure_Gauge1., QD2.
- net 3-8: now reaches SPRV1.

Commit message: more silwood stuff
Parts:
- renumbered MB_V3 to MB_V2, MB_V4 to MB_V3, MB_V2 to MB_V4, Manual_Pressure_Gauge2 to Manual_Pressure_Gauge1, Manual_Pressure_Gauge1 to Manual_Pressure_Gauge2
Changed lines of the file:
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@@
 	)
 	(symbol
+		(lib_name "MBallValve_2")
 		(lib_id "PID_symbols:MBallValve")
 		(at 65.405 83.185 0)
@@
 					(size 1.27 1.27)
 				)
+				(hide yes)
 			)
 		)
@@
 					(size 1.27 1.27)
 				)
-				(hide yes)
 			)
 		)
@@
 				)
 				(justify left)
+				(hide yes)
 			)
 		)
@@
 					(size 1.27 1.27)
 				)
-				(hide yes)
 			)
 		)
@@
 	)
 	(symbol
+		(lib_name "Manual_Pressure_Gauge_1")
 		(lib_id "PID_symbols:Manual_Pressure_Gauge")
 		(at 134.62 70.485 90)
@@
 		(on_board yes)
 		(dnp no)
-		(property "Reference" "Manual_Pressure_Gauge1"
+		(property "Reference" "Manual_Pressure_Gauge2"
 			(at 123.19 66.04 90)
 			(effects
@@
 				)
 				(justify right)
+				(hide yes)
 			)
 		)
@@
 					(size 1.27 1.27)
 				)
-				(hide yes)
-			)
-		)
-		(pin ""
-		)
-		(pin ""
-		)
-		(instances
-			(project "P_IDs"
-				(path "/045f1f05-3134-4b6d-91b6-463031104f1e/a0b6300e-76e9-4a18-afd6-e2d656b0d8f9/d375e00a-1ce3-4f93-9279-82acf09c7292/4035a438-db16-4119-8b4d-f938f5ee1d69"
-					(reference "Manual_Pressure_Gauge1")
+			)
+		)
+		(pin ""
+		)
+		(pin ""
+		)
+		(instances
+			(project "P_IDs"
+				(path "/045f1f05-3134-4b6d-91b6-463031104f1e/a0b6300e-76e9-4a18-afd6-e2d656b0d8f9/d375e00a-1ce3-4f93-9279-82acf09c7292/4035a438-db16-4119-8b4d-f938f5ee1d69"
+					(reference "Manual_Pressure_Gauge2")
 					(unit 1)
 				)
@@
 					(size 1.27 1.27)
 				)
+				(hide yes)
 			)
 		)
@@
 					(size 1.27 1.27)
 				)
-				(hide yes)
 			)
 		)
@@
 		(dnp no)
 		(fields_autoplaced yes)
-		(property "Reference" "MB_V2"
+		(property "Reference" "MB_V4"
 			(at 167.005 77.47 0)
 			(effects
@@
 					(size 1.27 1.27)
 				)
+				(hide yes)
 			)
 		)
@@
 					(size 1.27 1.27)
 				)
-				(hide yes)
-			)
-		)
-		(pin ""
-		)
-		(pin ""
-		)
-		(instances
-			(project "P_IDs"
-				(path "/045f1f05-3134-4b6d-91b6-463031104f1e/a0b6300e-76e9-4a18-afd6-e2d656b0d8f9/d375e00a-1ce3-4f93-9279-82acf09c7292/4035a438-db16-4119-8b4d-f938f5ee1d69"
-					(reference "MB_V2")
+			)
+		)
+		(pin ""
+		)
+		(pin ""
+		)
+		(instances
+			(project "P_IDs"
+				(path "/045f1f05-3134-4b6d-91b6-463031104f1e/a0b6300e-76e9-4a18-afd6-e2d656b0d8f9/d375e00a-1ce3-4f93-9279-82acf09c7292/4035a438-db16-4119-8b4d-f938f5ee1d69"
+					(reference "MB_V4")
 					(unit 1)
 				)
@@
 				)
 				(justify right)
+				(hide yes)
 			)
 		)
@@
 					(size 1.27 1.27)
 				)
-				(hide yes)
 			)
 		)
@@
 	)
 	(symbol
-		(lib_name "MBallValve_2")
+		(lib_name "MBallValve_3")
 		(lib_id "PID_symbols:MBallValve")
 		(at 134.62 95.25 90)
@@
 		(dnp no)
 		(fields_autoplaced yes)
-		(property "Reference" "MB_V4"
+		(property "Reference" "MB_V3"
 			(at 138.43 94.6149 90)
 			(effects
@@
 				)
 				(justify right)
+				(hide yes)
 			)
 		)
@@
 					(size 1.27 1.27)
 				)
-				(hide yes)
-			)
-		)
-		(pin ""
-		)
-		(pin ""
-		)
-		(instances
-			(project "P_IDs"
-				(path "/045f1f05-3134-4b6d-91b6-463031104f1e/a0b6300e-76e9-4a18-afd6-e2d656b0d8f9/d375e00a-1ce3-4f93-9279-82acf09c7292/4035a438-db16-4119-8b4d-f938f5ee1d69"
-					(reference "MB_V4")
-					(unit 1)
-				)
-			)
-		)
-	)
-	(symbol
-		(lib_name "Manual_Pressure_Gauge_1")
+			)
+		)
+		(pin ""
+		)
+		(pin ""
+		)
+		(instances
+			(project "P_IDs"
+				(path "/045f1f05-3134-4b6d-91b6-463031104f1e/a0b6300e-76e9-4a18-afd6-e2d656b0d8f9/d375e00a-1ce3-4f93-9279-82acf09c7292/4035a438-db16-4119-8b4d-f938f5ee1d69"
+					(reference "MB_V3")
+					(unit 1)
+				)
+			)
+		)
+	)
+	(symbol
 		(lib_id "PID_symbols:Manual_Pressure_Gauge")
 		(at 84.455 73.66 90)
@@
 		(on_board yes)
 		(dnp no)
-		(property "Reference" "Manual_Pressure_Gauge2"
+		(property "Reference" "Manual_Pressure_Gauge1"
 			(at 73.025 69.215 90)
 			(effects
@@
 				)
 				(justify right)
+				(hide yes)
 			)
 		)
@@
 					(size 1.27 1.27)
 				)
-				(hide yes)
-			)
-		)
-		(pin ""
-		)
-		(pin ""
-		)
-		(instances
-			(project "P_IDs"
-				(path "/045f1f05-3134-4b6d-91b6-463031104f1e/a0b6300e-76e9-4a18-afd6-e2d656b0d8f9/d375e00a-1ce3-4f93-9279-82acf09c7292/4035a438-db16-4119-8b4d-f938f5ee1d69"
-					(reference "Manual_Pressure_Gauge2")
+			)
+		)
+		(pin ""
+		)
+		(pin ""
+		)
+		(instances
+			(project "P_IDs"
+				(path "/045f1f05-3134-4b6d-91b6-463031104f1e/a0b6300e-76e9-4a18-afd6-e2d656b0d8f9/d375e00a-1ce3-4f93-9279-82acf09c7292/4035a438-db16-4119-8b4d-f938f5ee1d69"
+					(reference "Manual_Pressure_Gauge1")
 					(unit 1)
 				)
@@
 				)
 				(justify left)
+				(hide yes)
 			)
 		)
@@
 					(size 1.27 1.27)
 				)
-				(hide yes)
 			)
 		)
@@
 	)
 	(symbol
-		(lib_name "MBallValve_3")
 		(lib_id "PID_symbols:MBallValve")
 		(at 100.33 94.615 90)
@@
 		(dnp no)
 		(fields_autoplaced yes)
-		(property "Reference" "MB_V3"
+		(property "Reference" "MB_V2"
 			(at 104.14 93.9799 90)
 			(effects
@@
 				)
 				(justify right)
+				(hide yes)
 			)
 		)
@@
 					(size 1.27 1.27)
 				)
-				(hide yes)
-			)
-		)
-		(pin ""
-		)
-		(pin ""
-		)
-		(instances
-			(project "P_IDs"
-				(path "/045f1f05-3134-4b6d-91b6-463031104f1e/a0b6300e-76e9-4a18-afd6-e2d656b0d8f9/d375e00a-1ce3-4f93-9279-82acf09c7292/4035a438-db16-4119-8b4d-f938f5ee1d69"
-					(reference "MB_V3")
-					(unit 1)
-				)
+			)
+		)
+		(pin ""
+		)
+		(pin ""
+		)
+		(instances
+			(project "P_IDs"
+				(path "/045f1f05-3134-4b6d-91b6-463031104f1e/a0b6300e-76e9-4a18-afd6-e2d656b0d8f9/d375e00a-1ce3-4f93-9279-82acf09c7292/4035a438-db16-4119-8b4d-f938f5ee1d69"
+					(reference "MB_V2")
+					(unit 1)
+				)

Commit message: Formatiing
Parts:
- renumbered MB_V1 to MB_V14, MB_V2 to MB_V15, MB_V3 to MB_V16, MB_V4 to MB_V17, Manual_Pressure_Gauge1 to Manual_Pressure_Gauge7, Manual_Pressure_Gauge2 to Manual_Pressure_Gauge8, QD1 to QD3, QD2 to QD4, SPRV1 to SPRV3, Servo_Reg1 to Servo_Reg2
Connections:
- net 3-8 is gone; now on net N2_LP: MB_V17., SPRV3.
- net at QD4.: now also MB_V16., MB_V17., Manual_Pressure_Gauge8., Servo_Reg2.
- net N2_LP: now reaches SPRV3.
- removed net 1-4: MB_V14., MB_V15., MB_V16., MB_V17., Manual_Pressure_Gauge7., Manual_Pressure_Gauge8., QD3., QD4., Servo_Reg2.
- new net: MB_V14., MB_V15., Manual_Pressure_Gauge7., QD3., Servo_Reg2.
