File: Silwood/PressurePanel.kicad_sch (KiCad schematic)
At the start: 10 parts

Commit message: silwood upgrade
Other:
- moved on the sheet: QD1
Changed lines of the file:
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@@
 	(wire
 		(pts
-			(xy 84.455 88.265) (xy 84.455 83.185)
+			(xy 84.455 92.075) (xy 84.455 83.185)
 		)
 		(stroke
@@
 					(size 1.27 1.27)
 				)
+				(hide yes)
 			)
 		)
@@
 		(lib_name "Quick_Disconnect_1")
 		(lib_id "PID_symbols:Quick_Disconnect")
-		(at 84.455 92.075 90)
+		(at 84.455 95.885 90)
 		(unit 1)
 		(exclude_from_sim no)
@@
 		(fields_autoplaced yes)
 		(property "Reference" "QD1"
-			(at 81.28 90.8049 90)
+			(at 81.28 94.6149 90)
 			(effects
 				(font
@@
 		)
 		(property "Value" "~"
-			(at 81.28 92.71 90)
+			(at 81.28 96.52 90)
 			(effects
 				(font
@@
 		)
 		(property "Footprint" ""
-			(at 84.455 92.075 0)
-			(effects
-				(font
-					(size 1.27 1.27)
-				)
-				(hide yes)
-			)
-		)
-		(property "Datasheet" ""
-			(at 84.455 92.075 0)
+			(at 84.455 95.885 0)
+			(effects
+				(font
+					(size 1.27 1.27)
+				)
+				(hide yes)
+			)
+		)
+		(property "Datasheet" ""
+			(at 84.455 95.885 0)
 			(effects
 				(font
@@
 		)
 		(property "Description" ""
-			(at 84.455 92.075 0)
-			(effects
-				(font
+			(at 84.455 95.885 0)
+			(effects
+				(font

Commit message: big silwood update
Parts:
- added BV44: ~, symbol PID_symbols:Ball_Valve
- added Burst_Disc23: ~, symbol PID_symbols:Burst_Disc
- added CF8: ~, symbol PID_symbols:Coriolis_Flow
- added CV25: ~, symbol PID_symbols:Check_Valve
- added DP8: ~, symbol PID_symbols:DP_Sensor
- added Dome8: ~, symbol PID_symbols:Dome_Reg
- added Filter22: ~, symbol PID_symbols:Filter
- added MB_V19: ~, symbol PID_symbols:MBallValve
- added Manual_Pressure_Gauge26: ~, symbol PID_symbols:Manual_Pressure_Gauge
- added PT88: ~, symbol PID_symbols:Pressure_Transducer
- added Pmatic_B_Valve16: ~, symbol PID_symbols:Pneumatic_Rotary_Ball_Valve
- added QD29: ~, symbol PID_symbols:Quick_Disconnect
- added SPRV33: ~, symbol PID_symbols:SPRV
- added Servo_Reg22, Servo_Reg8: ~, symbol PID_symbols:Pressure_Regulator
- added TC14: ~, symbol PID_symbols:Thermocouple
- added nC_Sol13: ~, symbol PID_symbols:Normally_Closed_Solenoid
- added nO_Sol31: ~, symbol PID_symbols:Normally Open Solenoid
- renumbered MB_V1 to PP_MBV_N, MB_V2 to PP_MBV_V
Other:
- note added: "(4): Optional Numbering if multiple sensors in same local feed line Smaller number is upstream."
- note added: "1 INCH"
- note added: "1-2 INCH"
- note added: "1-4 INCH"
- note added: "1-8 INCH"
- note added: "1: Macro location of component KEY: O: Oxidiser panel F: Fuel panel N: Outer N2 System I: Igniter PP: Pressure Panel OB: Oxidiser outside bottles"
- note added: "2: Component Type KEY: Bv: Ball Valve (servo actuated) Mbv: Manual Ball Valve Mf: Massflow control Ball Valve Pn: Pneumatic Actuated Valves Sol: Solenoid Valves PT: Pressure Transducer Tc: Thermocouple Reg: Pressure Regulator CFM: Coriolis Flow Meter PG: Pressure Gauge Tk: Tank Prv: Pressure Relief Valve BD: Burst Disk DP: Differential Pressure Sensor"
- note added: "3-4 INCH"
- note added: "3-8 INCH"
- note added: "3: Local Location feed system of Component KEY: Ref: Dome reference pressure system M: Main run line V: Venting Line T: Tank Pressurisation Line N: Nitrogen High Pressure Source Line O: Oxidiser Source Line F: Fill Line D: Drain Line P: Purge Line LP: Low Pressure Impulse Air Line"
- note added: "Burst Disk"
- note added: "Check-Valve"
- note added: "Component Naming Scheme: 1_2_3(4)"
- note added: "Coriolis Flow Meter"
- note added: "Deployment Line 1: 'D1' Run Valves on N2 lines to tanks, and main lines."
- note added: "Deployment Line 2: 'D2' All venting valves."
- note added: "Differential Pressure Transducer"
- note added: "Direct Connection"
- note added: "Dome-Loaded Regulator"
- note added: "Filter"
- note added: "Low Pressure Pneumatics"
- note added: "Manual Ball Valve"
- note added: "Normally Closed Solenoid"
- note added: "Normally Open Solenoid"
- note added: "Pneumatic Actuated Valve, NO/NC (Normally Open/Closed)"
- note added: "Pressure Gauge"
- note added: "Pressure Regulator"
- note added: "Pressure Relief Valve"
- note added: "Pressure Transducer"
- note added: "Quick-Disconnect"
- note added: "Servo Ball Valve"
- note added: "Servo-Actuated Pressure Regulator"
- note added: "Thermocouple"
- note added: "Torch Igniter High Pressure Line"
- note added: "Torch Igniter Pneumatics Line"
